File: Power/LabPower/LabPower-power.brd (EAGLE design)
At the start: 92.7 x 172.7 mm, 82 parts, among them IC1 TNY264PN, IC2 TL494CD, Q1 STP11NM60ND, Q2 STP11NM60ND, T1 GDT_20X6.5, X1 MKDSN1,5/2-5,08

Commit message: _
Parts:
- removed C10: 1u, rcl:C0805
- removed C18: 2700u 63V, rcl:E7,5-18
- removed C20: 10n, rcl:C0805
- removed C7: 1n, rcl:C0805
- removed C8: 10u, rcl:C0805
- removed C9: 100n, rcl:C0805
- removed DRILEGEND: (no value), drilegend:DRILEGEND
- removed IC2: TL494CD, linear:SO16
- removed JP1: (no value), pinhead:1X08
- removed OUT-CUR, OUT-CUR1: (no value), pinhead:1X02
- removed R10, R8: 0, rcl:R1206
- removed R11: 4K7, rcl:R0805
- removed R13: 6K8, rcl:R0805
- removed R14, R15: 5K1, rcl:R0805
- removed R21, R22: 10K, rcl:R0805
- removed R23: 3R3, rcl:R1206
- removed R9: 51K, rcl:R0805
- removed U$2: IR2113SPBF, Namenlos:SO16W
- removed V+, V0: (no value), wirepad:3,81/1,4
- added JP3: (no value), pinhead:1X08
- added X2: MKDSN1,5/3-5,08, Namenlos:MKDSN1,5/3-5,08
- U$7, U$8: value SK95-3M3 -> (none); device heatsink:SK95-3M3 -> heatsink:SK95-3M3_HOLE
- X1: value MKDSN1,5/2-5,08 -> MKDSN1,5/3-5,08; device con-phoenix-508:MKDSN1,5/2-5,08 -> Namenlos:MKDSN1,5/3-5,08
- moved U$8 209.8 mm to (-29.8, -121.3)
- moved C19 204.0 mm to (-85.1, -106.0), turned to 270 degrees
- moved X1 203.6 mm to (-88.3, -5.71)
- moved R32 203.2 mm to (-83.6, -117.0), turned to 180 degrees
- moved D1 202.8 mm to (-45.1, -69.2)
- moved D10 202.8 mm to (-83.8, -48.9)
- moved F1 202.8 mm to (-78.7, -15.2)
- moved Q1 202.8 mm to (-10.8, -64.1)
- moved Q2 202.8 mm to (-29.8, -64.1)
- moved R19 202.8 mm to (-89.5, -48.9)
- moved R27 202.8 mm to (-15.2, -73.0)
- moved R5 202.8 mm to (-28.6, -13.6)
- moved T1 202.8 mm to (-32.4, -52.7)
- moved U$1 202.8 mm to (-29.8, -64.1)
- moved U$3 202.8 mm to (-10.8, -64.1)
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Connections:
- removed net +I1: IC2.1, R10.2
- removed net +I2: IC2.16, R8.2
- removed net COM: C10.1, C7.1, C9.1, IC2.7, JP1.2, JP1.5, R11.2, R13.2, R15.2, R21.2, R22.2, U$2.13, U$2.15, U$2.2, U$2.6
- removed net DTC: C8.1, IC2.4, JP1.6, R13.1
- removed net HO: JP1.3, R23.2
- removed net LO: JP1.4, U$2.1
- removed net N$11: C20.1, R9.1
- removed net N$12: C20.2, IC2.3
- removed net N$13: JP1.8, R10.1
- removed net N$14: IC2.6, R11.1
- removed net N$15: JP1.7, R8.1
- removed net N$16: C7.2, IC2.5
- removed net N$19: IC2.15, IC2.2, R14.2, R15.1, R9.2
- removed net N$25: IC2.10, R21.1, U$2.12
- removed net N$29: IC2.9, R22.1, U$2.14
- removed net N$31: C4.-, JP2.2, JP2.5, OK1.2, R20.1, R7.1, T2.S0, U$4.2-2
- removed net N$34: C18.+, C19.+, R32.2, U$6.7, U$6.8, U$6.9, V+.1
- removed net N$37: OUT-CUR.1, OUT-CUR.2, R31.P$2, V0.1
- removed net N$4: R23.1, U$2.8
- removed net N$41: C4.+, D10.C, D9.C, JP2.1
- removed net N$8: C8.2, C9.2, IC2.13, IC2.14, R14.1
- removed net VCC: C10.2, IC2.11, IC2.12, IC2.8, JP1.1, U$2.11, U$2.3, U$2.7
- new net +12: C4.+, D10.C, D9.C, JP2.1, JP3.1
- new net I-FB: JP2.8, JP3.8
- new net OUT+: C19.+, JP3.4, R32.2, U$6.7, U$6.8, U$6.9, X2.3
- new net OUT-/CUR+: JP3.3, JP3.5, R31.P$2, X2.1
- new net V-FB: JP2.7, JP3.7
- net GND: now also C4.-, JP2.2, JP2.5, JP3.2, JP3.6, OK1.2, R20.1, R7.1, T2.S0, U$4.2-2, U$5.10, U$5.11, U$5.12; no longer C18.-, OUT-CUR1.1, OUT-CUR1.2
- net LOWS+: now also U$5.14
- net LOWS-: now also U$5.8
- net N$6: now also X1.3; no longer X1.2
Routing:
- net GND: track 0.00 -> 279.2 mm
- net COM: track 111.2 -> 0.00 mm
- net VCC: track 89.8 -> 0.00 mm
- net N$31: track 82.3 -> 0.00 mm
- net +12: track 0.00 -> 82.3 mm
- net OUT+: track 0.00 -> 79.0 mm
- net OUT-/CUR+: track 0.00 -> 63.9 mm
- net N$26: track 0.00 -> 58.4 mm
- net DTC: track 40.1 -> 0.00 mm
- net V-FB: track 0.00 -> 39.1 mm
- net N$41: track 38.5 -> 0.00 mm
- net I-FB: track 0.00 -> 34.4 mm
- net N$8: track 32.6 -> 0.00 mm
- net N$29: track 20.6 -> 0.00 mm
- net N$19: track 20.5 -> 0.00 mm
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Other:
- board size 92.7 x 172.7 mm -> 97.8 x 128.9 mm

Commit message: _+
Parts:
- added C7: 2700u 63V, rcl:E7,5-18
- JP2, JP3: device pinhead:1X08 -> pinhead:1X10
- moved X2 55.4 mm to (-98.4, -69.8), turned to 270 degrees
- moved X1 14.9 mm to (-102.2, -10.8), turned to 270 degrees
- moved JP3 12.7 mm to (-73.0, -73.7)
- moved R32 11.3 mm to (-91.6, -109.0), turned to 0 degrees
- moved C19 9.92 mm to (-91.4, -98.4), turned to 180 degrees
- moved R31 7.10 mm to (-73.0, -83.2)
- moved JP2 4.02 mm to (-50.2, -56.5)
- moved R3 3.81 mm to (-78.7, -5.71)
- moved C4 3.70 mm to (-58.4, -45.7)
- moved D10 3.24 mm to (-87.0, -48.3)
- moved F1 3.24 mm to (-81.9, -14.6)
- moved R12 3.24 mm to (-74.9, -21.0)
- moved C2 3.24 mm to (-64.1, -27.3)
- moved B2 3.24 mm to (-37.5, -12.1)
- moved CX1 3.24 mm to (-64.1, -10.2)
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Connections:
- net I-FB renamed -V-FB
- net V-FB renamed +V-FB
- removed net OUT+: C19.+, JP3.4, R32.2, U$6.7, U$6.8, U$6.9, X2.3
- removed net OUT-/CUR+: JP3.3, JP3.5, R31.P$2, X2.1
- new net +I-FB: JP2.9, JP3.9
- new net -I-FB: JP2.10, JP3.10
- new net CUR+: C19.+, C7.+, JP3.6, R31.P$1, R32.2, U$6.7, U$6.8, U$6.9
- new net OUT+\CUR-: JP3.3, JP3.5, R31.P$2, X2.3
- net GND: now also C7.-, JP3.4, X2.1; no longer JP3.6, R31.P$1
Routing:
- net CUR+: track 0.00 -> 143.2 mm
- net OUT+: track 79.0 -> 0.00 mm
- net GND: track 279.2 -> 348.3 mm
- net OUT+\CUR-: track 0.00 -> 68.5 mm
- net OUT-/CUR+: track 63.9 -> 0.00 mm
- net +I-FB: track 0.00 -> 20.4 mm
- net -I-FB: track 0.00 -> 16.7 mm
- net N$7: track 4.53 -> 19.7 mm
- net +V-FB: track 39.1 -> 29.0 mm
- net -V-FB: track 34.4 -> 24.7 mm
- net +12: track 82.3 -> 88.1 mm
- net N$22: track 8.67 -> 13.0 mm
- net N$18: track 8.67 -> 12.0 mm
- net N$38: track 0.00 -> 2.39 mm
- net 300V: track 92.9 -> 95.2 mm
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Other:
- board size 97.8 x 128.9 mm -> 108 x 130.2 mm

Commit message: Some Changes
Parts:
- removed R31: 0R1, Namenlos:SQP-10
- added R10, R8, R9: N-Wire 39.6x0.5mm 0.3Om, rcl:0207/10
- moved X2 11.4 mm to (-94.6, -80.6)
- moved X1 11.1 mm to (-92.7, -5.08), turned to 180 degrees
- moved C1 1.25 mm to (-8.11, -39.6), turned to 270 degrees
- moved R3 0.90 mm to (-78.1, -5.08)
Connections:
- net CUR+: now also R10.1, R8.1, R9.1; no longer R31.P$1
- net OUT+\CUR-: now also R10.2, R8.2, R9.2; no longer R31.P$2
Routing:
- net CUR+: track 143.2 -> 114.4 mm
- net GND: track 348.3 -> 323.7 mm
- net OUT+\CUR-: track 68.5 -> 53.6 mm
- net N$7: track 19.7 -> 5.79 mm
- net N$1: track 45.1 -> 47.9 mm
- net N$3: track 33.5 -> 36.3 mm
- net N$6: track 9.50 -> 11.4 mm
- net 300V: track 95.2 -> 96.8 mm
- net N$9: track 20.0 -> 19.1 mm
Other:
- board size 108 x 130.2 mm -> 102.2 x 130.2 mm

Commit message: Final design
I hope...
Parts:
- added C10: (no value), rcl:E2,5-7
- added C8, C9: 330u 200V, rcl:EB22,5D
- moved C4 31.3 mm to (-88.3, -55.2), turned to 180 degrees
- moved C6 25.1 mm to (-34.9, -11.4)
- moved R5 21.5 mm to (-13.3, -24.1), turned to 0 degrees
- moved D9 18.2 mm to (-83.2, -49.5), turned to 90 degrees
- moved C1 13.6 mm to (-13.8, -51.9), turned to 0 degrees
- moved B2 12.1 mm to (-49.5, -13.3)
- moved R4 11.5 mm to (-55.2, -13.3)
- moved B1 11.0 mm to (-62.9, -33.4), turned to 90 degrees
- moved R12 11.0 mm to (-85.7, -19.1), turned to 270 degrees
- moved R19 9.92 mm to (-100.3, -41.9)
- moved D10 9.90 mm to (-96.9, -48.3), turned to 135 degrees
- moved R16 9.71 mm to (-88.3, -19.1), turned to 90 degrees
- moved C2 8.98 mm to (-73.0, -26.0)
- moved R17 8.47 mm to (-90.8, -19.1), turned to 270 degrees
- moved L1 8.35 mm to (-60.3, -13.3)
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Connections:
- net +12: now also C10.+
- net 300V: now also C8.+
- net GND: now also C10.-
- net N$1: now also C8.-, C9.+
- net N$17: now also C9.-
Routing:
- net N$1: track 47.9 -> 74.4 mm
- net GND: track 323.7 -> 308.3 mm
- net +12: track 88.1 -> 77.3 mm
- net N$50: track 2.59 -> 12.3 mm
- net N$17: track 74.9 -> 82.6 mm
- net 300V: track 96.8 -> 103.0 mm
- net N$48: track 7.33 -> 1.65 mm
- net -I-FB: track 16.7 -> 12.2 mm
- net N$24: track 5.17 -> 9.46 mm
- net -V-FB: track 24.7 -> 20.9 mm
- net +V-FB: track 29.0 -> 25.2 mm
- net +I-FB: track 20.4 -> 16.6 mm
- net N$3: track 36.3 -> 32.5 mm
- net N$9: track 19.1 -> 15.5 mm
- net AC2: track 24.6 -> 27.7 mm
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- added copper zone on layer 16, net N$4
- added copper zone on layer 16, net N$8
