File: Power/LabPower/LabPower-FB_V2.brd (EAGLE design)
At the start: 27.3 x 38.1 mm, 25 parts, among them IC1 INA168, IC2 LD117ASTR, U1 TSV621ILT

Commit message: Опять всё неправильно сделал
Parts:
- moved R7 24.9 mm to (-8.26, -27.9), flipped to the bottom, turned to 270 degrees
- moved JP1 24.0 mm to (10.8, -31.8), turned to 180 degrees
- moved R5 22.4 mm to (-10.8, -21.0), turned to 180 degrees
- moved U$1 22.4 mm to (-10.8, -17.8), turned to 180 degrees
- moved R8 21.1 mm to (-12.1, -11.4), turned to 180 degrees
- moved R9 21.1 mm to (-13.3, -16.5), turned to 90 degrees
- moved IC2 21.0 mm to (19.1, -24.1), turned to 180 degrees
- moved R4 19.7 mm to (-8.89, -12.7), turned to 90 degrees
- moved R12 19.7 mm to (14.6, -26.7), turned to 270 degrees
- moved R17 18.5 mm to (-6.99, -21.0), turned to 180 degrees
- moved R6 18.2 mm to (-8.26, -16.5), turned to 90 degrees
- moved R14 16.4 mm to (19.7, -15.9), turned to 270 degrees
- moved JP2 15.5 mm to (4.76, -31.8), turned to 180 degrees
- moved C1 14.0 mm to (14.0, -22.2), turned to 90 degrees
- moved R1 13.7 mm to (17.1, -12.7), turned to 90 degrees
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Connections:
- new net N$11: IC1.5, U1.5
- net N$9: no longer IC1.5, U1.5
Routing:
- net GND: track 47.5 -> 0.00 mm
- net +12V: track 43.1 -> 2.04 mm
- net N$9: track 24.1 -> 0.00 mm
- net -V-FB: track 27.2 -> 4.45 mm
- net N$1: track 22.4 -> 2.98 mm
- net N$7: track 13.6 -> 0.00 mm
- net N$10: track 26.0 -> 16.4 mm
- net N$6: track 9.24 -> 0.00 mm
- net +V-FB: track 7.68 -> 0.00 mm
- net C-IN+: track 6.68 -> 0.00 mm
- net C-IN-: track 6.67 -> 0.00 mm
- net N$8: track 5.29 -> 0.00 mm
- net N$3: track 5.21 -> 0.00 mm
- net V-IN+: track 4.43 -> 0.00 mm
- net +I-FB: track 3.27 -> 0.00 mm
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Other:
- board size 27.3 x 38.1 mm -> 38.1 x 27.3 mm

Commit message: ((
Parts:
- removed C1: 10u, rcl:C1210
- removed IC2: LD117ASTR, v-reg:SOT223
- removed R12: 200R, rcl:R0805
- removed R13: 510R, rcl:R0805
- removed R14: 5R, rcl:R0805
- added IC3: LD2985BM50R, v-reg:SOT25
Connections:
- removed net N$5: R13.1, R14.2
- removed net N$6: IC2.1, R12.1, R13.2
- removed net N$9: C1.1, IC2.4, R12.2
- new net +5V: IC3.5
- net +12V: now also IC3.1, IC3.3; no longer IC2.3
- net GND: now also IC3.2; no longer C1.2, R14.1
Changed lines of the file:
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@@
 <?xml version="1.0" encoding="utf-8"?>
 <!DOCTYPE eagle SYSTEM "eagle.dtd">
-<eagle version="7.6.0">
+<eagle version="7.7.0">
 <drawing>
 <settings>
@@
 <attribute name="OC_FARNELL" value="4375737" x="9.525" y="-16.51" size="1.778" layer="28" rot="MR90" display="off"/>
 </element>
-<element name="IC2" library="v-reg" package="SOT223" value="LD117ASTR" x="19.05" y="-24.13" rot="MR180"/>
-<element name="R12" library="rcl" package="R0805" value="200R" x="14.605" y="-26.67" rot="MR270"/>
-<element name="R13" library="rcl" package="R0805" value="510R" x="16.51" y="-17.145" rot="MR0"/>
-<element name="R14" library="rcl" package="R0805" value="5R" x="19.685" y="-15.875" rot="MR270"/>
 <element name="R15" library="rcl" package="R0805" value="33K" x="6.35" y="-17.78" rot="MR270"/>
-<element name="C1" library="rcl" package="C1210" value="10u" x="13.97" y="-22.225" rot="MR90"/>
 <element name="U1" library="ST Microelctronics_By_element14_Batch_1" package="SOT95P280X145-5N" value="TSV621ILT" x="9.525" y="-21.59" rot="MR270">
 <attribute name="OC_NEWARK" value="26R7211" x="9.525" y="-21.59" size="1.778" layer="28" rot="MR270" display="off"/>
@@
 <element name="R17" library="rcl" package="R0805" value="0" x="-6.985" y="-20.955" rot="MR180"/>
 <element name="JP2" library="pinhead" package="1X02/90" value="" x="4.7625" y="-31.75" rot="R180"/>
+<element name="IC3" library="v-reg" package="SOT25" value="LD2985BM50R" x="-28.575" y="-65.405"/>
 </elements>
 <signals>
@@
 <contactref element="R4" pad="2"/>
 <contactref element="R8" pad="2"/>
-<contactref element="IC2" pad="3"/>
 <wire x1="-10.89" y1="-11.43" x2="-8.985" y2="-11.43" width="0.6096" layer="16"/>
 <wire x1="-8.985" y1="-11.43" x2="-8.89" y2="-11.525" width="0.6096" layer="16"/>
+<contactref element="IC3" pad="1"/>
+<contactref element="IC3" pad="3"/>
+<wire x1="-27.625" y1="-66.705" x2="-29.525" y2="-66.705" width="0" layer="19" extent="1-1"/>
+<wire x1="-10.89" y1="-11.43" x2="-27.625" y2="-66.705" width="0" layer="19" extent="1-16"/>
 <wire x1="10.795" y1="-8.89" x2="-8.89" y2="-11.525" width="0" layer="19" extent="16-16"/>
-<wire x1="21.35" y1="-20.98" x2="10.795" y2="-8.89" width="0" layer="19" extent="16-16"/>
 </signal>
 <signal name="GND">
@@
 <contactref element="IC1" pad="2"/>
 <contactref element="R15" pad="1"/>
-<contactref element="C1" pad="2"/>
 <contactref element="U1" pad="2"/>
 <contactref element="JP1" pad="2"/>
 <contactref element="R17" pad="2"/>
 <contactref element="JP2" pad="2"/>
-<contactref element="R14" pad="1"/>
-<wire x1="3.4925" y1="-27.94" x2="-5.81" y2="-20.955" width="0" layer="19" extent="16-16"/>
+<contactref element="IC3" pad="2"/>
+<wire x1="3.4925" y1="-27.94" x2="-28.575" y2="-66.705" width="0" layer="19" extent="1-1"/>
 <wire x1="9.525" y1="-27.94" x2="3.4925" y2="-27.94" width="0" layer="19" extent="1-1"/>
 <wire x1="9.525" y1="-20.32" x2="9.525" y2="-27.94" width="0" layer="19" extent="16-16"/>
 <wire x1="8.219" y1="-16.51" x2="9.525" y2="-20.32" width="0" layer="19" extent="16-16"/>
 <wire x1="6.35" y1="-16.605" x2="8.219" y2="-16.51" width="0" layer="19" extent="16-16"/>
-<wire x1="13.97" y1="-20.825" x2="9.525" y2="-20.32" width="0" layer="19" extent="16-16"/>
 <wire x1="8.255" y1="-8.89" x2="8.219" y2="-16.51" width="0" layer="19" extent="16-16"/>
-<wire x1="19.685" y1="-14.7" x2="13.97" y2="-20.825" width="0" layer="19" extent="16-16"/>
+<wire x1="-5.81" y1="-20.955" x2="3.4925" y2="-27.94" width="0" layer="19" extent="16-16"/>
 </signal>
 <signal name="V-IN+">
@@
 <wire x1="11.97" y1="-13.97" x2="13.335" y2="-13.875" width="0" layer="19" extent="16-16"/>
 </signal>
-<signal name="N$5">
-<contactref element="R13" pad="1"/>
-<contactref element="R14" pad="2"/>
-<wire x1="17.685" y1="-17.145" x2="19.685" y2="-17.05" width="0" layer="19" extent="16-16"/>
-</signal>
-<signal name="N$6">
-<contactref element="R13" pad="2"/>
-<contactref element="IC2" pad="1"/>
-<contactref element="R12" pad="1"/>
-<wire x1="16.75" y1="-20.98" x2="14.605" y2="-25.495" width="0" layer="19" extent="16-16"/>
-<wire x1="15.335" y1="-17.145" x2="16.75" y2="-20.98" width="0" layer="19" extent="16-16"/>
-</signal>
 <signal name="N$8">
 <contactref element="IC1" pad="1"/>
@@
 <wire x1="8.219" y1="-17.46" x2="6.35" y2="-18.955" width="0" layer="19" extent="16-16"/>
 <wire x1="8.5852" y1="-20.32" x2="6.35" y2="-18.955" width="0" layer="19" extent="16-16"/>
-</signal>
-<signal name="N$9">
-<contactref element="R12" pad="2"/>
-<contactref element="IC2" pad="4"/>
-<contactref element="C1" pad="1"/>
-<wire x1="13.97" y1="-23.625" x2="14.605" y2="-27.845" width="0" layer="19" extent="16-16"/>
-<wire x1="19.05" y1="-27.28" x2="14.605" y2="-27.845" width="0" layer="19" extent="16-16"/>
 </signal>
 <signal name="N$7">
@@
 <wire x1="10.831" y1="-17.46" x2="8.5852" y2="-22.86" width="0" layer="19" extent="16-16"/>
 </signal>
+<signal name="+5V">
+<contactref element="IC3" pad="5"/>
+</signal>
 </signals>
