File: LED/CCR2.sch (EAGLE design)
At the start: 12 parts, among them Q1 STD6NF10, Q4 BC817-40SMD, X2 MKDSN1,5/2-5,08, X3 MKDSN1,5/2-5,08

Commit message: CCR
Parts:
- removed F1: FUSESH22,5, fuse:FUSESH22,5
- removed Q1: STD6NF10, Namenlos:STD6NF10
- removed Q4: BC817-40SMD, transistor-npn:BC817-40SMD
- removed R1, R4: 13R, rcl:R-EU_0411/12
- removed R2: 300k, rcl:R-EU_0411/12
Connections:
- removed net N$3: Q1.S, Q4.B, R1.2, R4.2
- removed net N$4: Q1.D, X2-2.KL
- removed net N$6: B1.AC2, F1.1
- removed net N$8: Q1.G, Q4.C, R2.1
- net GND: no longer Q4.E, R1.1, R4.1
- net N$1: no longer R2.2, X2-1.KL
- net N$5: now also B1.AC2; no longer F1.2
Changed lines of the file:
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@@
 <?xml version="1.0" encoding="utf-8"?>
 <!DOCTYPE eagle SYSTEM "eagle.dtd">
-<eagle version="7.1.0">
+<eagle version="7.6.0">
 <drawing>
 <settings>
@@
 </classes>
 <parts>
-<part name="R2" library="rcl" deviceset="R-EU_" device="0411/12" value="300k"/>
-<part name="R4" library="rcl" deviceset="R-EU_" device="0411/12" value="13R"/>
 <part name="X2" library="con-phoenix-508" deviceset="MKDSN1,5/2-5,08" device=""/>
-<part name="Q1" library="Namenlos" deviceset="STD6NF10" device=""/>
-<part name="Q4" library="transistor-npn" deviceset="BC817*" device="SMD" technology="-40"/>
 <part name="B1" library="rectifier" deviceset="RB1A" device=""/>
 <part name="C1" library="Namenlos" deviceset="CPOL-400V-100UF" device=""/>
 <part name="R6" library="rcl" deviceset="R-EU_" device="0204/7" value="160k"/>
 <part name="X3" library="con-phoenix-508" deviceset="MKDSN1,5/2-5,08" device=""/>
-<part name="R1" library="rcl" deviceset="R-EU_" device="0411/12" value="13R"/>
-<part name="F1" library="fuse" deviceset="FUSE" device="SH22,5"/>
 <part name="R3" library="rcl" deviceset="R-EU_" device="0309/10" value="NTC"/>
 </parts>
@@
 </plain>
 <instances>
-<instance part="R2" gate="G$1" x="53.34" y="68.58" rot="R90"/>
-<instance part="R4" gate="G$1" x="63.5" y="35.56" rot="R90"/>
 <instance part="X2" gate="-1" x="66.04" y="71.12"/>
 <instance part="X2" gate="-2" x="66.04" y="66.04"/>
-<instance part="Q1" gate="G$1" x="63.5" y="50.8"/>
-<instance part="Q4" gate="G$1" x="55.88" y="40.64" rot="MR0"/>
 <instance part="B1" gate="1" x="68.58" y="121.92" rot="R180"/>
 <instance part="C1" gate="G$1" x="68.58" y="101.6" rot="R90"/>
@@
 <instance part="X3" gate="-1" x="68.58" y="165.1" rot="R90"/>
 <instance part="X3" gate="-2" x="76.2" y="165.1" rot="R90"/>
-<instance part="R1" gate="G$1" x="71.12" y="35.56" rot="R90"/>
-<instance part="F1" gate="G$1" x="68.58" y="142.24" rot="R90"/>
 <instance part="R3" gate="G$1" x="76.2" y="142.24" rot="R90"/>
 </instances>
@@
 <net name="N$1" class="0">
 <segment>
-<pinref part="R2" gate="G$1" pin="2"/>
-<wire x1="53.34" y1="73.66" x2="53.34" y2="78.74" width="0.1524" layer="91"/>
-<wire x1="53.34" y1="78.74" x2="45.72" y2="78.74" width="0.1524" layer="91"/>
-<pinref part="X2" gate="-1" pin="KL"/>
-<wire x1="63.5" y1="71.12" x2="60.96" y2="71.12" width="0.1524" layer="91"/>
-<wire x1="60.96" y1="71.12" x2="60.96" y2="78.74" width="0.1524" layer="91"/>
-<wire x1="60.96" y1="78.74" x2="53.34" y2="78.74" width="0.1524" layer="91"/>
-<junction x="53.34" y="78.74"/>
-<wire x1="45.72" y1="78.74" x2="45.72" y2="101.6" width="0.1524" layer="91"/>
 <pinref part="C1" gate="G$1" pin="+"/>
-<wire x1="45.72" y1="101.6" x2="58.42" y2="101.6" width="0.1524" layer="91"/>
 <pinref part="B1" gate="1" pin="+"/>
 <wire x1="58.42" y1="101.6" x2="64.77" y2="101.6" width="0.1524" layer="91"/>
@@
 </segment>
 </net>
-<net name="N$4" class="0">
-<segment>
-<pinref part="X2" gate="-2" pin="KL"/>
-<wire x1="63.5" y1="66.04" x2="63.5" y2="55.88" width="0.1524" layer="91"/>
-<pinref part="Q1" gate="G$1" pin="D"/>
-</segment>
-</net>
-<net name="N$8" class="0">
-<segment>
-<wire x1="53.34" y1="48.26" x2="58.42" y2="48.26" width="0.1524" layer="91"/>
-<wire x1="53.34" y1="48.26" x2="53.34" y2="63.5" width="0.1524" layer="91"/>
-<pinref part="Q1" gate="G$1" pin="G"/>
-<pinref part="Q4" gate="G$1" pin="C"/>
-<wire x1="53.34" y1="45.72" x2="53.34" y2="48.26" width="0.1524" layer="91"/>
-<junction x="53.34" y="48.26"/>
-<pinref part="R2" gate="G$1" pin="1"/>
-</segment>
-</net>
-<net name="N$3" class="0">
-<segment>
-<pinref part="R4" gate="G$1" pin="2"/>
-<wire x1="63.5" y1="40.64" x2="63.5" y2="45.72" width="0.1524" layer="91"/>
-<pinref part="Q1" gate="G$1" pin="S"/>
-<pinref part="Q4" gate="G$1" pin="B"/>
-<wire x1="58.42" y1="40.64" x2="63.5" y2="40.64" width="0.1524" layer="91"/>
-<junction x="63.5" y="40.64"/>
-<pinref part="R1" gate="G$1" pin="2"/>
-<wire x1="71.12" y1="40.64" x2="63.5" y2="40.64" width="0.1524" layer="91"/>
-</segment>
-</net>
 <net name="GND" class="0">
 <segment>
-<wire x1="53.34" y1="22.86" x2="53.34" y2="35.56" width="0.1524" layer="91"/>
-<pinref part="Q4" gate="G$1" pin="E"/>
-<wire x1="53.34" y1="22.86" x2="53.34" y2="17.78" width="0.1524" layer="91"/>
-<wire x1="53.34" y1="17.78" x2="63.5" y2="17.78" width="0.1524" layer="91"/>
-<wire x1="63.5" y1="17.78" x2="71.12" y2="17.78" width="0.1524" layer="91"/>
-<wire x1="71.12" y1="17.78" x2="88.9" y2="17.78" width="0.1524" layer="91"/>
-<wire x1="88.9" y1="17.78" x2="88.9" y2="93.98" width="0.1524" layer="91"/>
+<wire x1="88.9" y1="17.78" x2="88.9" y2="101.6" width="0.1524" layer="91"/>
 <pinref part="C1" gate="G$1" pin="-"/>
 <wire x1="72.39" y1="101.6" x2="81.28" y2="101.6" width="0.1524" layer="91"/>
 <wire x1="81.28" y1="101.6" x2="88.9" y2="101.6" width="0.1524" layer="91"/>
-<wire x1="88.9" y1="101.6" x2="88.9" y2="93.98" width="0.1524" layer="91"/>
 <pinref part="B1" gate="1" pin="-"/>
 <wire x1="73.66" y1="121.92" x2="81.28" y2="121.92" width="0.1524" layer="91"/>
@@
 <wire x1="76.2" y1="96.52" x2="81.28" y2="96.52" width="0.1524" layer="91"/>
 <wire x1="81.28" y1="96.52" x2="81.28" y2="101.6" width="0.1524" layer="91"/>
-<pinref part="R4" gate="G$1" pin="1"/>
-<wire x1="63.5" y1="30.48" x2="63.5" y2="17.78" width="0.1524" layer="91"/>
-<junction x="63.5" y="17.78"/>
-<pinref part="R1" gate="G$1" pin="1"/>
-<wire x1="71.12" y1="30.48" x2="71.12" y2="17.78" width="0.1524" layer="91"/>
-<junction x="71.12" y="17.78"/>
 </segment>
 </net>
@@
 <segment>
 <pinref part="X3" gate="-1" pin="KL"/>
-<pinref part="F1" gate="G$1" pin="2"/>
-<wire x1="68.58" y1="147.32" x2="68.58" y2="162.56" width="0.1524" layer="91"/>
-</segment>
-</net>
-<net name="N$6" class="0">
-<segment>
-<pinref part="F1" gate="G$1" pin="1"/>
 <pinref part="B1" gate="1" pin="AC2"/>
-<wire x1="68.58" y1="137.16" x2="68.58" y2="127" width="0.1524" layer="91"/>
-</segment>
-</net>
+<wire x1="68.58" y1="162.56" x2="68.58" y2="127" width="0.1524" layer="91"/>
+</segment>
+</net>
