File: Power/PrinterPower/Printer Power.brd (EAGLE design)
At the start: 172.7 x 86 mm, 90 parts, among them IC1 TNY264PN, Q3 IRF740, Q4 IRF740, Q5 STD6NF10, U1 SG3525AN, X1 MKDSN1,5/2-5,08, X2 1751248, X3 1751248

Commit message: Printer Power
Parts:
- removed D13: (no value), diode:DO220S
- removed Q5: STD6NF10, Namenlos:DPAK
- removed R10: 100R, Namenlos:SQP-5
- removed R25: 5K1, rcl:R0805
- removed X2, X3: 1751248, con-phoenix-350:1751248
- added C21: 100n, rcl:C0805
- added IC2: 78L05SMD, linear:SO08
- added JP3: (no value), pinhead:1X02
- C13: value 1500u 63V -> 2200u 35V
- C15: value 1500u 63V -> 6v3 330u; device rcl:E7,5-18 -> rcl:E2,5-7
- JP1: value (none) -> MKDSN1,5/2-5,08; device pinhead:1X02 -> con-phoenix-508:MKDSN1,5/2-5,08
- L1: value 82721K -> EE20-DROSSEL; device _Transformers:82721K -> _Transformers:EE20_DROSSEL
- TR1: value ETD_CNC -> ETD39_PRINTER
- moved D7 41.6 mm to (165.1, 19.1), turned to 270 degrees
- moved U$7 41.6 mm to (165.1, 19.1), turned to 270 degrees
- moved D10 41.5 mm to (127.0, 54.6), turned to 0 degrees
- moved U$6 41.5 mm to (127.0, 54.6), turned to 0 degrees
- moved U$5 41.5 mm to (146.1, 54.6), turned to 0 degrees
- moved C13 38.3 mm to (128.3, 73.7)
- moved JP1 29.9 mm to (108.0, 80.0), turned to 90 degrees
- moved C14 20.7 mm to (147.3, 73.7), turned to 270 degrees
- moved D9 20.3 mm to (165.1, 38.1)
- moved C15 17.8 mm to (91.4, 77.5), flipped to the bottom
- moved U$8 16.7 mm to (165.1, 38.1), turned to 270 degrees
- moved D8 16.5 mm to (146.1, 54.6)
- moved L1 16.3 mm to (163.8, 59.7), turned to 90 degrees
- moved R22 10.2 mm to (72.4, 72.4), turned to 270 degrees
- moved TR1 1.27 mm to (133.3, 24.1), flipped to the bottom, turned to 0 degrees
Connections:
- removed net N$33: D10.C, D9.C, L1.2
- removed net N$34: C13.-, C14.-, C15.-, C16.2, CY1.2, JP1.2, Q5.S, R10.2, R24.2, R25.2, TR1.12, TR1.13, U$9.2, U$9.3, U$9.6, U$9.7, X2.2
- removed net N$35: C14.+, L1.4, R10.1, X2.1
- removed net N$43: JP1.1, Q5.G, R25.1
- removed net N$45: D13.A, Q5.D, X3.2
- net N$26: now also C13.-, C14.-, C15.-, C16.2, C21.2, CY1.2, D8.A, IC2.2, IC2.3, IC2.6, IC2.7, JP1.1, JP3.2, R24.2, U$9.2, U$9.3, U$9.6, U$9.7; no longer TR1.16
- net N$27: now also D10.C, D8.C, TR1.4, TR1.5, TR1.6, TR1.7, TR1.8; no longer D8.A, TR1.11
- net N$31: now also D7.A, TR1.10, TR1.11, TR1.12, TR1.13
- net N$32: now also C15.+, IC2.1, JP3.1; no longer D7.C, D8.C, L1.1
- net N$36: now also C14.+, C21.1, IC2.8, JP1.2, L1.5; no longer C15.+, D13.C, L1.3, X3.1
- net N$4: now also D7.C, D9.C, L1.10; no longer D7.A, TR1.14
- net N$9: now also TR1.15, TR1.16; no longer TR1.8
- net VS: now also TR1.1, TR1.2; no longer TR1.6
Routing:
- net N$26: track 16.1 -> 242.9 mm
- net N$34: track 226.6 -> 0.00 mm
- net N$33: track 67.2 -> 0.00 mm
- net N$35: track 54.3 -> 0.00 mm
- net N$31: track 18.2 -> 60.1 mm
- net N$32: track 39.9 -> 13.4 mm
- net N$4: track 29.8 -> 48.1 mm
- net N$45: track 14.7 -> 0.00 mm
- net N$27: track 61.6 -> 48.4 mm
- net N$9: track 27.8 -> 38.5 mm
- net VS: track 107.6 -> 114.4 mm
- net N$36: track 120.1 -> 126.9 mm
- net N$43: track 5.18 -> 0.00 mm
- net N$42: track 7.01 -> 11.8 mm
- net N$15: track 4.69 -> 7.33 mm
