File: LED/DeskLamp/LAm-v2.brd (EAGLE design)
At the start: 200.6 x 44.1 mm, 30 parts, among them IC1 HV9910BLG

Commit message: Some lamps
Parts:
- R3: value 68K -> 91K
- R7: value 300K -> 1M3
Changed lines of the file:
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@@
 <?xml version="1.0" encoding="utf-8"?>
 <!DOCTYPE eagle SYSTEM "eagle.dtd">
-<eagle version="8.1.0">
+<eagle version="8.1.1">
 <drawing>
 <settings>
@@
 </element>
 <element name="R2" library="Namenlos" package="MF-2" value="27K" x="13.97" y="21.59" rot="MR270"/>
-<element name="R3" library="Namenlos" package="R0805" value="68K" x="19.05" y="24.13" rot="R90"/>
+<element name="R3" library="Namenlos" package="R0805" value="91K" x="19.05" y="24.13" rot="R90"/>
 <element name="VT1" library="Namenlos" package="DPAK" value="STD2HNK60Z" x="22.86" y="34.29"/>
 <element name="L1" library="Namenlos" package="SL1016" value="4m7" x="7.62" y="36.83" rot="MR270"/>
@@
 <element name="R4" library="Namenlos" package="R0805" value="15K" x="20.32" y="13.335"/>
 <element name="R5" library="Namenlos" package="KNP-100B" value="1R3" x="29.21" y="20.32" rot="MR90"/>
-<element name="R7" library="Namenlos" package="R0805" value="300K" x="21.59" y="10.795"/>
+<element name="R7" library="Namenlos" package="R0805" value="1M3" x="21.59" y="10.795"/>
 <element name="R6" library="Namenlos" package="R0805" value="3R3" x="29.21" y="24.13" rot="R90"/>
 <element name="R8" library="Namenlos" package="R0805" value="3R3" x="29.21" y="19.05" rot="R90"/>
