File: LED/lustre/Lamp.brd (EAGLE design)
At the start: 95.5 x 72.6 mm, 12 parts

Commit message: Люстра-Ламп
Parts:
- added D11, D12, D13, D14, D15: LED1W, Namenlos:LED-1W
Connections:
- new net N$13: D11.K, D12.A
- new net N$14: D12.K, D13.A
- new net N$15: D13.K, D14.A
- new net N$16: D14.K, D15.A
- new net N$17: D15.K, PAD2.1
- net N$11: now also D11.A; no longer PAD2.1
Routing:
- net N$11: track 3.74 -> 0.00 mm
- removed copper zone on layer 1, net N$12
Other:
- board size 95.5 x 72.6 mm -> 4.8 x 30.1 mm
