File: LED/lustre/Lamp.sch (EAGLE design)
At the start: 12 parts

Commit message: Люстра-Ламп
Parts:
- added D11, D12, D13, D14, D15: LED1W, Namenlos:LED1W
Connections:
- new net N$13: D11.C, D12.A
- new net N$14: D12.C, D13.A
- new net N$15: D13.C, D14.A
- new net N$16: D14.C, D15.A
- new net N$17: D15.C, PAD2.P
- net N$11: now also D11.A; no longer PAD2.P
Other:
- moved on the sheet: PAD2
Changed lines of the file:
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@@
 <part name="PAD1" library="wirepad" deviceset="3,81/1,4" device=""/>
 <part name="PAD2" library="wirepad" deviceset="3,81/1,4" device=""/>
+<part name="D11" library="Namenlos" deviceset="LED" device="1W"/>
+<part name="D12" library="Namenlos" deviceset="LED" device="1W"/>
+<part name="D13" library="Namenlos" deviceset="LED" device="1W"/>
+<part name="D14" library="Namenlos" deviceset="LED" device="1W"/>
+<part name="D15" library="Namenlos" deviceset="LED" device="1W"/>
 </parts>
 <sheets>
@@
 <instance part="D10" gate="G$1" x="88.9" y="40.64" rot="R90"/>
 <instance part="PAD1" gate="1" x="12.7" y="40.64"/>
-<instance part="PAD2" gate="1" x="93.98" y="40.64" rot="R180"/>
+<instance part="PAD2" gate="1" x="132.08" y="40.64" rot="R180"/>
+<instance part="D11" gate="G$1" x="96.52" y="40.64" rot="R90"/>
+<instance part="D12" gate="G$1" x="104.14" y="40.64" rot="R90"/>
+<instance part="D13" gate="G$1" x="111.76" y="40.64" rot="R90"/>
+<instance part="D14" gate="G$1" x="119.38" y="40.64" rot="R90"/>
+<instance part="D15" gate="G$1" x="127" y="40.64" rot="R90"/>
 </instances>
 <busses>
@@
 <segment>
 <pinref part="D10" gate="G$1" pin="C"/>
+<pinref part="D11" gate="G$1" pin="A"/>
+</segment>
+</net>
+<net name="N$13" class="0">
+<segment>
+<pinref part="D11" gate="G$1" pin="C"/>
+<pinref part="D12" gate="G$1" pin="A"/>
+</segment>
+</net>
+<net name="N$14" class="0">
+<segment>
+<pinref part="D12" gate="G$1" pin="C"/>
+<pinref part="D13" gate="G$1" pin="A"/>
+</segment>
+</net>
+<net name="N$15" class="0">
+<segment>
+<pinref part="D13" gate="G$1" pin="C"/>
+<pinref part="D14" gate="G$1" pin="A"/>
+</segment>
+</net>
+<net name="N$16" class="0">
+<segment>
+<pinref part="D14" gate="G$1" pin="C"/>
+<pinref part="D15" gate="G$1" pin="A"/>
+</segment>
+</net>
+<net name="N$17" class="0">
+<segment>
+<pinref part="D15" gate="G$1" pin="C"/>
 <pinref part="PAD2" gate="1" pin="P"/>
 </segment>

Commit message: Не уверен
Parts:
- removed D13, D14, D15: LED1W, Namenlos:LED1W
Connections:
- removed net N$14: D12.C, D13.A
- removed net N$15: D13.C, D14.A
- removed net N$16: D14.C, D15.A
- removed net N$17: D15.C, PAD2.P
- new net N$13: D12.C, D5.A
- net N$11: now also PAD2.P; no longer D11.A
- net N$4: now also D11.A; no longer D5.A
Other:
- moved on the sheet: D10, D11, D12, D5, D6, D7, D8, D9, PAD2
Changed lines of the file:
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@@
 <part name="D11" library="Namenlos" deviceset="LED" device="1W"/>
 <part name="D12" library="Namenlos" deviceset="LED" device="1W"/>
-<part name="D13" library="Namenlos" deviceset="LED" device="1W"/>
-<part name="D14" library="Namenlos" deviceset="LED" device="1W"/>
-<part name="D15" library="Namenlos" deviceset="LED" device="1W"/>
 </parts>
 <sheets>
@@
 <instance part="D3" gate="G$1" x="35.56" y="40.64" rot="R90"/>
 <instance part="D4" gate="G$1" x="43.18" y="40.64" rot="R90"/>
-<instance part="D5" gate="G$1" x="50.8" y="40.64" rot="R90"/>
-<instance part="D6" gate="G$1" x="58.42" y="40.64" rot="R90"/>
-<instance part="D7" gate="G$1" x="66.04" y="40.64" rot="R90"/>
-<instance part="D8" gate="G$1" x="73.66" y="40.64" rot="R90"/>
-<instance part="D9" gate="G$1" x="81.28" y="40.64" rot="R90"/>
-<instance part="D10" gate="G$1" x="88.9" y="40.64" rot="R90"/>
+<instance part="D5" gate="G$1" x="66.04" y="40.64" rot="R90"/>
+<instance part="D6" gate="G$1" x="73.66" y="40.64" rot="R90"/>
+<instance part="D7" gate="G$1" x="81.28" y="40.64" rot="R90"/>
+<instance part="D8" gate="G$1" x="88.9" y="40.64" rot="R90"/>
+<instance part="D9" gate="G$1" x="96.52" y="40.64" rot="R90"/>
+<instance part="D10" gate="G$1" x="104.14" y="40.64" rot="R90"/>
 <instance part="PAD1" gate="1" x="12.7" y="40.64"/>
-<instance part="PAD2" gate="1" x="132.08" y="40.64" rot="R180"/>
-<instance part="D11" gate="G$1" x="96.52" y="40.64" rot="R90"/>
-<instance part="D12" gate="G$1" x="104.14" y="40.64" rot="R90"/>
-<instance part="D13" gate="G$1" x="111.76" y="40.64" rot="R90"/>
-<instance part="D14" gate="G$1" x="119.38" y="40.64" rot="R90"/>
-<instance part="D15" gate="G$1" x="127" y="40.64" rot="R90"/>
+<instance part="PAD2" gate="1" x="114.3" y="40.64" rot="R180"/>
+<instance part="D11" gate="G$1" x="50.8" y="40.64" rot="R90"/>
+<instance part="D12" gate="G$1" x="58.42" y="40.64" rot="R90"/>
 </instances>
 <busses>
@@
 <pinref part="D3" gate="G$1" pin="C"/>
 <pinref part="D4" gate="G$1" pin="A"/>
-</segment>
-</net>
-<net name="N$4" class="0">
-<segment>
-<pinref part="D4" gate="G$1" pin="C"/>
-<pinref part="D5" gate="G$1" pin="A"/>
 </segment>
 </net>
@@
 <segment>
 <pinref part="D10" gate="G$1" pin="C"/>
+<pinref part="PAD2" gate="1" pin="P"/>
+<wire x1="111.76" y1="40.64" x2="106.68" y2="40.64" width="0.1524" layer="91"/>
+</segment>
+</net>
+<net name="N$4" class="0">
+<segment>
+<pinref part="D4" gate="G$1" pin="C"/>
 <pinref part="D11" gate="G$1" pin="A"/>
 </segment>
 </net>
-<net name="N$13" class="0">
+<net name="N$12" class="0">
 <segment>
 <pinref part="D11" gate="G$1" pin="C"/>
@@
 </segment>
 </net>
-<net name="N$14" class="0">
+<net name="N$13" class="0">
 <segment>
 <pinref part="D12" gate="G$1" pin="C"/>
-<pinref part="D13" gate="G$1" pin="A"/>
+<pinref part="D5" gate="G$1" pin="A"/>
 </segment>
 </net>
-<net name="N$15" class="0">
-<segment>
-<pinref part="D13" gate="G$1" pin="C"/>
-<pinref part="D14" gate="G$1" pin="A"/>
-</segment>
-</net>
-<net name="N$16" class="0">
-<segment>
-<pinref part="D14" gate="G$1" pin="C"/>
-<pinref part="D15" gate="G$1" pin="A"/>
-</segment>
-</net>
-<net name="N$17" class="0">
-<segment>
-<pinref part="D15" gate="G$1" pin="C"/>
-<pinref part="PAD2" gate="1" pin="P"/>
-</segment>
-</net>
