File: LED/Flash/Flash.sch (EAGLE design)
At the start: 14 parts

Commit message: More Flash
Parts:
- added C1: 0u1, rcl:C-EUC0805
- added C10: 10u, rcl:C-EUC1206
- added C2: 1n5, rcl:C-EUC0805
- added C3, C4, C5, C6, C7, C8: 47u16v, rcl:CPOL-EU153CLV-0605
- added C9: 10u, rcl:C-EUC0805
- added D1, D2, D3: RB520S30T1G, diode:DIODE-SOD523
- added IC1: 4098D, 40xx:4098D
- added PAD1, PAD10, PAD11, PAD12, PAD2, PAD3, PAD4, PAD5, PAD6, PAD7, PAD8, PAD9: (no value), wirepad:SMD2
- added R1, R2, R3, R4: 1R, rcl:R-EU_R0805
- added R10: 1K, rcl:R-EU_R0805
- added R11: 43K, rcl:R-EU_R0805
- added R12: 11K, rcl:R-EU_R0805
- added R5: 180R, rcl:R-EU_R0805
- added R6: 12K, rcl:R-EU_R0805
- added R7: 1K3, rcl:R-EU_R0805
- added R8: 1M, rcl:R-EU_R0805
- added R9: 0R, rcl:R-EU_R0805
- added TL1: TL431CDBZR, Namenlos:TL431CDBZR
- added U$15: MC33063/MC34063D, Namenlos at:MC33063/MC34063D
- added U$16: 150uH, Namenlos:INDUCTOR6045
- added U$17: STL6N3LLH6, Namenlos:STL6N3LLH6
- added U1: TSV621ILT, ST Microelctronics_By_element14_Batch_1:TSV621ILT
Connections:
- new net +12V: C1.1, C3.+, C4.+, C5.+, C6.+, C7.+, C8.+, D1.C, D2.C, D3.C, PAD6.P, PAD9.P, R11.1, R6.1, U$1.A, U$11.A, U$13.A, U$3.A, U$5.A, U$7.A, U$9.A
- new net B+: C10.1, IC1A.RES, IC1P.VDD, PAD1.P, PAD11.P, PAD8.P, R1.1, R10.1, R2.1, R3.1, R4.1, R8.2, U$15.VCC, U1.VCC
- new net GND: C1.2, C10.2, C2.2, C3.-, C4.-, C5.-, C6.-, C7.-, C8.-, IC1P.VSS, PAD12.P, PAD2.P, PAD7.P, R12.2, R7.2, TL1.A, U$15.GND, U$15.SWE, U$17.S, U1.VDD
- new net N$11: R6.2, R7.1, U$15.COMP
- new net N$12: D1.A, D2.A, D3.A, U$15.SWC, U$16.2
- new net N$14: C2.1, U$15.TC
- new net N$17: C9.2, IC1A.C
- new net N$18: C9.1, IC1A.R/C, R8.1
- new net N$20: IC1A.Q, R9.2
- new net N$21: R9.1, U$17.G
- new net N$5: R11.2, R12.1, U1.IN+
- new net N$6: IC1A.+TR, PAD3.P
- new net N$8: R1.2, R2.2, R3.2, R4.2, R5.2, U$15.IPK, U$16.1
- new net N$9: R5.1, U$15.DC
- new net TR-: IC1A.!Q, IC1A.-TR, PAD10.P, PAD4.P, U1.OUT
- net N$2: now also R10.2, TL1.C, TL1.R, U1.IN-; no longer U$1.A, U$11.A, U$13.A, U$3.A, U$5.A, U$7.A, U$9.A
- net N$3: now also PAD5.P, U$17.D
Other:
- moved on the sheet: U$1, U$10, U$11, U$12, U$13, U$14, U$2, U$3, U$4, U$5, U$6, U$7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
