File: Power/Step-Down Tests/NCP1200.brd (EAGLE design)
At the start: 115.5 x 28.9 mm, 20 parts, among them Q1 NTD20P06LT4G, Q2 NTD20P06LT4G, Q3 BSS84, Q4 BSS123, X1 MKDSN1,5/3-5,08, X2 MKDSN1,5/3-5,08

Commit message: Some minor changes
Parts:
- added C3: 10u, rcl:C1210
- moved Q3 2.54 mm to (31.8, 16.5)
- moved Q4 2.54 mm to (31.8, 12.7)
- moved R1 1.90 mm to (34.9, 20.3)
Connections:
- new net N$10: C3.2, Q3.3, Q4.3
- net N$4: now also C3.1; no longer Q3.3, Q4.3
Routing:
- net N$4: track 22.9 -> 14.1 mm
- net N$10: track 0.00 -> 6.92 mm
- net GND: track 210.5 -> 207.9 mm
- net N$6: track 11.9 -> 9.36 mm
- net N$2: track 16.3 -> 13.8 mm
- net N$1: track 78.0 -> 79.9 mm
Changed lines of the file:
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@@
 <element name="Q1" library="transistor-fet" package="TO252" value="NTD20P06LT4G" x="45.72" y="24.13" rot="MR90"/>
 <element name="Q2" library="transistor-fet" package="TO252" value="NTD20P06LT4G" x="45.72" y="15.24" rot="MR90"/>
-<element name="Q3" library="transistor-small-signal" package="SOT23" value="BSS84" x="34.29" y="16.51" rot="MR90"/>
-<element name="Q4" library="transistor-small-signal" package="SOT23" value="BSS123" x="34.29" y="12.7" rot="MR90"/>
-<element name="R1" library="rcl" package="R0805" value="4k7" x="33.02" y="20.32" rot="MR180"/>
+<element name="Q3" library="transistor-small-signal" package="SOT23" value="BSS84" x="31.75" y="16.51" rot="MR90"/>
+<element name="Q4" library="transistor-small-signal" package="SOT23" value="BSS123" x="31.75" y="12.7" rot="MR90"/>
+<element name="R1" library="rcl" package="R0805" value="4k7" x="34.925" y="20.32" rot="MR180"/>
 <element name="R2" library="rcl" package="R0805" value="4k7" x="26.67" y="3.81" rot="MR180"/>
 <element name="R3" library="Namenlos" package="SQP-10" value="0R1" x="39.37" y="19.05"/>
@@
 <element name="X2" library="Namenlos" package="MKDSN1,5/3-5,08" value="MKDSN1,5/3-5,08" x="109.22" y="10.16" rot="R90"/>
 <element name="C2" library="rcl" package="E3,5-8" value="1000u 16V" x="99.06" y="7.62" rot="R90"/>
+<element name="C3" library="rcl" package="C1210" value="10u" x="36.83" y="16.51" rot="MR0"/>
 </elements>
 <signals>
@@
 <wire x1="17.65" y1="17.78" x2="16.38" y2="19.05" width="0.4064" layer="16"/>
 <wire x1="16.38" y1="19.05" x2="12.7" y2="19.05" width="0.4064" layer="16"/>
-<wire x1="33.19" y1="13.65" x2="30.16" y2="13.65" width="0.4064" layer="16"/>
+<wire x1="30.65" y1="13.65" x2="30.16" y2="13.65" width="0.4064" layer="16"/>
 <wire x1="30.16" y1="13.65" x2="27.94" y2="11.43" width="0.4064" layer="16"/>
 <wire x1="27.94" y1="11.43" x2="24.13" y2="11.43" width="0.4064" layer="16"/>
@@
 <contactref element="D6" pad="A"/>
 <wire x1="24.13" y1="17.35" x2="24.13" y2="13.97" width="1.27" layer="16"/>
-<wire x1="24.13" y1="17.35" x2="33.08" y2="17.35" width="0.4064" layer="16"/>
-<wire x1="33.08" y1="17.35" x2="33.19" y2="17.46" width="0.4064" layer="16"/>
+<wire x1="24.13" y1="17.35" x2="30.54" y2="17.35" width="0.4064" layer="16"/>
+<wire x1="30.54" y1="17.35" x2="30.65" y2="17.46" width="0.4064" layer="16"/>
 <wire x1="20.45" y1="17.78" x2="20.88" y2="17.35" width="0.4064" layer="16"/>
 <wire x1="20.88" y1="17.35" x2="24.13" y2="17.35" width="0.4064" layer="16"/>
@@
 </signal>
 <signal name="N$4">
-<contactref element="Q4" pad="3"/>
-<contactref element="Q3" pad="3"/>
 <contactref element="Q1" pad="1"/>
 <contactref element="Q2" pad="1"/>
 <contactref element="R1" pad="2"/>
-<wire x1="35.39" y1="12.7" x2="35.39" y2="16.51" width="0.4064" layer="16"/>
-<wire x1="34.195" y1="20.32" x2="35.39" y2="19.125" width="0.4064" layer="16"/>
-<wire x1="35.39" y1="19.125" x2="35.39" y2="16.51" width="0.4064" layer="16"/>
-<wire x1="40.92" y1="12.96" x2="37.37" y2="16.51" width="0.4064" layer="16"/>
-<wire x1="37.37" y1="16.51" x2="35.39" y2="16.51" width="0.4064" layer="16"/>
-<wire x1="40.92" y1="21.85" x2="35.58" y2="16.51" width="0.4064" layer="16"/>
-<wire x1="35.58" y1="16.51" x2="35.39" y2="16.51" width="0.4064" layer="16"/>
+<contactref element="C3" pad="1"/>
+<wire x1="36.1" y1="20.32" x2="38.23" y2="18.19" width="0.4064" layer="16"/>
+<wire x1="38.23" y1="18.19" x2="38.23" y2="16.51" width="0.4064" layer="16"/>
+<wire x1="40.92" y1="21.85" x2="38.23" y2="19.16" width="0.4064" layer="16"/>
+<wire x1="38.23" y1="19.16" x2="38.23" y2="18.19" width="0.4064" layer="16"/>
+<wire x1="40.92" y1="12.96" x2="38.23" y2="15.65" width="0.4064" layer="16"/>
+<wire x1="38.23" y1="15.65" x2="38.23" y2="16.51" width="0.4064" layer="16"/>
 </signal>
 <signal name="N$6">
@@
 <contactref element="Q4" pad="1"/>
 <contactref element="Q3" pad="1"/>
-<wire x1="33.19" y1="15.56" x2="28.26" y2="15.56" width="0.4064" layer="16"/>
+<wire x1="30.65" y1="15.56" x2="28.26" y2="15.56" width="0.4064" layer="16"/>
 <wire x1="28.26" y1="15.56" x2="26.67" y2="13.97" width="0.4064" layer="16"/>
-<wire x1="33.19" y1="15.56" x2="34.29" y2="14.46" width="0.4064" layer="16"/>
-<wire x1="34.29" y1="14.46" x2="34.29" y2="12.85" width="0.4064" layer="16"/>
-<wire x1="34.29" y1="12.85" x2="33.19" y2="11.75" width="0.4064" layer="16"/>
+<wire x1="30.65" y1="15.56" x2="31.75" y2="14.46" width="0.4064" layer="16"/>
+<wire x1="31.75" y1="14.46" x2="31.75" y2="12.85" width="0.4064" layer="16"/>
+<wire x1="31.75" y1="12.85" x2="30.65" y2="11.75" width="0.4064" layer="16"/>
 </signal>
 <signal name="N$9">
@@
 <wire x1="8.89" y1="21.59" x2="23.29" y2="21.59" width="1.27" layer="16"/>
 <wire x1="23.29" y1="21.59" x2="24.13" y2="20.75" width="1.27" layer="16"/>
-<wire x1="31.845" y1="20.32" x2="24.56" y2="20.32" width="0.4064" layer="16"/>
+<wire x1="33.75" y1="20.32" x2="24.56" y2="20.32" width="0.4064" layer="16"/>
 <wire x1="24.56" y1="20.32" x2="24.13" y2="20.75" width="0.4064" layer="16"/>
 <wire x1="40.92" y1="26.41" x2="13.71" y2="26.41" width="1.27" layer="16"/>
@@
 </polygon>
 </signal>
+<signal name="N$10">
+<contactref element="Q4" pad="3"/>
+<contactref element="Q3" pad="3"/>
+<wire x1="32.85" y1="12.7" x2="32.85" y2="15.24" width="0.4064" layer="16"/>
+<contactref element="C3" pad="2"/>
+<wire x1="32.85" y1="15.24" x2="32.85" y2="16.51" width="0.4064" layer="16"/>
+<wire x1="35.43" y1="16.51" x2="34.12" y2="16.51" width="0.4064" layer="16"/>
+<wire x1="34.12" y1="16.51" x2="32.85" y2="15.24" width="0.4064" layer="16"/>
+</signal>
 </signals>
