File: Power/Step-Down Tests/NCP1200.sch (EAGLE design)
At the start: 20 parts, among them Q1 NTD20P06LT4G, Q2 NTD20P06LT4G, Q3 BSS84, Q4 BSS123, X1 MKDSN1,5/3-5,08, X2 MKDSN1,5/3-5,08

Commit message: Some minor changes
Parts:
- added C3: 10u, rcl:C-EUC1210
Connections:
- new net N$10: C3.2, Q3.D, Q4.D
- net N$4: now also C3.1; no longer Q3.D, Q4.D
Changed lines of the file:
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@@
 <part name="GND6" library="supply1" deviceset="GND" device=""/>
 <part name="C2" library="rcl" deviceset="CPOL-EU" device="E3.5-8" value="1000u 16V"/>
+<part name="C3" library="rcl" deviceset="C-EU" device="C1210" value="10u"/>
 </parts>
 <sheets>
@@
 <instance part="GND6" gate="1" x="137.16" y="30.48"/>
 <instance part="C2" gate="G$1" x="137.16" y="81.28"/>
+<instance part="C3" gate="G$1" x="66.04" y="58.42"/>
 </instances>
 <busses>
@@
 <net name="N$4" class="0">
 <segment>
-<pinref part="Q4" gate="G$1" pin="D"/>
-<pinref part="Q3" gate="G$1" pin="D"/>
-<wire x1="73.66" y1="30.48" x2="73.66" y2="33.02" width="0.1524" layer="91"/>
 <pinref part="Q1" gate="G$1" pin="G"/>
-<wire x1="73.66" y1="33.02" x2="73.66" y2="35.56" width="0.1524" layer="91"/>
 <wire x1="66.04" y1="83.82" x2="66.04" y2="71.12" width="0.1524" layer="91"/>
 <pinref part="Q2" gate="G$1" pin="G"/>
 <wire x1="73.66" y1="73.66" x2="73.66" y2="71.12" width="0.1524" layer="91"/>
 <wire x1="73.66" y1="71.12" x2="66.04" y2="71.12" width="0.1524" layer="91"/>
-<wire x1="73.66" y1="33.02" x2="66.04" y2="33.02" width="0.1524" layer="91"/>
-<wire x1="66.04" y1="33.02" x2="66.04" y2="66.04" width="0.1524" layer="91"/>
-<junction x="73.66" y="33.02"/>
 <junction x="66.04" y="71.12"/>
 <pinref part="R1" gate="G$1" pin="2"/>
 <wire x1="66.04" y1="66.04" x2="66.04" y2="71.12" width="0.1524" layer="91"/>
+<pinref part="C3" gate="G$1" pin="1"/>
+<wire x1="66.04" y1="66.04" x2="66.04" y2="60.96" width="0.1524" layer="91"/>
 <junction x="66.04" y="66.04"/>
 </segment>
@@
 </segment>
 </net>
+<net name="N$10" class="0">
+<segment>
+<pinref part="Q3" gate="G$1" pin="D"/>
+<pinref part="Q4" gate="G$1" pin="D"/>
+<wire x1="73.66" y1="30.48" x2="73.66" y2="33.02" width="0.1524" layer="91"/>
+<wire x1="73.66" y1="33.02" x2="73.66" y2="35.56" width="0.1524" layer="91"/>
+<junction x="73.66" y="33.02"/>
+<wire x1="73.66" y1="33.02" x2="66.04" y2="33.02" width="0.1524" layer="91"/>
+<pinref part="C3" gate="G$1" pin="2"/>
+<wire x1="66.04" y1="53.34" x2="66.04" y2="33.02" width="0.1524" layer="91"/>
+</segment>
+</net>
