File: Power/Nichrome/Power_5V-8A_CurLim.brd (EAGLE design)
At the start: 105.4 x 61.3 mm, 56 parts, among them IC1 LM358D, Q1 STP13NK60Z, T1 TRANS-1/1EFD25-10, T2 TRANS-1/1220-12, X1 CON-5.08-03P, X2 CON-5.08-03P

Commit message: Аккуратность
Parts:
- Q1: device transistor-power:TO220BV -> Namenlos:TO-220V
- R10: device rcl:0207/10 -> Namenlos:MF-0125
- R5, R6: device rcl:0411/12 -> Namenlos:KNP-100B
- moved D2 11.4 mm to (30.5, 50.8)
- moved D4 3.81 mm to (30.5, 39.4)
- moved D6 3.81 mm to (30.5, 43.2)
- moved D5 3.81 mm to (30.5, 47.0)
- moved R16 3.42 mm to (82.5, 55.2), turned to 270 degrees
- moved R5 2.54 mm to (57.1, 27.9)
- moved R6 1.90 mm to (61.7, 17.2)
- moved NTC 1.27 mm to (6.99, 3.17)
- moved B1 1.27 mm to (17.1, 11.4)
- moved X1 1.27 mm to (5.08, 14.0)
- moved R17 0.64 mm to (57.1, 42.5)
- moved U$2 0.64 mm to (34.9, 66.7)
Connections:
- net N$11: now also Q1.1; no longer Q1.G
- net N$12: now also Q1.3; no longer Q1.S
- net N$8: now also Q1.2; no longer Q1.D
Routing:
- net N$19: track 9.03 -> 26.6 mm
- net N$18: track 66.3 -> 81.5 mm
- net N$30: track 26.2 -> 15.6 mm
- net N$6: track 66.8 -> 61.1 mm
- net N$12: track 26.4 -> 21.8 mm
- net N$33: track 45.9 -> 42.4 mm
- net N$5: track 148.0 -> 146.5 mm
- net N$1: track 33.0 -> 34.2 mm
- net N$35: track 10.3 -> 11.4 mm
- net GND: track 199.6 -> 200.7 mm
- net N$36: track 17.5 -> 16.7 mm
- net N$2: track 52.1 -> 52.8 mm
- net +3V3: track 55.4 -> 56.0 mm
- added copper zone on layer 16, net GND
- added copper zone on layer 16, net N$44
Other:
- board size 105.4 x 61.3 mm -> 105.4 x 62.5 mm

Commit message: Перделка
Надо всё переделать
Parts:
- B1: value RECTIFIER-KBL -> (none); device rectifier:KBL -> Namenlos:KBL
- C1: device rcl:EB22,5D -> Namenlos:C_D25-G10-CLAMP
- C10, C9: device rcl:C1206 -> Namenlos:C1206
- C11, C4, C7: device rcl:C0805 -> Namenlos:C0805
- C2: device rcl:C050-024X044 -> Namenlos:C050-024X044
- C3: device rcl:E5-5 -> Namenlos:E5-5
- C5, C8: device rcl:E3,5-8 -> Namenlos:E3,5-8
- C6: device rcl:E5-10,5 -> Namenlos:E5-10,5
- D1: device diode:DO41-7.6 -> Namenlos:DO15-12
- D2, D4, D5, D6: device diode:DO-214AC -> Namenlos:DO214AC
- D3: device diode:TO220ABS -> Namenlos:TO-220V
- D7, D8: device diode:SOD523 -> Namenlos:SOD523
- IC1: value LM358D -> OP-AMP-2LM358D; device linear:SO08 -> Namenlos:SO8
- OK1: value PC817 -> (none); device optocoupler:DIL04 -> Namenlos:DIL04
- P6KE200: device diode:DO15-12 -> Namenlos:DO201-15
- R11, R13, R15, R16, R17, R18, R2, R3, R4, R7, R8, R9: device rcl:R1206 -> Namenlos:R1206
- R12: device rcl:R2512 -> Namenlos:R2512
- R19, R20, R21: device rcl:R0805 -> Namenlos:R0805
- T1: device _Transformers:EFD25_10PIN -> Namenlos:EFD25_10PIN
- T2: device _Transformers:32.5-27.5-27.5 -> Namenlos:32.5-27.5-27.5
- U$1: value NCP1200-100SO -> PW-NCP12NCP1200D; device NCP1200:SOP8 -> Namenlos:SO8
- U$3: value TL431-IDBVR -> IC-TL431DBV; device TL431:SOT23-5 -> Namenlos:SOT23-5L
- U$4, U$5: device heatsink:SK95-3M3_HOLE -> Namenlos:SK95-3M3_HOLE
- moved U$3 1.27 mm to (53.3, 49.5)
Connections:
- net +2V5: now also U$3.3, U$3.4; no longer U$3.C, U$3.R
- net GND: now also U$3.5; no longer U$3.A
- net N$17: now also D3.1, D3.3; no longer D3.A1, D3.A2
- net N$18: now also D3.2; no longer D3.C
Routing:
- net N$6: track 61.1 -> 59.8 mm
- net N$7: track 2.54 -> 1.27 mm
- net GND: track 200.7 -> 199.4 mm
- net N$8: track 31.8 -> 33.0 mm
- net N$3: track 9.99 -> 10.7 mm
- net N$12: track 21.8 -> 22.4 mm
- net N$15: track 11.4 -> 12.0 mm
- net N$14: track 8.30 -> 8.85 mm
- net N$10: track 9.79 -> 9.24 mm
- net N$5: track 146.5 -> 147.1 mm

Commit message: _
Parts:
- removed P6KE200: (no value), Namenlos:DO201-15
- added C12: 470u, Namenlos:E5-10,5
- added D9: HER, Namenlos:DO201-15
- D1: value ES1J -> P6KE200
- moved R10 24.8 mm to (60.3, 11.4)
- moved D1 20.8 mm to (67.3, 7.20), flipped to the top, turned to 290 degrees
- moved C6 11.8 mm to (106.0, 32.1)
- moved D3 8.64 mm to (105.4, 14.0)
- moved U$5 8.13 mm to (104.8, 14.0)
- moved R12 8.08 mm to (85.7, 46.4)
- moved C2 6.02 mm to (85.7, 29.8)
- moved T1 5.75 mm to (86.4, 14.0)
- moved R6 5.08 mm to (61.7, 22.3)
- moved C1 2.54 mm to (45.7, 12.1)
- moved R1 1.82 mm to (28.1, 16.1), turned to 260 degrees
- moved Q1 1.42 mm to (48.9, 33.0)
- moved U$4 1.42 mm to (48.9, 33.0)
- moved T2 1.27 mm to (14.6, 45.7)
- moved R5 0.90 mm to (56.5, 28.6)
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Connections:
- net GND: now also C12.-
- net N$18: now also C12.+
- net N$6: now also D1.A, T1.5; no longer P6KE200.A, T1.4
- net N$7: now also D9.C; no longer P6KE200.C
- net N$8: now also D9.A, T1.1; no longer D1.A, T1.2
Routing:
- net GND: track 199.4 -> 58.1 mm
- net N$17: track 20.8 -> 32.4 mm
- net N$6: track 59.8 -> 69.1 mm
- net N$8: track 33.0 -> 27.4 mm
- net N$20: track 8.82 -> 13.7 mm
- net N$4: track 6.40 -> 11.1 mm
- net N$30: track 15.5 -> 20.1 mm
- net N$5: track 147.1 -> 150.5 mm
- net N$11: track 12.1 -> 14.9 mm
- net N$7: track 1.27 -> 3.58 mm
- net N$12: track 22.4 -> 20.9 mm
- net N$2: track 52.8 -> 54.1 mm
- net N$1: track 34.4 -> 35.6 mm
- net N$19: track 26.4 -> 25.3 mm
- net N$10: track 9.24 -> 8.46 mm
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Other:
- board size 105.4 x 62.5 mm -> 111.1 x 62.5 mm
