File: MicroControl/Noise Maker/Main.sch (EAGLE design)
At the start: 1 part, among them IC1 STM8L151G6U6

Commit message: Noise Maker
Parts:
- added C1, C2: (no value), rcl:C-EUC0805
- added IC2: 317EMP, linear:317EMP
- added Q1: BSS123, transistor-small-signal:BSS123
- added R1, R2, R3, R8: (no value), rcl:R-EU_R0805
- added R4, R5, R6, R7: (no value), rcl:R-EU_R1206
- added R9: 680R, rcl:R-US_R0805
- added X1, X2: MKDSN1,5/2-5,08, con-phoenix-508:MKDSN1,5/2-5,08
Connections:
- new net GND: C1.2, C2.2, IC1.GND, R3.1, R5.1, R7.2, R8.1, X1-1.KL, X2-2.KL
- new net N$10: Q1.D, R9.1
- new net N$11: Q1.S, X2-1.KL
- new net N$3: IC2.ADJ, R2.1, R3.2, R4.1, R5.2
- new net N$4: C2.1, IC1.VCC, IC2.VO, R2.2, R4.2
- new net N$8: Q1.G, R1.2, R6.1, R7.1, R8.2
- new net VCC: C1.1, IC2.VI, R9.2, X1-2.KL
- net N$1: now also R1.1, R6.2
Changed lines of the file:
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@@
 <parts>
 <part name="IC1" library="Namenlos" deviceset="STM8L151G6U6" device=""/>
+<part name="Q1" library="transistor-small-signal" deviceset="BSS123" device=""/>
+<part name="R1" library="rcl" deviceset="R-EU_" device="R0805"/>
+<part name="IC2" library="linear" deviceset="*317" device="EMP"/>
+<part name="R2" library="rcl" deviceset="R-EU_" device="R0805"/>
+<part name="R3" library="rcl" deviceset="R-EU_" device="R0805"/>
+<part name="R4" library="rcl" deviceset="R-EU_" device="R1206"/>
+<part name="R5" library="rcl" deviceset="R-EU_" device="R1206"/>
+<part name="C1" library="rcl" deviceset="C-EU" device="C0805"/>
+<part name="C2" library="rcl" deviceset="C-EU" device="C0805"/>
+<part name="GND1" library="supply1" deviceset="GND" device=""/>
+<part name="GND2" library="supply1" deviceset="GND" device=""/>
+<part name="R6" library="rcl" deviceset="R-EU_" device="R1206"/>
+<part name="R7" library="rcl" deviceset="R-EU_" device="R1206"/>
+<part name="R8" library="rcl" deviceset="R-EU_" device="R0805"/>
+<part name="P+1" library="supply1" deviceset="VCC" device=""/>
+<part name="P+2" library="supply1" deviceset="VCC" device=""/>
+<part name="R9" library="rcl" deviceset="R-US_" device="R0805" value="680R"/>
+<part name="X1" library="con-phoenix-508" deviceset="MKDSN1,5/2-5,08" device=""/>
+<part name="P+3" library="supply1" deviceset="VCC" device=""/>
+<part name="GND3" library="supply1" deviceset="GND" device=""/>
+<part name="X2" library="con-phoenix-508" deviceset="MKDSN1,5/2-5,08" device=""/>
+<part name="GND4" library="supply1" deviceset="GND" device=""/>
 </parts>
 <sheets>
@@
 <instances>
 <instance part="IC1" gate="G$1" x="68.58" y="71.12"/>
+<instance part="Q1" gate="G$1" x="121.92" y="48.26"/>
+<instance part="R1" gate="G$1" x="109.22" y="45.72"/>
+<instance part="IC2" gate="A1" x="12.7" y="40.64"/>
+<instance part="R2" gate="G$1" x="25.4" y="38.1" rot="R90"/>
+<instance part="R3" gate="G$1" x="25.4" y="22.86" rot="R90"/>
+<instance part="R4" gate="G$1" x="30.48" y="38.1" rot="R90"/>
+<instance part="R5" gate="G$1" x="30.48" y="22.86" rot="R90"/>
+<instance part="C1" gate="G$1" x="0" y="38.1"/>
+<instance part="C2" gate="G$1" x="35.56" y="40.64"/>
+<instance part="GND1" gate="1" x="15.24" y="15.24"/>
+<instance part="GND2" gate="1" x="109.22" y="20.32"/>
+<instance part="R6" gate="G$1" x="109.22" y="43.18" rot="R180"/>
+<instance part="R7" gate="G$1" x="116.84" y="30.48" rot="R270"/>
+<instance part="R8" gate="G$1" x="119.38" y="30.48" rot="R90"/>
+<instance part="P+1" gate="VCC" x="-7.62" y="68.58"/>
+<instance part="P+2" gate="VCC" x="121.92" y="78.74"/>
+<instance part="R9" gate="G$1" x="121.92" y="63.5" rot="R90"/>
+<instance part="X1" gate="-1" x="-20.32" y="104.14" rot="R180"/>
+<instance part="X1" gate="-2" x="-20.32" y="109.22" rot="R180"/>
+<instance part="P+3" gate="VCC" x="-12.7" y="114.3"/>
+<instance part="GND3" gate="1" x="-12.7" y="99.06"/>
+<instance part="X2" gate="-1" x="139.7" y="48.26" rot="R90"/>
+<instance part="X2" gate="-2" x="144.78" y="48.26" rot="R90"/>
+<instance part="GND4" gate="1" x="144.78" y="25.4"/>
 </instances>
 <busses>
@@
 <segment>
 <pinref part="IC1" gate="G$1" pin="PD2/TIM1_CH1"/>
-<wire x1="96.52" y1="45.72" x2="134.62" y2="45.72" width="0.1524" layer="91"/>
-<wire x1="134.62" y1="45.72" x2="134.62" y2="43.18" width="0.1524" layer="91"/>
-</segment>
-</net>
+<wire x1="96.52" y1="45.72" x2="101.6" y2="45.72" width="0.1524" layer="91"/>
+<pinref part="R1" gate="G$1" pin="1"/>
+<pinref part="R6" gate="G$1" pin="2"/>
+<wire x1="101.6" y1="45.72" x2="104.14" y2="45.72" width="0.1524" layer="91"/>
+<wire x1="104.14" y1="43.18" x2="101.6" y2="43.18" width="0.1524" layer="91"/>
+<wire x1="101.6" y1="43.18" x2="101.6" y2="45.72" width="0.1524" layer="91"/>
+<junction x="101.6" y="45.72"/>
+</segment>
+</net>
+<net name="N$3" class="0">
+<segment>
+<pinref part="IC2" gate="A1" pin="ADJ"/>
+<wire x1="12.7" y1="35.56" x2="12.7" y2="30.48" width="0.1524" layer="91"/>
+<wire x1="12.7" y1="30.48" x2="25.4" y2="30.48" width="0.1524" layer="91"/>
+<pinref part="R4" gate="G$1" pin="1"/>
+<wire x1="25.4" y1="30.48" x2="30.48" y2="30.48" width="0.1524" layer="91"/>
+<wire x1="30.48" y1="30.48" x2="30.48" y2="33.02" width="0.1524" layer="91"/>
+<pinref part="R5" gate="G$1" pin="2"/>
+<wire x1="30.48" y1="27.94" x2="30.48" y2="30.48" width="0.1524" layer="91"/>
+<junction x="30.48" y="30.48"/>
+<pinref part="R2" gate="G$1" pin="1"/>
+<wire x1="25.4" y1="33.02" x2="25.4" y2="30.48" width="0.1524" layer="91"/>
+<junction x="25.4" y="30.48"/>
+<pinref part="R3" gate="G$1" pin="2"/>
+<wire x1="25.4" y1="30.48" x2="25.4" y2="27.94" width="0.1524" layer="91"/>
+</segment>
+</net>
+<net name="N$4" class="0">
+<segment>
+<pinref part="IC2" gate="A1" pin="VO"/>
+<pinref part="R2" gate="G$1" pin="2"/>
+<wire x1="22.86" y1="43.18" x2="25.4" y2="43.18" width="0.1524" layer="91"/>
+<pinref part="R4" gate="G$1" pin="2"/>
+<wire x1="25.4" y1="43.18" x2="30.48" y2="43.18" width="0.1524" layer="91"/>
+<junction x="25.4" y="43.18"/>
+<pinref part="IC1" gate="G$1" pin="VCC"/>
+<wire x1="30.48" y1="43.18" x2="35.56" y2="43.18" width="0.1524" layer="91"/>
+<junction x="30.48" y="43.18"/>
+<pinref part="C2" gate="G$1" pin="1"/>
+<wire x1="35.56" y1="43.18" x2="43.18" y2="43.18" width="0.1524" layer="91"/>
+<junction x="35.56" y="43.18"/>
+</segment>
+</net>
+<net name="GND" class="0">
+<segment>
+<pinref part="IC1" gate="G$1" pin="GND"/>
+<wire x1="43.18" y1="40.64" x2="40.64" y2="40.64" width="0.1524" layer="91"/>
+<wire x1="40.64" y1="40.64" x2="40.64" y2="17.78" width="0.1524" layer="91"/>
+<pinref part="R5" gate="G$1" pin="1"/>
+<wire x1="40.64" y1="17.78" x2="35.56" y2="17.78" width="0.1524" layer="91"/>
+<pinref part="R3" gate="G$1" pin="1"/>
+<wire x1="35.56" y1="17.78" x2="30.48" y2="17.78" width="0.1524" layer="91"/>
+<wire x1="30.48" y1="17.78" x2="25.4" y2="17.78" width="0.1524" layer="91"/>
+<junction x="30.48" y="17.78"/>
+<pinref part="C2" gate="G$1" pin="2"/>
+<wire x1="35.56" y1="35.56" x2="35.56" y2="17.78" width="0.1524" layer="91"/>
+<junction x="35.56" y="17.78"/>
+<pinref part="C1" gate="G$1" pin="2"/>
+<wire x1="0" y1="33.02" x2="0" y2="17.78" width="0.1524" layer="91"/>
+<wire x1="0" y1="17.78" x2="15.24" y2="17.78" width="0.1524" layer="91"/>
+<junction x="25.4" y="17.78"/>
+<pinref part="GND1" gate="1" pin="GND"/>
+<wire x1="15.24" y1="17.78" x2="25.4" y2="17.78" width="0.1524" layer="91"/>
+<junction x="15.24" y="17.78"/>
+</segment>
+<segment>
+<pinref part="R7" gate="G$1" pin="2"/>
+<pinref part="R8" gate="G$1" pin="1"/>
+<wire x1="116.84" y1="25.4" x2="119.38" y2="25.4" width="0.1524" layer="91"/>
+<pinref part="GND2" gate="1" pin="GND"/>
+<wire x1="116.84" y1="25.4" x2="109.22" y2="25.4" width="0.1524" layer="91"/>
+<wire x1="109.22" y1="25.4" x2="109.22" y2="22.86" width="0.1524" layer="91"/>
+<junction x="116.84" y="25.4"/>
+</segment>
+<segment>
+<pinref part="X1" gate="-1" pin="KL"/>
+<pinref part="GND3" gate="1" pin="GND"/>
+<wire x1="-17.78" y1="104.14" x2="-12.7" y2="104.14" width="0.1524" layer="91"/>
+<wire x1="-12.7" y1="104.14" x2="-12.7" y2="101.6" width="0.1524" layer="91"/>
+</segment>
+<segment>
+<pinref part="X2" gate="-2" pin="KL"/>
+<wire x1="144.78" y1="45.72" x2="144.78" y2="27.94" width="0.1524" layer="91"/>
+<pinref part="GND4" gate="1" pin="GND"/>
+</segment>
+</net>
+<net name="N$8" class="0">
+<segment>
+<pinref part="R7" gate="G$1" pin="1"/>
+<pinref part="R8" gate="G$1" pin="2"/>
+<wire x1="116.84" y1="35.56" x2="119.38" y2="35.56" width="0.1524" layer="91"/>
+<pinref part="Q1" gate="G$1" pin="G"/>
+<pinref part="R1" gate="G$1" pin="2"/>
+<wire x1="116.84" y1="45.72" x2="114.3" y2="45.72" width="0.1524" layer="91"/>
+<pinref part="R6" gate="G$1" pin="1"/>
+<wire x1="114.3" y1="43.18" x2="114.3" y2="45.72" width="0.1524" layer="91"/>
+<junction x="114.3" y="45.72"/>
+<wire x1="116.84" y1="35.56" x2="116.84" y2="45.72" width="0.1524" layer="91"/>
+<junction x="116.84" y="35.56"/>
+<junction x="116.84" y="45.72"/>
+</segment>
+</net>
+<net name="VCC" class="0">
+<segment>
+<pinref part="IC2" gate="A1" pin="VI"/>
+<pinref part="C1" gate="G$1" pin="1"/>
+<wire x1="2.54" y1="43.18" x2="0" y2="43.18" width="0.1524" layer="91"/>
+<wire x1="0" y1="43.18" x2="0" y2="40.64" width="0.1524" layer="91"/>
+<wire x1="0" y1="43.18" x2="-7.62" y2="43.18" width="0.1524" layer="91"/>
+<junction x="0" y="43.18"/>
+<wire x1="-7.62" y1="43.18" x2="-7.62" y2="66.04" width="0.1524" layer="91"/>
+<pinref part="P+1" gate="VCC" pin="VCC"/>
+</segment>
+<segment>
+<pinref part="R9" gate="G$1" pin="2"/>
+<pinref part="P+2" gate="VCC" pin="VCC"/>
+<wire x1="121.92" y1="68.58" x2="121.92" y2="76.2" width="0.1524" layer="91"/>
+</segment>
+<segment>
+<pinref part="P+3" gate="VCC" pin="VCC"/>
+<pinref part="X1" gate="-2" pin="KL"/>
+<wire x1="-12.7" y1="111.76" x2="-12.7" y2="109.22" width="0.1524" layer="91"/>
+<wire x1="-12.7" y1="109.22" x2="-17.78" y2="109.22" width="0.1524" layer="91"/>
+</segment>
+</net>
+<net name="N$10" class="0">
+<segment>
+<pinref part="R9" gate="G$1" pin="1"/>
+<pinref part="Q1" gate="G$1" pin="D"/>
+<wire x1="121.92" y1="58.42" x2="121.92" y2="53.34" width="0.1524" layer="91"/>
+</segment>
+</net>
+<net name="N$11" class="0">
+<segment>
+<pinref part="Q1" gate="G$1" pin="S"/>
+<wire x1="121.92" y1="43.18" x2="137.16" y2="43.18" width="0.1524" layer="91"/>
+<pinref part="X2" gate="-1" pin="KL"/>
+<wire x1="137.16" y1="43.18" x2="139.7" y2="43.18" width="0.1524" layer="91"/>
+<wire x1="139.7" y1="43.18" x2="139.7" y2="45.72" width="0.1524" layer="91"/>
+</segment>
+</net>

Commit message: Тщшыу
Parts:
- removed IC2: 317EMP, linear:317EMP
- removed R3, R8: (no value), rcl:R-EU_R0805
- removed R4, R5, R6: (no value), rcl:R-EU_R1206
- removed R9: 680R, rcl:R-US_R0805
- removed X1, X2: MKDSN1,5/2-5,08, con-phoenix-508:MKDSN1,5/2-5,08
- added C3, C4: 10n, rcl:C-EUC0805
- added IC3: TS520533, v-reg:TS520533
- added JP1, JP2: (no value), pinhead:PINHD-1X2
- C1, C2: value (none) -> 10u
- IC1: value STM8L151G6U6 -> STM8L151X4/6G6U6; device Namenlos:STM8L151G6U6 -> Namenlos:STM8L151X4/6G6U6
- Q1: value BSS123 -> (none); device transistor-small-signal:BSS123 -> Namenlos:FET-NPF-2X2
- R1, R2: device rcl:R-EU_R0805 -> Namenlos:R_0805
- R7: device rcl:R-EU_R1206 -> Namenlos:R_0805
Connections:
- removed net N$10: Q1.D, R9.1
- removed net N$11: Q1.S, X2-1.KL
- new net N$13: JP2.2
- new net N$2: C3.1, IC3.CB
- new net N$7: Q1.S, R2.2
- new net N$9: JP1.2, Q1.D
- net GND: now also C3.2, IC3.GND, JP2.1, R2.1; no longer R3.1, R5.1, R8.1, X1-1.KL, X2-2.KL
- net N$1: now also IC1.PD4/TIM1_CH2; no longer IC1.PD2/TIM1_CH1, R6.2
- net N$3: now also C4.1, IC1.NRST/PA1; no longer IC2.ADJ, R2.1, R3.2, R4.1, R5.2
- net N$4: now also C4.2, IC3.VOUT; no longer IC2.VO, R2.2, R4.2
- net N$8: no longer R6.1, R8.2
- net VCC: now also IC3.CE, IC3.VIN, JP1.1; no longer IC2.VI, R9.2, X1-2.KL
Other:
- moved on the sheet: R2
