File: Thermoneter/Main.brd (EAGLE design)
At the start: 66.7 x 55.5 mm, 65 parts, among them IC1 POWER-TNY264PN, IC2 STM8L151X4/6G6U6, T1 TRANS-1/1EFD20, X1 CON-5.08-03P, X2 STM-SWIMPINS

Commit message: _
Parts:
- moved R38 4.45 mm to (50.2, 36.2)
- moved C6 3.59 mm to (44.5, 30.5)
- moved D4 2.54 mm to (40.6, 40.6)
- moved X2 2.54 mm to (38.7, 39.4)
Routing:
- net +3V3: track 154.0 -> 147.0 mm
- net GND: track 110.1 -> 114.6 mm
- net N$4: track 70.8 -> 74.6 mm
- net N$28: track 2.48 -> 6.07 mm
- net N$26: track 3.73 -> 6.82 mm
- net N$27: track 5.70 -> 3.91 mm
- net N$3: track 59.4 -> 61.2 mm
- net N$49: track 97.8 -> 99.4 mm
- net N$14: track 15.2 -> 14.3 mm
- net N$13: track 17.0 -> 16.3 mm
- added copper zone on layer 16, net N$50
