File: Thermoneter/RefVolt.brd (EAGLE design)
At the start: 15.2 x 16.5 mm, 8 parts

Commit message: _
Parts:
- removed JP2, JP3: (no value), pinhead:1X02
- removed R2, R3, R4: 0, Namenlos:R0805
- removed U$1, U$2: FET-N/PNTZD3155C, Namenlos:SOT-563
- added C1: (no value), Namenlos:C0805
- added IC1: OP-AMP-1TSV521ICT, Namenlos:SC70-5L
- added R1: (no value), Namenlos:RJ9W
- JP1: device pinhead:1X02 -> pinhead:1X03/90
- moved JP1 13.0 mm to (3.81, -1.27), turned to 180 degrees
Connections:
- removed net N$10: R2.2, R3.1, U$2.3
- removed net N$11: JP1.1, R4.2, U$1.5
- removed net N$12: JP2.2, U$1.2
- removed net N$5: R4.1, U$2.1, U$2.4
- removed net N$7: JP1.2, U$1.1, U$1.4, U$2.5
- removed net N$8: JP2.1, U$2.2
- removed net N$9: R2.1, U$1.3
- new net N$1: IC1.3, IC1.4, JP1.2
- new net N$4: IC1.1, R1.W
- net GND: now also C1.2, IC1.2, JP1.3, R1.A; no longer JP3.1, U$1.6, U$2.6
- net VCC: now also C1.1, IC1.5, JP1.1, R1.B; no longer JP3.2, R3.2
Routing:
- net N$12: track 13.3 -> 0.00 mm
- net GND: track 21.0 -> 10.9 mm
- net VCC: track 3.35 -> 10.9 mm
- net N$7: track 7.19 -> 0.00 mm
- net N$10: track 5.59 -> 0.00 mm
- net N$1: track 0.00 -> 5.50 mm
- net N$11: track 5.08 -> 0.00 mm
- net N$8: track 4.67 -> 0.00 mm
- net N$5: track 4.44 -> 0.00 mm
- net N$4: track 0.00 -> 2.88 mm
- net N$9: track 2.35 -> 0.00 mm
- net N$2: track 0.00 -> 1.27 mm
- net N$6: track 0.00 -> 1.27 mm
- net N$3: track 0.00 -> 1.27 mm
- added copper zone on layer 1, net N$5
- removed copper zone on layer 1, net GND
Other:
- board size 15.2 x 16.5 mm -> 10.1 x 12.4 mm

Commit message: _Something
Parts:
- added R2: (no value), Namenlos:R0805
- added TL1: IC-TL431CDBZR, Namenlos:SOT23
- moved C1 8.03 mm to (6.35, 12.7)
- moved R1 5.08 mm to (3.81, 5.71), turned to 0 degrees
- moved IC1 3.24 mm to (4.45, 10.2), turned to 180 degrees
Connections:
- new net N$7: IC1.1, R2.1, TL1.1, TL1.2
- net GND: now also R1.B, TL1.3; no longer R1.A
- net N$1: now also R1.W; no longer IC1.4, JP1.2
- net N$4: now also IC1.4, JP1.2, R1.A; no longer IC1.1, R1.W
- net VCC: now also R2.2; no longer R1.B
Routing:
- net N$7: track 0.00 -> 11.7 mm
- net GND: track 10.9 -> 18.0 mm
- net N$4: track 2.88 -> 8.88 mm
- net N$1: track 5.50 -> 11.5 mm
- net VCC: track 10.9 -> 15.6 mm
- net N$2: track 1.27 -> 0.00 mm
- net N$3: track 1.27 -> 0.00 mm
- added copper zone on layer 1, net N$2
- removed copper zone on layer 1, net N$5
Other:
- board size 10.1 x 12.4 mm -> 10.1 x 16.2 mm
- board text added: "C1"
- board text added: "IC1"
- board text added: "JP1"
- board text added: "R1"
- board text added: "R2"
- board text added: "TL1"
Changed lines of the file:
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@@
 <?xml version="1.0" encoding="utf-8"?>
 <!DOCTYPE eagle SYSTEM "eagle.dtd">
-<eagle version="8.0.0">
+<eagle version="8.0.1">
 <drawing>
 <settings>
@@
 <setting verticaltext="up"/>
 </settings>
-<grid distance="0.05" unitdist="inch" unit="mil" style="lines" multiple="1" display="no" altdistance="0.025" altunitdist="inch" altunit="mil"/>
+<grid distance="25" unitdist="mil" unit="mil" style="lines" multiple="1" display="no" altdistance="12.5" altunitdist="mil" altunit="mil"/>
 <layers>
 <layer number="1" name="Top" color="4" fill="1" visible="yes" active="yes"/>
@@
 <layer number="123" name="tTestmark" color="7" fill="1" visible="no" active="yes"/>
 <layer number="124" name="bTestmark" color="7" fill="1" visible="no" active="yes"/>
-<layer number="125" name="_tNames" color="7" fill="1" visible="no" active="yes"/>
+<layer number="125" name="_tNames" color="14" fill="1" visible="yes" active="yes"/>
 <layer number="126" name="_bNames" color="7" fill="1" visible="no" active="yes"/>
 <layer number="127" name="_tValues" color="7" fill="1" visible="no" active="yes"/>
@@
 <board>
 <plain>
-<wire x1="-1.27" y1="12.37" x2="-1.27" y2="1.27" width="0" layer="20"/>
+<wire x1="-1.27" y1="16.18" x2="-1.27" y2="1.27" width="0" layer="20"/>
 <wire x1="-1.27" y1="1.27" x2="0" y2="0" width="0" layer="20"/>
 <wire x1="0" y1="0" x2="7.6" y2="0" width="0" layer="20"/>
 <wire x1="7.6" y1="0" x2="8.87" y2="1.27" width="0" layer="20"/>
-<wire x1="8.87" y1="1.27" x2="8.87" y2="12.37" width="0" layer="20"/>
-<wire x1="8.87" y1="12.37" x2="-1.27" y2="12.37" width="0" layer="20"/>
+<wire x1="8.87" y1="1.27" x2="8.87" y2="16.18" width="0" layer="20"/>
+<wire x1="8.87" y1="16.18" x2="-1.27" y2="16.18" width="0" layer="20"/>
+<text x="7.62" y="11.43" size="1.27" layer="125" rot="R180">C1</text>
+<text x="5.644996875" y="8.809990625" size="1.016" layer="125" rot="R180">IC1</text>
+<text x="8.255" y="2.54" size="1.27" layer="125" ratio="10" rot="R270">JP1</text>
+<text x="-0.762" y="8.382" size="1.27" layer="125" ratio="10">R1</text>
+<text x="5.715" y="15.875" size="1.27" layer="125">R2</text>
+<text x="-1.27" y="8.255" size="1.27" layer="125" rot="R90">TL1</text>
 </plain>
 <attributes>
@@
 </autorouter>
 <elements>
-<element name="IC1" library="Namenlos" package="SC70-5L" value="OP-AMP-1TSV521ICT" x="3.81" y="6.985" rot="R270"/>
+<element name="IC1" library="Namenlos" package="SC70-5L" value="OP-AMP-1TSV521ICT" x="4.445" y="10.16" rot="R180"/>
 <element name="JP1" library="pinhead" package="1X03/90" value="" x="3.81" y="-1.27" rot="R180"/>
-<element name="R1" library="Namenlos" package="RJ9W" value="" x="3.81" y="10.795" rot="R180"/>
-<element name="C1" library="Namenlos" package="C0805" value="" x="3.81" y="5.08" rot="R180"/>
+<element name="R1" library="Namenlos" package="RJ9W" value="" x="3.81" y="5.715"/>
+<element name="C1" library="Namenlos" package="C0805" value="" x="6.35" y="12.7" rot="R180"/>
+<element name="TL1" library="Namenlos" package="SOT23" value="IC-TL431CDBZR" x="0.635" y="10.16" rot="R90"/>
+<element name="R2" library="Namenlos" package="R0805" value="" x="6.35" y="14.605"/>
 </elements>
 <signals>
 <signal name="N$1">
 <contactref element="IC1" pad="3"/>
-<contactref element="IC1" pad="4"/>
-<contactref element="JP1" pad="2"/>
-<wire x1="3.81" y1="6.335" x2="2.96" y2="6.335" width="0.3048" layer="1"/>
-<wire x1="3.81" y1="6.335" x2="4.66" y2="6.335" width="0.3048" layer="1"/>
-<wire x1="3.81" y1="2.54" x2="3.81" y2="6.335" width="0.3048" layer="1"/>
-</signal>
-<signal name="N$4">
 <contactref element="R1" pad="W"/>
-<contactref element="IC1" pad="1"/>
-<wire x1="2.96" y1="7.635" x2="3.81" y2="8.485" width="0.3048" layer="1"/>
-<wire x1="3.81" y1="8.485" x2="3.81" y2="10.16" width="0.3048" layer="1"/>
+<wire x1="3.81" y1="6.35" x2="1.905" y2="8.255" width="0.3048" layer="1"/>
+<wire x1="1.905" y1="8.255" x2="0.9525" y2="8.255" width="0.3048" layer="1"/>
+<wire x1="0.9525" y1="8.255" x2="0.635" y2="8.5725" width="0.3048" layer="1"/>
+<wire x1="0.635" y1="8.5725" x2="0.635" y2="11.7475" width="0.3048" layer="1"/>
+<wire x1="0.635" y1="11.7475" x2="0.9525" y2="12.065" width="0.3048" layer="1"/>
+<wire x1="0.9525" y1="12.065" x2="3.4925" y2="12.065" width="0.3048" layer="1"/>
+<wire x1="3.4925" y1="12.065" x2="3.81" y2="11.7475" width="0.3048" layer="1"/>
+<wire x1="3.81" y1="11.7475" x2="3.81" y2="11.025" width="0.3048" layer="1"/>
+<wire x1="3.81" y1="11.025" x2="3.795" y2="11.01" width="0.3048" layer="1"/>
 </signal>
 <signal name="GND">
 <contactref element="IC1" pad="2"/>
 <contactref element="JP1" pad="3"/>
-<contactref element="R1" pad="A"/>
 <contactref element="C1" pad="2"/>
-<wire x1="2.96" y1="6.985" x2="1.905" y2="6.985" width="0.3048" layer="1"/>
-<wire x1="1.27" y1="6.35" x2="1.905" y2="6.985" width="0.3048" layer="1"/>
-<wire x1="1.27" y1="5.08" x2="1.27" y2="6.35" width="0.3048" layer="1"/>
-<wire x1="1.27" y1="5.08" x2="1.27" y2="2.54" width="0.3048" layer="1"/>
-<wire x1="1.27" y1="10.16" x2="1.27" y2="6.35" width="0.3048" layer="1"/>
-<wire x1="2.635" y1="5.08" x2="1.27" y2="5.08" width="0.3048" layer="1"/>
+<contactref element="R1" pad="B"/>
+<contactref element="TL1" pad="3"/>
+<wire x1="-0.465" y1="10.16" x2="-0.465" y2="8.085" width="0.3048" layer="1"/>
+<wire x1="-0.465" y1="8.085" x2="1.27" y2="6.35" width="0.3048" layer="1"/>
+<wire x1="1.27" y1="6.35" x2="1.27" y2="2.54" width="0.3048" layer="1"/>
+<wire x1="4.445" y1="11.01" x2="4.445" y2="11.97" width="0.3048" layer="1"/>
+<wire x1="4.445" y1="11.97" x2="5.175" y2="12.7" width="0.3048" layer="1"/>
+<wire x1="5.175" y1="12.7" x2="0.635" y2="12.7" width="0.3048" layer="1"/>
+<wire x1="0.635" y1="12.7" x2="-0.635" y2="11.43" width="0.3048" layer="1"/>
+<wire x1="-0.635" y1="11.43" x2="-0.635" y2="10.33" width="0.3048" layer="1"/>
+<wire x1="-0.635" y1="10.33" x2="-0.465" y2="10.16" width="0.3048" layer="1"/>
 </signal>
 <signal name="VCC">
 <contactref element="IC1" pad="5"/>
 <contactref element="JP1" pad="1"/>
-<contactref element="R1" pad="B"/>
 <contactref element="C1" pad="1"/>
-<wire x1="6.35" y1="5.08" x2="4.985" y2="5.08" width="0.3048" layer="1"/>
-<wire x1="6.35" y1="5.08" x2="6.35" y2="2.54" width="0.3048" layer="1"/>
-<wire x1="6.35" y1="6.985" x2="6.35" y2="10.16" width="0.3048" layer="1"/>
-<wire x1="6.35" y1="6.985" x2="6.35" y2="5.08" width="0.3048" layer="1"/>
-<wire x1="4.66" y1="7.635" x2="5.7" y2="7.635" width="0.3048" layer="1"/>
-<wire x1="5.7" y1="7.635" x2="6.35" y2="6.985" width="0.3048" layer="1"/>
+<contactref element="R2" pad="2"/>
+<wire x1="6.35" y1="2.54" x2="7.62" y2="3.81" width="0.3048" layer="1"/>
+<wire x1="7.62" y1="8.255" x2="7.62" y2="3.81" width="0.3048" layer="1"/>
+<wire x1="5.095" y1="9.31" x2="6.565" y2="9.31" width="0.3048" layer="1"/>
+<wire x1="6.565" y1="9.31" x2="7.62" y2="8.255" width="0.3048" layer="1"/>
+<wire x1="7.525" y1="14.605" x2="7.525" y2="12.7" width="0.3048" layer="1"/>
+<wire x1="7.525" y1="12.7" x2="7.525" y2="8.35" width="0.3048" layer="1"/>
+<wire x1="7.525" y1="8.35" x2="7.62" y2="8.255" width="0.3048" layer="1"/>
 </signal>
 <signal name="N$6">
-<wire x1="-0.635" y1="5.08" x2="0.635" y2="5.08" width="0.3048" layer="1"/>
+<wire x1="-0.635" y1="4.7625" x2="0.635" y2="4.7625" width="0.3048" layer="1"/>
+</signal>
+<signal name="N$4">
+<contactref element="R1" pad="A"/>
+<contactref element="IC1" pad="4"/>
+<contactref element="JP1" pad="2"/>
+<wire x1="3.81" y1="2.54" x2="3.81" y2="3.81" width="0.3048" layer="1"/>
+<wire x1="6.35" y1="6.35" x2="3.81" y2="3.81" width="0.3048" layer="1"/>
+<wire x1="3.795" y1="9.31" x2="3.795" y2="8.905" width="0.3048" layer="1"/>
+<wire x1="3.795" y1="8.905" x2="6.35" y2="6.35" width="0.3048" layer="1"/>
+</signal>
+<signal name="N$7">
+<contactref element="TL1" pad="1"/>
+<contactref element="R2" pad="1"/>
+<contactref element="TL1" pad="2"/>
+<contactref element="IC1" pad="1"/>
+<wire x1="5.93" y1="11.01" x2="5.095" y2="11.01" width="0.3048" layer="1"/>
+<wire x1="5.93" y1="11.01" x2="6.35" y2="11.43" width="0.3048" layer="1"/>
+<wire x1="6.35" y1="11.43" x2="6.35" y2="13.97" width="0.3048" layer="1"/>
+<wire x1="6.35" y1="13.97" x2="5.715" y2="14.605" width="0.3048" layer="1"/>
+<wire x1="5.715" y1="14.605" x2="5.175" y2="14.605" width="0.3048" layer="1"/>
+<wire x1="1.735" y1="11.11" x2="1.735" y2="9.21" width="0.3048" layer="1"/>
+<wire x1="5.095" y1="11.01" x2="5.095" y2="10.4925" width="0.3048" layer="1"/>
+<wire x1="5.095" y1="10.4925" x2="4.7625" y2="10.16" width="0.3048" layer="1"/>
+<wire x1="4.7625" y1="10.16" x2="2.685" y2="10.16" width="0.3048" layer="1"/>
+<wire x1="2.685" y1="10.16" x2="1.735" y2="11.11" width="0.3048" layer="1"/>
 </signal>
 <signal name="N$2">
-<wire x1="6.985" y1="5.08" x2="8.255" y2="5.08" width="0.3048" layer="1"/>
-</signal>
-<signal name="N$3">
-<wire x1="7.62" y1="5.715" x2="7.62" y2="4.445" width="0.3048" layer="1"/>
-</signal>
-<signal name="N$5">
-<polygon width="0.3048" layer="1" isolate="0.4064" orphans="yes">
+<polygon width="0.3048" layer="1" isolate="0.3048">
 <vertex x="0" y="0"/>
 <vertex x="-1.27" y="1.27"/>
-<vertex x="-1.27" y="12.7"/>
-<vertex x="8.89" y="12.7"/>
+<vertex x="-1.27" y="16.51"/>
+<vertex x="8.89" y="16.51"/>
 <vertex x="8.89" y="1.27"/>
 <vertex x="7.62" y="0"/>
