File: MicroControl/ST-linkV2/ST link V2_my-2.brd (EAGLE design)
At the start: 57.4 x 22.5 mm, 29 parts, among them IC1 LD117-3.3, Q1 8000 kHz, U1 STM32F103CBT6, X1 STM-SWIMPINS

Commit message: Ещё немного
Parts:
- removed X1: STM-SWIMPINS, Namenlos:1X04/90
- added ESD1, ESD2: ESDA5V3SC5, Namenlos:SOT23-5L
- added R17, R18, R19, R20, R4, R5: 22R, Namenlos:R0805
- added X2: CON-PH12-EDGE, Namenlos:ML12_EDGE_SMD
- C10, C3, C4, C7, C8: device rcl:C0805 -> Namenlos:C0805
- C9: device rcl:C0805 -> Namenlos:R0805
- R1, R11, R12, R14, R15, R16, R2, R3, R6, R7, R8: device rcl:R0805 -> Namenlos:R0805
- R10, R9: device rcl:R0603 -> Namenlos:R0603
- R13: device rcl:R0805 -> Namenlos:C0805
- moved R12 17.9 mm to (9.84, 10.1), turned to 270 degrees
- moved R7 10.5 mm to (19.7, 4.13), turned to 0 degrees
- moved R14 10.2 mm to (14.3, 4.92), turned to 0 degrees
- moved U1 9.26 mm to (16.2, 11.1), turned to 270 degrees
- moved R8 8.67 mm to (32.4, 5.08), turned to 270 degrees
- moved IC1 5.91 mm to (6.03, 18.7)
- moved R1 5.48 mm to (8.89, 3.17), turned to 270 degrees
- moved R3 5.40 mm to (11.1, 3.17)
- moved C1 4.46 mm to (3.17, 12.1)
- moved R2 3.42 mm to (6.67, 3.17), turned to 270 degrees
- moved C4 3.19 mm to (11.4, 20.0)
- moved C2 3.19 mm to (13.7, 19.7)
- moved R11 3.17 mm to (22.9, 8.10), turned to 90 degrees
- moved U$1 2.54 mm to (1.91, 5.40)
- moved C3 0.32 mm to (2.86, 14.3)
Connections:
- new net N$11: R5.2, X2.7
- new net N$13: R17.1, X2.4
- new net N$14: R18.1, X2.8
- new net N$15: R19.1, X2.10
- new net N$16: R20.1, X2.12
- new net N$3: R4.2, X2.3
- net +3V3: now also X2.1, X2.2
- net GND: now also ESD1.2, ESD2.2, X2.5, X2.6
- net SWIM: now also ESD1.3, R4.1
- net SWIM_RST: now also ESD1.1, R5.1
- net T_NRST: now also ESD2.4, R19.2
- net T_SWCLK: now also ESD2.3, R17.2
- net T_SWDIO: now also ESD2.1, R18.2
- net U1_BL_RX_T-SWO: now also ESD2.5, R20.2
- net U1_BL_TX: now also X2.11
Routing:
- net GND: track 151.0 -> 50.3 mm
- net U1_BL_TX: track 77.0 -> 0.00 mm, vias 2 -> 0
- net U1_BL_RX_T-SWO: track 60.7 -> 0.00 mm, vias 1 -> 0
- net +3V3: track 106.2 -> 66.9 mm, vias 4 -> 2
- net SWIM_RST: track 42.5 -> 5.94 mm, vias 2 -> 0
- net T_NRST: track 35.4 -> 0.00 mm, vias 1 -> 0
- net T_SWCLK: track 46.5 -> 17.8 mm, vias 2 -> 1
- net SWIM: track 53.6 -> 27.6 mm, vias 3 -> 2
- net T_SWDIO: track 48.6 -> 30.3 mm
- net N$7: track 15.1 -> 0.00 mm
- net N$6: track 14.4 -> 0.00 mm
- net N$4: track 10.3 -> 0.00 mm
- net BOOT0: track 12.4 -> 3.66 mm
- net !STMRST: track 5.95 -> 0.00 mm
- net N$9: track 5.68 -> 2.11 mm
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- removed copper zone on layer 1, net GND
- removed copper zone on layer 16, net GND
Other:
- outline, holes or cut-outs redrawn

Commit message: Хорошо
Parts:
- added R21: 0, Namenlos:R0805
- moved LED2 17.9 mm to (43.2, 3.49)
- moved R9 16.8 mm to (16.2, 17.8), turned to 180 degrees
- moved R10 15.0 mm to (15.6, 20.3), turned to 90 degrees
- moved R13 14.8 mm to (10.2, 12.1), turned to 270 degrees
- moved C7 14.2 mm to (24.1, 19.1)
- moved C10 13.7 mm to (18.7, 20.0), turned to 180 degrees
- moved C9 13.3 mm to (21.7, 18.9), turned to 270 degrees
- moved Q1 11.2 mm to (30.2, 13.3)
- moved R6 11.1 mm to (23.9, 14.9), turned to 270 degrees
- moved C8 10.8 mm to (32.7, 19.1), turned to 270 degrees
- moved R4 8.90 mm to (42.2, 15.9)
- moved R5 8.58 mm to (42.2, 10.2)
- moved ESD1 8.57 mm to (38.1, 13.0)
- moved ESD2 8.57 mm to (38.1, 6.67)
- moved R17 8.57 mm to (42.2, 15.6)
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Connections:
- new net N$17: R21.1, U1.43
- net N$5: now also R21.2; no longer U1.43
Routing:
- net GND: track 50.3 -> 156.9 mm, vias 0 -> 2
- net T_NRST: track 0.00 -> 51.7 mm, vias 0 -> 1
- net +3V3: track 66.9 -> 112.6 mm, vias 2 -> 5
- net T_SWCLK: track 17.8 -> 62.8 mm
- net U1_BL_TX: track 0.00 -> 43.4 mm, vias 0 -> 2
- net U1_BL_RX_T-SWO: track 0.00 -> 38.2 mm, vias 0 -> 1
- net N$6: track 0.00 -> 26.0 mm
- net SWIM_RST: track 5.94 -> 31.6 mm
- net SWIM: track 27.6 -> 48.4 mm, vias 2 -> 0
- net N$7: track 0.00 -> 18.5 mm
- net T_SWDIO: track 30.3 -> 41.2 mm
- net N$17: track 0.00 -> 9.83 mm
- net N$10: track 0.00 -> 9.52 mm
- net N$4: track 0.00 -> 8.82 mm
- net !STMRST: track 0.00 -> 8.25 mm
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Other:
- board size 57.4 x 22.5 mm -> 48.9 x 22.5 mm

Commit message: _
Parts:
- moved C2 0.32 mm to (13.7, 19.4)
Routing:
- net T_SWCLK: track 62.8 -> 61.8 mm
- net T_NRST: track 51.7 -> 50.8 mm
- net GND: track 156.9 -> 157.5 mm
- added copper zone on layer 1, net GND
- added copper zone on layer 16, net GND
Other:
- outline, holes or cut-outs redrawn
Changed lines of the file:
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@@
 <board>
 <plain>
-<wire x1="0" y1="0" x2="48.875" y2="0" width="0" layer="20"/>
-<wire x1="48.875" y1="0" x2="48.875" y2="22.53" width="0" layer="20"/>
-<wire x1="48.875" y1="22.53" x2="0.2375" y2="22.53" width="0" layer="20"/>
-<wire x1="0.2375" y1="22.53" x2="0" y2="22.2925" width="0" layer="20"/>
-<wire x1="0" y1="22.2925" x2="0" y2="0" width="0" layer="20"/>
+<wire x1="46.875" y1="22.2125" x2="2" y2="22.2125" width="0" layer="20"/>
+<wire x1="2" y1="22.2125" x2="0" y2="20.2125" width="0" layer="20"/>
+<wire x1="0" y1="20.2125" x2="0" y2="1.6825" width="0" layer="20"/>
+<wire x1="0" y1="1.6825" x2="2" y2="-0.3175" width="0" layer="20"/>
+<wire x1="2" y1="-0.3175" x2="46.875" y2="-0.3175" width="0" layer="20"/>
+<wire x1="46.875" y1="-0.3175" x2="48.875" y2="1.6825" width="0" layer="20"/>
+<wire x1="48.875" y1="1.6825" x2="48.875" y2="20.2125" width="0" layer="20"/>
+<wire x1="48.875" y1="20.2125" x2="46.875" y2="22.2125" width="0" layer="20"/>
 <dimension x1="0" y1="0" x2="48.875" y2="0" x3="24.4375" y3="-4.1275" textsize="1.778" layer="47"/>
 <dimension x1="0" y1="22.2925" x2="0" y2="0" x3="-4.7625" y3="11.14625" textsize="1.778" layer="47"/>
@@
 </class>
 </classes>
-<designrules name="EagleDesignRules">
+<designrules name="EagleDesignRules *">
 <description language="de">&lt;b&gt;EAGLE Design Rules&lt;/b&gt;
 &lt;p&gt;
@@
 <param name="mdViaViaSameLayer" value="8mil"/>
 <param name="mnLayersViaInSmd" value="2"/>
-<param name="mdCopperDimension" value="1mm"/>
+<param name="mdCopperDimension" value="0.5mm"/>
 <param name="mdDrill" value="0.2mm"/>
 <param name="mdSmdStop" value="0mil"/>
@@
 <element name="C1" library="rcl" package="SMC_A" value="10u 16V" x="3.175" y="12.065" rot="R180"/>
 <element name="C10" library="Namenlos" package="C0805" value="100n" x="18.7325" y="20.0025" rot="R180"/>
-<element name="C2" library="rcl" package="SMC_A" value="10u 16V" x="13.6525" y="19.685" rot="R90"/>
+<element name="C2" library="rcl" package="SMC_A" value="10u 16V" x="13.6525" y="19.3675" rot="R90"/>
 <element name="C3" library="Namenlos" package="C0805" value="100n" x="2.8575" y="14.2875" rot="R180"/>
 <element name="C4" library="Namenlos" package="C0805" value="100n" x="11.43" y="20.0025" rot="R90"/>
@@
 <wire x1="4.63" y1="4.0975" x2="3.205" y2="4.0975" width="0.254" layer="1"/>
 <wire x1="3.205" y1="4.0975" x2="1.905" y2="5.3975" width="0.254" layer="1"/>
-<wire x1="13.6525" y1="21.185" x2="11.4375" y2="21.185" width="0.254" layer="1"/>
 <wire x1="11.43" y1="21.1775" x2="11.4375" y2="21.185" width="0.254" layer="1"/>
 <wire x1="2.8825" y1="21.0325" x2="3.8875" y2="21.0325" width="0.254" layer="1"/>
@@
 <wire x1="19.9075" y1="20.0025" x2="18.69" y2="21.22" width="0.254" layer="1"/>
 <wire x1="15.5575" y1="21.22" x2="13.6875" y2="21.22" width="0.254" layer="1"/>
-<wire x1="13.6875" y1="21.22" x2="13.6525" y2="21.185" width="0.254" layer="1"/>
+<wire x1="13.6525" y1="20.8675" x2="13.6875" y2="21.22" width="0.254" layer="1"/>
 <wire x1="24.13" y1="21.22" x2="21.74875" y2="21.22" width="0.254" layer="1"/>
 <wire x1="24.13" y1="21.22" x2="32.7025" y2="21.22" width="0.254" layer="1"/>
@@
 <wire x1="37.56" y1="1.5875" x2="37.56" y2="4.35" width="0.254" layer="1"/>
 <wire x1="37.56" y1="4.35" x2="35.2425" y2="6.6675" width="0.254" layer="1"/>
+<wire x1="11.4375" y1="21.185" x2="13.6525" y2="21.185" width="0.4064" layer="1"/>
+<wire x1="13.6525" y1="21.185" x2="13.6525" y2="20.8675" width="0.4064" layer="1"/>
+<polygon width="0.254" layer="1" spacing="0.3048" isolate="0.3048" orphans="yes">
+<vertex x="46.895" y="22.225"/>
+<vertex x="2" y="22.225"/>
+<vertex x="0" y="20.225"/>
+<vertex x="0" y="1.6825"/>
+<vertex x="2" y="-0.3175"/>
+<vertex x="46.895" y="-0.3175"/>
+<vertex x="48.895" y="1.6825"/>
+<vertex x="48.895" y="20.225"/>
+</polygon>
+<polygon width="0.254" layer="16" spacing="0.3048" isolate="0.3048" orphans="yes">
+<vertex x="46.895" y="22.225"/>
+<vertex x="2" y="22.225"/>
+<vertex x="0" y="20.225"/>
+<vertex x="0" y="1.6825"/>
+<vertex x="2" y="-0.3175"/>
+<vertex x="46.895" y="-0.3175"/>
+<vertex x="48.895" y="1.6825"/>
+<vertex x="48.895" y="20.225"/>
+</polygon>
 </signal>
 <signal name="+5V">
@@
 <wire x1="9.1825" y1="18.7325" x2="11.335" y2="18.7325" width="0.254" layer="1"/>
 <wire x1="11.43" y1="18.8275" x2="11.335" y2="18.7325" width="0.254" layer="1"/>
-<wire x1="12.47" y1="18.185" x2="12.0725" y2="18.185" width="0.254" layer="1"/>
-<wire x1="12.0725" y1="18.185" x2="11.43" y2="18.8275" width="0.254" layer="1"/>
 <wire x1="7.62" y1="16.1925" x2="7.62" y2="10.16" width="0.254" layer="16"/>
 <wire x1="7.62" y1="16.1925" x2="8.5725" y2="17.145" width="0.254" layer="16"/>
 <wire x1="11.43" y1="17.145" x2="8.5725" y2="17.145" width="0.254" layer="16"/>
 <via x="11.43" y="17.145" extent="1-16" drill="0.3" shape="octagon"/>
-<wire x1="11.43" y1="17.145" x2="12.47" y2="18.185" width="0.254" layer="1"/>
-<wire x1="12.47" y1="18.185" x2="13.6525" y2="18.185" width="0.254" layer="1"/>
 <via x="14.605" y="0.9525" extent="1-16" drill="0.3" shape="octagon"/>
 <wire x1="9.525" y1="0.9525" x2="14.605" y2="0.9525" width="0.254" layer="16"/>
@@
 <wire x1="20.955" y1="10.72553125" x2="21.655684375" y2="11.426215625" width="0.254" layer="1"/>
 <wire x1="20.955" y1="10.72553125" x2="20.955" y2="10.043478125" width="0.254" layer="1"/>
-<wire x1="13.6525" y1="18.185" x2="13.991740625" y2="17.845759375" width="0.254" layer="1"/>
+<wire x1="13.991740625" y1="17.845759375" x2="13.6525" y2="17.8675" width="0.254" layer="1"/>
 <wire x1="13.991740625" y1="17.845759375" x2="15.331021875" y2="17.845759375" width="0.254" layer="1"/>
 <wire x1="15.331021875" y1="17.845759375" x2="16.748125" y2="16.42865625" width="0.254" layer="1"/>
@@
 <wire x1="42.545" y1="17.4625" x2="43.18" y2="18.0975" width="0.254" layer="1"/>
 <wire x1="43.18" y1="18.0975" x2="44.45" y2="18.0975" width="0.254" layer="1"/>
+<wire x1="11.43" y1="17.145" x2="11.43" y2="18.8275" width="0.254" layer="1"/>
+<wire x1="13.6525" y1="17.8675" x2="12.39" y2="17.8675" width="0.254" layer="1"/>
+<wire x1="12.39" y1="17.8675" x2="11.43" y2="18.8275" width="0.254" layer="1"/>
 </signal>
 <signal name="N$6">
@@
 <contactref element="ESD2" pad="4"/>
 <wire x1="13.932665625" y1="13.54555625" x2="12.7" y2="14.778221875" width="0.254" layer="1"/>
-<wire x1="12.7" y1="14.778221875" x2="12.7" y2="15.24" width="0.254" layer="1"/>
-<via x="12.7" y="15.24" extent="1-16" drill="0.3" shape="octagon"/>
+<wire x1="12.7" y1="14.778221875" x2="12.7" y2="14.605" width="0.254" layer="1"/>
+<via x="12.7" y="14.605" extent="1-16" drill="0.3" shape="octagon"/>
 <wire x1="39.4" y1="7.6175" x2="40.7325" y2="7.6175" width="0.254" layer="16"/>
 <wire x1="40.7325" y1="7.6175" x2="41.0525" y2="7.9375" width="0.254" layer="16"/>
-<wire x1="12.7" y1="15.24" x2="12.7" y2="13.335" width="0.254" layer="16"/>
+<wire x1="12.7" y1="14.605" x2="12.7" y2="13.335" width="0.254" layer="16"/>
 <wire x1="12.7" y1="13.335" x2="7.3025" y2="7.9375" width="0.254" layer="16"/>
 <wire x1="7.3025" y1="7.9375" x2="7.3025" y2="5.3975" width="0.254" layer="16"/>
@@
 <wire x1="8.255" y1="7.9375" x2="6.6675" y2="9.525" width="0.254" layer="1"/>
 <wire x1="6.6675" y1="9.525" x2="6.6675" y2="10.795" width="0.254" layer="1"/>
-<wire x1="8.255" y1="7.9375" x2="8.255" y2="6.985" width="0.254" layer="1"/>
-<via x="8.255" y="6.985" extent="1-16" drill="0.3" shape="octagon"/>
-<wire x1="8.255" y1="6.985" x2="9.525" y2="6.985" width="0.254" layer="16"/>
-<wire x1="9.525" y1="6.985" x2="10.16" y2="7.62" width="0.254" layer="16"/>
-<wire x1="10.16" y1="7.62" x2="36.7975" y2="7.62" width="0.254" layer="16"/>
+<via x="8.255" y="7.9375" extent="1-16" drill="0.3" shape="octagon"/>
+<wire x1="8.255" y1="7.9375" x2="8.5725" y2="7.62" width="0.254" layer="16"/>
+<wire x1="8.5725" y1="7.62" x2="36.7975" y2="7.62" width="0.254" layer="16"/>
 <wire x1="36.7975" y1="7.62" x2="36.8" y2="7.6175" width="0.254" layer="16"/>
 <wire x1="40.005" y1="15.5575" x2="41.0525" y2="15.5575" width="0.254" layer="16"/>
@@
 <wire x1="14.12875" y1="4.445" x2="16.51" y2="4.445" width="0.254" layer="16"/>
 <via x="16.51" y="4.445" extent="1-16" drill="0.3" shape="octagon"/>
-<wire x1="19.05" y1="1.5875" x2="16.51" y2="4.1275" width="0.254" layer="1"/>
+<wire x1="20.32" y1="0.3175" x2="16.51" y2="4.1275" width="0.254" layer="1"/>
 <wire x1="16.51" y1="4.1275" x2="16.51" y2="4.445" width="0.254" layer="1"/>
 <wire x1="44.93" y1="1.115" x2="44.93" y2="1.5875" width="0.254" layer="1"/>
 <wire x1="44.93" y1="1.115" x2="44.1325" y2="0.3175" width="0.254" layer="1"/>
-<wire x1="44.1325" y1="0.3175" x2="36.83" y2="0.3175" width="0.254" layer="1"/>
-<wire x1="36.83" y1="0.3175" x2="35.56" y2="1.5875" width="0.254" layer="1"/>
-<wire x1="35.56" y1="1.5875" x2="19.05" y2="1.5875" width="0.254" layer="1"/>
+<wire x1="44.1325" y1="0.3175" x2="20.32" y2="0.3175" width="0.254" layer="1"/>
 <wire x1="44.93" y1="1.5875" x2="44.93" y2="3.4925" width="0.254" layer="1"/>
 <wire x1="44.93" y1="3.4925" x2="45.085" y2="3.4925" width="0.254" layer="1"/>

Commit message: _
Parts:
- moved C8 9.88 mm to (25.7, 12.1), turned to 90 degrees
- moved C7 2.03 mm to (25.7, 17.8)
- moved R3 2.03 mm to (13.3, 2.54), turned to 270 degrees
- moved C10 0.71 mm to (19.1, 19.4)
- moved ESD1 0.32 mm to (37.8, 13.0)
- moved ESD2 0.32 mm to (37.8, 6.67)
- moved LED1 0.32 mm to (42.9, 1.59)
- moved LED2 0.32 mm to (42.9, 3.49)
- moved R15 0.32 mm to (43.2, 13.0)
- moved R16 0.32 mm to (38.4, 1.59)
- moved R17 0.32 mm to (41.9, 15.6)
- moved R18 0.32 mm to (41.9, 10.5)
- moved R19 0.32 mm to (41.9, 7.94)
- moved R20 0.32 mm to (41.9, 5.40)
- moved R4 0.32 mm to (41.9, 15.9)
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Routing:
- net GND: track 157.5 -> 134.8 mm
- net +3V3: track 112.8 -> 126.8 mm
- net N$6: track 26.0 -> 16.7 mm
- net N$7: track 18.5 -> 13.8 mm
- net USB_D+: track 12.3 -> 13.4 mm
- net T_SWCLK: track 61.8 -> 61.1 mm
- net U1_BL_TX: track 43.4 -> 42.9 mm
Other:
- board size 48.9 x 22.5 mm -> 48.9 x 22.8 mm
