File: 3DPrinter/1280.sch (EAGLE design)
At the start: 20 parts, among them IC1 ATMEGA1280-16AU, IC2 7805DT, IC3 CP2102, Q1 16 MHz, X1 PN61729-S

Commit message: Some 1280
Parts:
- added IC4: X, Namenlos:STEP-DRV
- added IC5: Y, Namenlos:STEP-DRV
- added IC6: Z, Namenlos:STEP-DRV
- added IC7: E0, Namenlos:STEP-DRV
- added IC8: E1, Namenlos:STEP-DRV
- added J2, J3, J4, J5: 22-27-2041-04, con-molex:22-27-2041-04
- added JP2: (no value), pinhead:PINHD-1X2
- added SV1, SV2: (no value), con-harting-ml:ML10
- added VT1, VT2, VT3, VT4: (no value), Namenlos:FET-NPF-6X5
- added X2, X3: CON-5.08-03P, Namenlos:CON-5.08-03P
- added X4: CON-7.62-02P, Namenlos:CON-7.62-02P
- J1: value (none) -> 22-27-2041-04; device con-jack:DCJ0303 -> con-molex:22-27-2041-04
Connections:
- net N$5 renamed AREF
- new net E0-: VT1.D, X2-2.KL
- new net E1-: VT2.D, X3-1.KL
- new net FAN: IC1.(OC0B)PG5, VT4.G
- new net FAN-: JP2.2, VT4.D
- new net HB-: VT3.D, X3-3.KL
- new net N$10: IC7.!RST, IC7.!SLEEP
- new net N$11: IC6.!RST, IC6.!SLEEP
- new net N$12: IC7.2B, J4-1.S
- new net N$13: IC7.2A, J4-2.S
- new net N$14: IC8.!RST, IC8.!SLEEP
- new net N$15: IC7.1A, J4-3.S
- new net N$16: IC7.1B, J4-4.S
- new net N$17: IC6.2B, J3-1.S
- new net N$18: IC6.2A, J3-2.S
- new net N$19: IC6.1A, J3-3.S
- new net N$2: IC3.D+, X1.3
- new net N$20: IC6.1B, J3-4.S
- new net N$21: IC5.2B, J2-1.S
- new net N$22: IC5.2A, J2-2.S
- new net N$23: IC5.1A, J2-3.S
- new net N$24: IC5.1B, J2-4.S
- new net N$25: IC4.2B, J1-1.S
- new net N$26: IC4.2A, J1-2.S
- new net N$27: IC4.1A, J1-3.S
- new net N$28: IC4.1B, J1-4.S
- new net N$3: IC8.2B, J5-1.S
- new net N$5: IC8.2A, J5-2.S
- new net N$6: IC8.1A, J5-3.S
- new net N$7: IC4.!RST, IC4.!SLEEP
- new net N$8: IC5.!RST, IC5.!SLEEP
- new net N$9: IC8.1B, J5-4.S
- net +5V: now also IC4.VDD, IC5.VDD, IC6.VDD, IC7.VDD, IC8.VDD, X1.1; no longer IC3.D+, X1.3
- net E0-DIR: now also IC7.DIR
- net E0-EN: now also IC7.!EN
- net E0-PWM: now also VT1.G
- net E0-STEP: now also IC7.STEP
- net E1-DIR: now also IC8.DIR
- net E1-EN: now also IC8.!EN
- net E1-PWM: now also VT2.G
- net E1-STEP: now also IC8.STEP
- net EX1-1: now also SV1.1
- net EX1-10: now also SV1.10
- net EX1-2: now also SV1.2
- net EX1-3: now also SV1.3
- net EX1-4: now also SV1.4
- net EX1-5: now also SV1.5
- net EX1-6: now also SV1.6
- net EX1-7: now also SV1.7
- net EX1-8: now also SV1.8
- net EX2-1: now also SV2.1
- net EX2-2: now also SV2.2
- net EX2-3: now also SV2.3
- net EX2-4: now also SV2.4
- net EX2-5: now also SV2.5
- net EX2-6: now also SV2.6
- net EX2-8: now also SV2.8
- net GND: now also IC4.GND, IC4.MGND, IC5.GND, IC5.MGND, IC6.GND, IC6.MGND, IC7.GND, IC7.MGND, IC8.GND, IC8.MGND, VT1.S, VT2.S, VT3.S, VT4.S, X42.KL; no longer J1.1
- net HB-PWM: now also VT3.G
- net V-IN: now also IC4.VMOT, IC5.VMOT, IC6.VMOT, IC7.VMOT, IC8.VMOT, JP2.1, X2-1.KL, X2-3.KL, X3-2.KL, X41.KL; no longer J1.3
- net X-DIR: now also IC4.DIR
- net X-EN: now also IC4.!EN
- net X-STEP: now also IC4.STEP
- net Y-DIR: now also IC5.DIR
- net Y-EN: now also IC5.!EN
- net Y-STEP: now also IC5.STEP
- net Z-DIR: now also IC6.DIR
- net Z-EN: now also IC6.!EN
- net Z-STEP: now also IC6.STEP

Commit message: полная ардуйня
Parts:
- added C12, C13, C14: 10u, Namenlos:CAP_1210
- added C15, C16, C17: 100n, Namenlos:CAP_0805
- added JP3, JP4: (no value), pinhead:PINHD-2X3
- added R2, R3, R4: 4k7, Namenlos:R_0805
- added R5, R6, R7: 12k, Namenlos:R_0805
Connections:
- net !RST: now also IC3.DTR
- net +5V: now also R2.2, R3.2, R4.2, R5.2, R6.2, R7.2
- net FAN: now also IC1.PH4(OC4B); no longer IC1.(OC0B)PG5
- net GND: now also C12.2, C13.2, C14.2, C15.2, C16.2, C17.2, JP3.2, JP3.4, JP3.6, JP4.2, JP4.4, JP4.6
- net THERM-0: now also C12.1, JP3.1, R2.1
- net THERM-1: now also C13.1, JP3.3, R3.1
- net THERM-2: now also C14.1, JP3.5, R4.1
- net X-MAX: now also C17.1, JP4.1, R7.1
- net Y-MAX: now also C16.1, JP4.3, R6.1
- net Z-MIN: now also C15.1, JP4.5, R5.1

Commit message: _
Connections:
- net +5V: now also SV2.7
- net GND: now also SV1.9
Changed lines of the file:
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@@
 <part name="GND26" library="supply1" deviceset="GND" device=""/>
 <part name="GND27" library="supply1" deviceset="GND" device=""/>
+<part name="GND28" library="supply1" deviceset="GND" device=""/>
+<part name="P+16" library="supply1" deviceset="+5V" device=""/>
 </parts>
 <sheets>
@@
 <instance part="GND26" gate="1" x="180.34" y="-48.26"/>
 <instance part="GND27" gate="1" x="198.12" y="-17.78"/>
+<instance part="GND28" gate="1" x="134.62" y="68.58"/>
+<instance part="P+16" gate="1" x="132.08" y="40.64" rot="R90"/>
 </instances>
 <busses>
@@
 <wire x1="134.62" y1="45.72" x2="147.32" y2="45.72" width="0.1524" layer="91"/>
 <pinref part="SV2" gate="G$1" pin="3"/>
-<label x="137.16" y="45.72" size="1.778" layer="95" rot="R180"/>
+<label x="137.16" y="48.26" size="1.778" layer="95" rot="R180"/>
 </segment>
 </net>
@@
 <wire x1="134.62" y1="43.18" x2="147.32" y2="43.18" width="0.1524" layer="91"/>
 <pinref part="SV2" gate="G$1" pin="5"/>
-<label x="137.16" y="43.18" size="1.778" layer="95" rot="R180"/>
+<label x="137.16" y="45.72" size="1.778" layer="95" rot="R180"/>
 </segment>
 </net>
@@
 <wire x1="162.56" y1="40.64" x2="175.26" y2="40.64" width="0.1524" layer="91"/>
 <pinref part="SV2" gate="G$1" pin="8"/>
-<label x="175.26" y="40.64" size="1.778" layer="95" rot="R180"/>
+<label x="175.26" y="43.18" size="1.778" layer="95" rot="R180"/>
 </segment>
 </net>
@@
 <wire x1="134.62" y1="48.26" x2="147.32" y2="48.26" width="0.1524" layer="91"/>
 <pinref part="SV2" gate="G$1" pin="1"/>
-<label x="137.16" y="48.26" size="1.778" layer="95" rot="R180"/>
+<label x="137.16" y="50.8" size="1.778" layer="95" rot="R180"/>
 </segment>
 </net>
@@
 <wire x1="162.56" y1="48.26" x2="175.26" y2="48.26" width="0.1524" layer="91"/>
 <pinref part="SV2" gate="G$1" pin="2"/>
-<label x="175.26" y="48.26" size="1.778" layer="95" rot="R180"/>
+<label x="175.26" y="50.8" size="1.778" layer="95" rot="R180"/>
 </segment>
 </net>
@@
 <wire x1="162.56" y1="45.72" x2="175.26" y2="45.72" width="0.1524" layer="91"/>
 <pinref part="SV2" gate="G$1" pin="4"/>
-<label x="175.26" y="45.72" size="1.778" layer="95" rot="R180"/>
+<label x="175.26" y="48.26" size="1.778" layer="95" rot="R180"/>
 </segment>
 </net>
@@
 <wire x1="162.56" y1="43.18" x2="175.26" y2="43.18" width="0.1524" layer="91"/>
 <pinref part="SV2" gate="G$1" pin="6"/>
-<label x="175.26" y="43.18" size="1.778" layer="95" rot="R180"/>
+<label x="175.26" y="45.72" size="1.778" layer="95" rot="R180"/>
 </segment>
 </net>
@@
 <junction x="198.12" y="-7.62"/>
 </segment>
+<segment>
+<pinref part="SV1" gate="G$1" pin="9"/>
+<wire x1="147.32" y1="73.66" x2="134.62" y2="73.66" width="0.1524" layer="91"/>
+<wire x1="134.62" y1="73.66" x2="134.62" y2="71.12" width="0.1524" layer="91"/>
+<pinref part="GND28" gate="1" pin="GND"/>
+</segment>
 </net>
 <net name="XTAL1" class="0">
@@
 <pinref part="P+15" gate="1" pin="+5V"/>
 </segment>
-</net>
+<segment>
+<pinref part="SV2" gate="G$1" pin="7"/>
+<wire x1="147.32" y1="40.64" x2="134.62" y2="40.64" width="0.1524" layer="91"/>
+<pinref part="P+16" gate="1" pin="+5V"/>
+</segment>
+</net>

Commit message: Done
Parts:
- removed J1, J2, J3, J4, J5: 22-27-2041-04, con-molex:22-27-2041-04
- removed JP2: (no value), pinhead:PINHD-1X2
- removed JP3, JP4: (no value), pinhead:PINHD-2X3
- added C18, C19, C20: 100n, Namenlos:CAP_0805
- added R10, R8, R9: 12k, Namenlos:R_0805
- added S1, S2, S3, S4, S5: (no value), Namenlos:SW-DIP03S
- added X10, X17, X18, X19: (no value), Namenlos:CON-CP-02
- added X11, X12, X13, X14, X15, X16: CON-CP-03, Namenlos:CON-CP-03
- added X5, X6, X7, X8, X9: CON-CP-04, Namenlos:CON-CP-04
- JP1: value AVR-ISP-6HORZ -> AVR-ISP-6VERT; device avr-7:AVR-ISP-6HORZ -> avr-7:AVR-ISP-6VERT
Connections:
- new net N$29: IC4.MS1, S1.1
- new net N$30: IC4.MS2, S1.2
- new net N$31: IC4.MS3, S1.3
- new net N$32: IC5.MS1, S2.1
- new net N$33: IC5.MS2, S2.2
- new net N$34: IC5.MS3, S2.3
- new net N$35: IC6.MS1, S3.1
- new net N$36: IC6.MS2, S3.2
- new net N$37: IC6.MS3, S3.3
- new net N$38: IC7.MS1, S4.1
- new net N$39: IC7.MS2, S4.2
- new net N$40: IC7.MS3, S4.3
- new net N$41: IC8.MS1, S5.1
- new net N$42: IC8.MS2, S5.2
- new net N$43: IC8.MS3, S5.3
- net +5V: now also R10.2, R8.2, R9.2, S1.4, S1.5, S1.6, S2.4, S2.5, S2.6, S3.4, S3.5, S3.6, S4.4, S4.5, S4.6, S5.4, S5.5, S5.6, X11.1, X12.1, X13.1, X14.1, X15.1, X16.1
- net E1-PWM: now also VT3.G; no longer VT2.G
- net FAN-: now also X10.2; no longer JP2.2
- net GND: now also C18.2, C19.2, C20.2, X11.3, X12.3, X13.3, X14.3, X15.3, X16.3, X17.2, X18.2, X19.2; no longer JP3.2, JP3.4, JP3.6, JP4.2, JP4.4, JP4.6
- net HB-PWM: now also VT2.G; no longer VT3.G
- net N$12: now also IC5.2B, X6.1; no longer IC7.2B, J4-1.S
- net N$13: now also IC5.2A, X6.2; no longer IC7.2A, J4-2.S
- net N$15: now also IC5.1A, X6.3; no longer IC7.1A, J4-3.S
- net N$16: now also IC5.1B, X6.4; no longer IC7.1B, J4-4.S
- net N$17: now also X7.1; no longer J3-1.S
- net N$18: now also X7.2; no longer J3-2.S
- net N$19: now also X7.3; no longer J3-3.S
- net N$20: now also X7.4; no longer J3-4.S
- net N$21: now also IC7.2B, X8.1; no longer IC5.2B, J2-1.S
- net N$22: now also IC7.2A, X8.2; no longer IC5.2A, J2-2.S
- net N$23: now also IC7.1A, X8.3; no longer IC5.1A, J2-3.S
- net N$24: now also IC7.1B, X8.4; no longer IC5.1B, J2-4.S
- net N$25: now also IC8.2B, X9.1; no longer IC4.2B, J1-1.S
- net N$26: now also IC8.2A, X9.2; no longer IC4.2A, J1-2.S
- net N$27: now also IC8.1A, X9.3; no longer IC4.1A, J1-3.S
- net N$28: now also IC8.1B, X9.4; no longer IC4.1B, J1-4.S
- net N$3: now also IC4.2B, X5.1; no longer IC8.2B, J5-1.S
- net N$5: now also IC4.2A, X5.2; no longer IC8.2A, J5-2.S
- net N$6: now also IC4.1A, X5.3; no longer IC8.1A, J5-3.S
- net N$9: now also IC4.1B, X5.4; no longer IC8.1B, J5-4.S
- net THERM-0: now also X17.1; no longer JP3.1
- net THERM-1: now also X18.1; no longer JP3.3
- net THERM-2: now also X19.1; no longer JP3.5
- net V-IN: now also X10.1; no longer JP2.1
- net X-MAX: now also C19.1, R9.1, X15.2; no longer C17.1, JP4.1, R7.1
- net X-MIN: now also C20.1, R10.1, X16.2
- net Y-MAX: now also C17.1, R7.1, X13.2; no longer C16.1, JP4.3, R6.1
- net Y-MIN: now also C18.1, R8.1, X14.2
- net Z-MAX: now also C15.1, R5.1, X11.2
- net Z-MIN: now also C16.1, R6.1, X12.2; no longer C15.1, JP4.5, R5.1

Commit message: _
Parts:
- added R11, R12, R13, R14: (no value), Namenlos:R_0805
- added X20, X21: (no value), Namenlos:CON-CP-02
- JP1: device avr-7:AVR-ISP-6VERT -> pinhead:PINHD-2X3
Connections:
- new net N$44: R11.1, VT1.G
- new net N$45: R13.1, VT2.G
- new net N$46: R14.1, VT4.G
- new net N$47: R12.1, VT3.G
- net E0-PWM: now also R11.2; no longer VT1.G
- net E1-PWM: now also R12.2; no longer VT3.G
- net FAN: now also R14.2; no longer VT4.G
- net GND: now also X20.2, X21.2
- net HB-PWM: now also R13.2; no longer VT2.G
- net V-IN: now also X20.1, X21.1
Other:
- note added: "MISO"
- note added: "MOSI"
- note added: "RST"
- note added: "SCK"
Changed lines of the file:
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@@
 <part name="P+1" library="supply1" deviceset="+5V" device=""/>
 <part name="R1" library="Namenlos" deviceset="R_" device="0805" value="20k"/>
-<part name="JP1" library="avr-7" deviceset="AVR-ISP-6" device="VERT" value="AVR-ISP-6VERT"/>
+<part name="JP1" library="pinhead" deviceset="PINHD-2X3" device="" value="AVR-ISP-6VERT"/>
 <part name="P+2" library="supply1" deviceset="+5V" device=""/>
 <part name="GND3" library="supply1" deviceset="GND" device=""/>
@@
 <part name="S5" library="Namenlos" deviceset="SW-DIP03S" device=""/>
 <part name="P+26" library="supply1" deviceset="+5V" device=""/>
+<part name="R11" library="Namenlos" deviceset="R_" device="0805"/>
+<part name="R12" library="Namenlos" deviceset="R_" device="0805"/>
+<part name="R13" library="Namenlos" deviceset="R_" device="0805"/>
+<part name="R14" library="Namenlos" deviceset="R_" device="0805"/>
+<part name="X20" library="Namenlos" deviceset="CON-CP-02" device=""/>
+<part name="X21" library="Namenlos" deviceset="CON-CP-02" device=""/>
+<part name="GND36" library="supply1" deviceset="GND" device=""/>
 </parts>
 <sheets>
@@
 <instance part="X3" gate="-3" x="30.48" y="35.56" rot="MR90"/>
 <instance part="X10" gate="X$1" x="66.04" y="35.56" rot="MR0"/>
+<instance part="R11" gate="G$1" x="25.4" y="71.12" rot="R180"/>
+<instance part="R12" gate="G$1" x="25.4" y="20.32" rot="R180"/>
+<instance part="R13" gate="G$1" x="66.04" y="71.12" rot="R180"/>
+<instance part="R14" gate="G$1" x="66.04" y="20.32" rot="R180"/>
+<instance part="X20" gate="X$1" x="96.52" y="35.56" rot="MR0"/>
+<instance part="X21" gate="X$1" x="111.76" y="35.56"/>
+<instance part="GND36" gate="1" x="104.14" y="30.48"/>
 </instances>
 <busses>
@@
 <net name="E0-PWM" class="0">
 <segment>
-<pinref part="VT1" gate="G$1" pin="G"/>
-<wire x1="30.48" y1="71.12" x2="17.78" y2="71.12" width="0.1524" layer="91"/>
-<label x="17.78" y="71.12" size="1.778" layer="95"/>
+<label x="7.62" y="71.12" size="1.778" layer="95"/>
+<pinref part="R11" gate="G$1" pin="2"/>
+<wire x1="20.32" y1="71.12" x2="7.62" y2="71.12" width="0.1524" layer="91"/>
 </segment>
 </net>
 <net name="E1-PWM" class="0">
 <segment>
-<wire x1="27.94" y1="20.32" x2="17.78" y2="20.32" width="0.1524" layer="91"/>
-<pinref part="VT3" gate="G$1" pin="G"/>
-<wire x1="27.94" y1="20.32" x2="30.48" y2="20.32" width="0.1524" layer="91"/>
-<label x="20.32" y="20.32" size="1.778" layer="95"/>
+<wire x1="20.32" y1="20.32" x2="7.62" y2="20.32" width="0.1524" layer="91"/>
+<label x="7.62" y="20.32" size="1.778" layer="95"/>
+<pinref part="R12" gate="G$1" pin="2"/>
 </segment>
 </net>
 <net name="HB-PWM" class="0">
 <segment>
-<wire x1="68.58" y1="71.12" x2="55.88" y2="71.12" width="0.1524" layer="91"/>
-<label x="58.42" y="71.12" size="1.778" layer="95"/>
-<pinref part="VT2" gate="G$1" pin="G"/>
-<wire x1="68.58" y1="71.12" x2="71.12" y2="71.12" width="0.1524" layer="91"/>
+<label x="48.26" y="71.12" size="1.778" layer="95"/>
+<wire x1="60.96" y1="71.12" x2="48.26" y2="71.12" width="0.1524" layer="91"/>
+<pinref part="R13" gate="G$1" pin="2"/>
 </segment>
 </net>
 <net name="FAN" class="0">
 <segment>
-<pinref part="VT4" gate="G$1" pin="G"/>
-<wire x1="71.12" y1="20.32" x2="58.42" y2="20.32" width="0.1524" layer="91"/>
-<label x="58.42" y="20.32" size="1.778" layer="95"/>
+<label x="50.8" y="20.32" size="1.778" layer="95"/>
+<pinref part="R14" gate="G$1" pin="2"/>
+<wire x1="60.96" y1="20.32" x2="50.8" y2="20.32" width="0.1524" layer="91"/>
 </segment>
 </net>
@@
 <pinref part="VT1" gate="G$1" pin="S"/>
 <pinref part="GND9" gate="1" pin="GND"/>
+</segment>
+<segment>
+<pinref part="GND36" gate="1" pin="GND"/>
+<pinref part="X20" gate="X$1" pin="2"/>
+<wire x1="104.14" y1="33.02" x2="104.14" y2="35.56" width="0.1524" layer="91"/>
+<wire x1="104.14" y1="35.56" x2="99.06" y2="35.56" width="0.1524" layer="91"/>
+<pinref part="X21" gate="X$1" pin="2"/>
+<wire x1="109.22" y1="35.56" x2="104.14" y2="35.56" width="0.1524" layer="91"/>
+<junction x="104.14" y="35.56"/>
 </segment>
 </net>
@@
 <pinref part="X10" gate="X$1" pin="1"/>
 </segment>
+<segment>
+<wire x1="99.06" y1="38.1" x2="104.14" y2="38.1" width="0.1524" layer="91"/>
+<pinref part="X20" gate="X$1" pin="1"/>
+<pinref part="X21" gate="X$1" pin="1"/>
+<wire x1="104.14" y1="38.1" x2="109.22" y2="38.1" width="0.1524" layer="91"/>
+<wire x1="104.14" y1="38.1" x2="104.14" y2="53.34" width="0.1524" layer="91"/>
+<junction x="104.14" y="38.1"/>
+<label x="104.14" y="50.8" size="1.778" layer="95"/>
+</segment>
 </net>
 <net name="FAN-" class="0">
@@
 </segment>
 </net>
+<net name="N$44" class="0">
+<segment>
+<pinref part="VT1" gate="G$1" pin="G"/>
+<pinref part="R11" gate="G$1" pin="1"/>
+</segment>
+</net>
+<net name="N$45" class="0">
+<segment>
+<pinref part="VT2" gate="G$1" pin="G"/>
+<pinref part="R13" gate="G$1" pin="1"/>
+</segment>
+</net>
+<net name="N$46" class="0">
+<segment>
+<pinref part="VT4" gate="G$1" pin="G"/>
+<pinref part="R14" gate="G$1" pin="1"/>
+</segment>
+</net>
+<net name="N$47" class="0">
+<segment>
+<pinref part="VT3" gate="G$1" pin="G"/>
+<pinref part="R12" gate="G$1" pin="1"/>
+</segment>
+</net>
 </nets>
 </sheet>
 <sheet>
 <plain>
+<text x="40.64" y="165.1" size="1.778" layer="97">MISO</text>
+<text x="40.64" y="162.56" size="1.778" layer="97">SCK</text>
+<text x="40.64" y="160.02" size="1.778" layer="97">RST</text>
+<text x="60.96" y="162.56" size="1.778" layer="97">MOSI</text>
 </plain>
 <instances>
@@
 <instance part="P+1" gate="1" x="-22.86" y="127"/>
 <instance part="R1" gate="G$1" x="-15.24" y="114.3"/>
-<instance part="JP1" gate="G$1" x="53.34" y="162.56"/>
+<instance part="JP1" gate="A" x="53.34" y="162.56"/>
 <instance part="P+2" gate="1" x="66.04" y="170.18"/>
 <instance part="GND3" gate="1" x="66.04" y="154.94"/>
@@
 <segment>
 <wire x1="58.42" y1="162.56" x2="71.12" y2="162.56" width="0.1524" layer="91"/>
-<pinref part="JP1" gate="G$1" pin="4"/>
+<pinref part="JP1" gate="A" pin="4"/>
 </segment>
 <segment>
@@
 </segment>
 <segment>
-<wire x1="35.56" y1="162.56" x2="48.26" y2="162.56" width="0.1524" layer="91"/>
-<pinref part="JP1" gate="G$1" pin="3"/>
+<wire x1="35.56" y1="162.56" x2="50.8" y2="162.56" width="0.1524" layer="91"/>
+<pinref part="JP1" gate="A" pin="3"/>
 </segment>
 <segment>
@@
 </segment>
 <segment>
-<wire x1="35.56" y1="165.1" x2="48.26" y2="165.1" width="0.1524" layer="91"/>
-<pinref part="JP1" gate="G$1" pin="1"/>
+<wire x1="35.56" y1="165.1" x2="50.8" y2="165.1" width="0.1524" layer="91"/>
+<pinref part="JP1" gate="A" pin="1"/>
 </segment>
 <segment>
@@
 <wire x1="66.04" y1="157.48" x2="66.04" y2="160.02" width="0.1524" layer="91"/>
 <wire x1="66.04" y1="160.02" x2="58.42" y2="160.02" width="0.1524" layer="91"/>
-<pinref part="JP1" gate="G$1" pin="6"/>
+<pinref part="JP1" gate="A" pin="6"/>
 </segment>
 <segment>
@@
 <wire x1="66.04" y1="167.64" x2="66.04" y2="165.1" width="0.1524" layer="91"/>
 <wire x1="66.04" y1="165.1" x2="58.42" y2="165.1" width="0.1524" layer="91"/>
-<pinref part="JP1" gate="G$1" pin="2"/>
+<pinref part="JP1" gate="A" pin="2"/>
 </segment>
 <segment>
@@
 </segment>
 <segment>
-<wire x1="35.56" y1="160.02" x2="48.26" y2="160.02" width="0.1524" layer="91"/>
-<pinref part="JP1" gate="G$1" pin="5"/>
-</segment>
-<segment>
+<wire x1="35.56" y1="160.02" x2="50.8" y2="160.02" width="0.1524" layer="91"/>
+<pinref part="JP1" gate="A" pin="5"/>
+</segment>
+<segment>

Commit message: Some Tweaks
Parts:
- added C21, C22, C23, C24, C25: (no value), Namenlos:CAP-POL_D6
Connections:
- net GND: now also C21.-, C22.-, C23.-, C24.-, C25.-
- net V-IN: now also C21.+, C22.+, C23.+, C24.+, C25.+
Changed lines of the file:
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@@
 <part name="X21" library="Namenlos" deviceset="CON-CP-02" device=""/>
 <part name="GND36" library="supply1" deviceset="GND" device=""/>
+<part name="C21" library="Namenlos" deviceset="CAP-POL_" device="D6"/>
+<part name="C22" library="Namenlos" deviceset="CAP-POL_" device="D6"/>
+<part name="C23" library="Namenlos" deviceset="CAP-POL_" device="D6"/>
+<part name="C24" library="Namenlos" deviceset="CAP-POL_" device="D6"/>
+<part name="C25" library="Namenlos" deviceset="CAP-POL_" device="D6"/>
+<part name="GND37" library="supply1" deviceset="GND" device=""/>
+<part name="GND38" library="supply1" deviceset="GND" device=""/>
+<part name="GND39" library="supply1" deviceset="GND" device=""/>
+<part name="GND40" library="supply1" deviceset="GND" device=""/>
+<part name="GND41" library="supply1" deviceset="GND" device=""/>
 </parts>
 <sheets>
@@
 <instance part="S5" gate="1" x="12.7" y="-58.42" rot="MR270"/>
 <instance part="P+26" gate="1" x="2.54" y="81.28"/>
+<instance part="C21" gate="C$1" x="83.82" y="68.58" rot="R90"/>
+<instance part="C22" gate="C$1" x="83.82" y="38.1" rot="R90"/>
+<instance part="C23" gate="C$1" x="83.82" y="7.62" rot="R90"/>
+<instance part="C24" gate="C$1" x="83.82" y="-22.86" rot="R90"/>
+<instance part="C25" gate="C$1" x="83.82" y="-53.34" rot="R90"/>
+<instance part="GND37" gate="1" x="91.44" y="-53.34" rot="R90"/>
+<instance part="GND38" gate="1" x="91.44" y="-22.86" rot="R90"/>
+<instance part="GND39" gate="1" x="91.44" y="7.62" rot="R90"/>
+<instance part="GND40" gate="1" x="91.44" y="38.1" rot="R90"/>
+<instance part="GND41" gate="1" x="91.44" y="68.58" rot="R90"/>
 </instances>
 <busses>
@@
 <pinref part="GND19" gate="1" pin="GND"/>
 </segment>
+<segment>
+<pinref part="C25" gate="C$1" pin="-"/>
+<pinref part="GND37" gate="1" pin="GND"/>
+</segment>
+<segment>
+<pinref part="C24" gate="C$1" pin="-"/>
+<pinref part="GND38" gate="1" pin="GND"/>
+</segment>
+<segment>
+<pinref part="C23" gate="C$1" pin="-"/>
+<pinref part="GND39" gate="1" pin="GND"/>
+</segment>
+<segment>
+<pinref part="C22" gate="C$1" pin="-"/>
+<pinref part="GND40" gate="1" pin="GND"/>
+</segment>
+<segment>
+<pinref part="C21" gate="C$1" pin="-"/>
+<pinref part="GND41" gate="1" pin="GND"/>
+</segment>
 </net>
 <net name="V-IN" class="0">
@@
 <wire x1="73.66" y1="-53.34" x2="81.28" y2="-53.34" width="0.1524" layer="91"/>
 <label x="76.2" y="-53.34" size="1.778" layer="95"/>
+<pinref part="C25" gate="C$1" pin="+"/>
 </segment>
 <segment>
@@
 <wire x1="73.66" y1="-22.86" x2="81.28" y2="-22.86" width="0.1524" layer="91"/>
 <label x="76.2" y="-22.86" size="1.778" layer="95"/>
+<pinref part="C24" gate="C$1" pin="+"/>
 </segment>
 <segment>
@@
 <wire x1="73.66" y1="7.62" x2="81.28" y2="7.62" width="0.1524" layer="91"/>
 <label x="76.2" y="7.62" size="1.778" layer="95"/>
+<pinref part="C23" gate="C$1" pin="+"/>
 </segment>
 <segment>
@@
 <wire x1="73.66" y1="38.1" x2="81.28" y2="38.1" width="0.1524" layer="91"/>
 <label x="76.2" y="38.1" size="1.778" layer="95"/>
+<pinref part="C22" gate="C$1" pin="+"/>
 </segment>
 <segment>
@@
 <wire x1="73.66" y1="68.58" x2="81.28" y2="68.58" width="0.1524" layer="91"/>
 <label x="76.2" y="68.58" size="1.778" layer="95"/>
-</segment>
-</net>
+<pinref part="C21" gate="C$1" pin="+"/>
+</segment>
+</net>
