File: 3DPrinter/1280 V2 SMPS.sch (EAGLE design)
At the start: 84 parts, among them IC1 ATMEGA1280-16AU, IC10 TS520533, IC2 7805DT, IC3 CP2102, IC4 X, IC5 Y, IC6 Z, IC7 E0, IC8 E1, IC9 4050D, Q1 16 MHz, X1 USBBF, X2 CON-5.08-03P, X3 CON-5.08-03P, X4 CON-7.62-02P

Commit message: SMPS
Parts:
- removed IC2: 7805DT, linear:7805DT
- added D1: MBRA130LT3G, Namenlos:DIODE-SH_SMA
- added L2: SCDS127T-221M-N, inductors:DR127
- added R18, R19, R20: 1R, Namenlos:R_0805
- added R21: 3K9, Namenlos:R_0805
- added R22: 1K3, Namenlos:R_0805
- added U$1: MC33063/MC34063D, adafruit:MC33063/MC34063D
- C4: value 100n -> 470p
Connections:
- new net N$47: C10.1, C8.+, R18.1, R19.1, R20.1, U$1.VCC, X41.KL
- new net N$55: R18.2, R19.2, R20.2, U$1.DC, U$1.IPK, U$1.SWC
- new net N$56: D1.C, L2.1, U$1.SWE
- new net N$57: C4.1, U$1.TC
- new net N$59: R21.1, R22.2, U$1.COMP
- net +5V: now also L2.2, R21.2; no longer C4.1, IC2.VO
- net GND: now also D1.A, R22.1, U$1.GND; no longer IC2.GND
- net V-IN: no longer C10.1, C8.+, IC2.VI, X41.KL
Other:
- moved on the sheet: C10, C11, C15, C4, C8, C9, IC10, X41, X42

Commit message: SMPS
Parts:
- removed C10: 100n, Namenlos:CAP_0805
- removed C8: (no value), Namenlos:CAP-POL_D8
- L2: device inductors:DR127 -> Namenlos:INDUCTOR0705
Connections:
- removed net N$47: C10.1, C8.+, R18.1, R19.1, R20.1, U$1.VCC, X41.KL
- net GND: no longer C10.2, C8.-
- net V-IN: now also R18.1, R19.1, R20.1, U$1.VCC, X41.KL
Changed lines of the file:
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@@
 <part name="GND4" library="supply1" deviceset="GND" device=""/>
 <part name="C7" library="Namenlos" deviceset="CAP_" device="0805" value="1u"/>
-<part name="C8" library="Namenlos" deviceset="CAP-POL_" device="D8"/>
 <part name="C9" library="Namenlos" deviceset="CAP-POL_" device="D8"/>
-<part name="C10" library="Namenlos" deviceset="CAP_" device="0805" value="100n"/>
 <part name="C11" library="Namenlos" deviceset="CAP_" device="0805" value="100n"/>
 <part name="P+4" library="supply1" deviceset="+5V" device=""/>
@@
 <part name="R5" library="Namenlos" deviceset="R_POT" device="TURN-X"/>
 <part name="JP2" library="pinhead" deviceset="PINHD-1X8" device=""/>
-<part name="IC9" library="40xx" deviceset="4050" device="D"/>
+<part name="IC9" library="40xx" library_urn="urn:adsk.eagle:library:80" deviceset="4050" device="D"/>
 <part name="+3V1" library="supply1" deviceset="+3V3" device=""/>
 <part name="GND24" library="supply1" deviceset="GND" device=""/>
 <part name="GND28" library="supply1" deviceset="GND" device=""/>
 <part name="+3V2" library="supply1" deviceset="+3V3" device=""/>
-<part name="IC10" library="v-reg" deviceset="TS5205" device="" technology="33"/>
+<part name="IC10" library="v-reg" library_urn="urn:adsk.eagle:library:409" deviceset="TS5205" device="" technology="33"/>
 <part name="P+13" library="supply1" deviceset="+5V" device=""/>
 <part name="+3V3" library="supply1" deviceset="+3V3" device=""/>
@@
 <part name="C4" library="Namenlos" deviceset="CAP_" device="0805" value="470p"/>
 <part name="GND35" library="supply1" deviceset="GND" device=""/>
-<part name="L2" library="inductors" library_urn="urn:adsk.eagle:library:243" deviceset="DR127" device="" value="SCDS127T-221M-N"/>
+<part name="L2" library="Namenlos" deviceset="INDUCTOR" device="0705" value="SCDS127T-221M-N"/>
 <part name="GND42" library="supply1" deviceset="GND" device=""/>
 <part name="R21" library="Namenlos" deviceset="R_" device="0805" value="3K9"/>
@@
 <instance part="GND4" gate="1" x="88.9" y="195.58"/>
 <instance part="C7" gate="G$1" x="109.22" y="205.74" rot="R90"/>
-<instance part="C8" gate="C$1" x="-27.94" y="195.58"/>
 <instance part="C9" gate="C$1" x="68.58" y="187.96"/>
-<instance part="C10" gate="G$1" x="-22.86" y="195.58"/>
 <instance part="C11" gate="G$1" x="63.5" y="187.96"/>
 <instance part="P+4" gate="1" x="73.66" y="200.66"/>
@@
 <wire x1="-35.56" y1="187.96" x2="-33.02" y2="187.96" width="0.1524" layer="91"/>
 <wire x1="-33.02" y1="187.96" x2="-33.02" y2="185.42" width="0.1524" layer="91"/>
-<pinref part="C10" gate="G$1" pin="2"/>
-<wire x1="-33.02" y1="187.96" x2="-27.94" y2="187.96" width="0.1524" layer="91"/>
-<wire x1="-27.94" y1="187.96" x2="-22.86" y2="187.96" width="0.1524" layer="91"/>
-<wire x1="-22.86" y1="187.96" x2="-22.86" y2="190.5" width="0.1524" layer="91"/>
-<junction x="-33.02" y="187.96"/>
-<pinref part="C8" gate="C$1" pin="-"/>
-<wire x1="-27.94" y1="190.5" x2="-27.94" y2="187.96" width="0.1524" layer="91"/>
-<junction x="-27.94" y="187.96"/>
 </segment>
 <segment>
@@
 </segment>
 </net>
-<net name="N$47" class="0">
+<net name="V-IN" class="0">
 <segment>
 <pinref part="X4" gate="1" pin="KL"/>
-<pinref part="C8" gate="C$1" pin="+"/>
-<wire x1="-35.56" y1="203.2" x2="-27.94" y2="203.2" width="0.1524" layer="91"/>
-<wire x1="-27.94" y1="203.2" x2="-27.94" y2="198.12" width="0.1524" layer="91"/>
-<pinref part="C10" gate="G$1" pin="1"/>
-<wire x1="-27.94" y1="203.2" x2="-22.86" y2="203.2" width="0.1524" layer="91"/>
-<wire x1="-22.86" y1="203.2" x2="-22.86" y2="198.12" width="0.1524" layer="91"/>
-<junction x="-27.94" y="203.2"/>
+<wire x1="-35.56" y1="203.2" x2="-15.24" y2="203.2" width="0.1524" layer="91"/>
 <pinref part="U$1" gate="G$1" pin="VCC"/>
 <wire x1="2.54" y1="187.96" x2="-5.08" y2="187.96" width="0.1524" layer="91"/>
@@
 <wire x1="-10.16" y1="187.96" x2="-15.24" y2="187.96" width="0.1524" layer="91"/>
 <wire x1="-15.24" y1="187.96" x2="-15.24" y2="203.2" width="0.1524" layer="91"/>
-<wire x1="-15.24" y1="203.2" x2="-22.86" y2="203.2" width="0.1524" layer="91"/>
-<junction x="-22.86" y="203.2"/>
 <pinref part="R18" gate="G$1" pin="1"/>
 <wire x1="-10.16" y1="190.5" x2="-10.16" y2="187.96" width="0.1524" layer="91"/>

Commit message: IDC
Parts:
- removed JP1: (no value), pinhead:PINHD-1X16
- removed JP2: (no value), pinhead:PINHD-1X8
- removed R17: (no value), Namenlos:R_0805
- removed X20, X21: (no value), pinhead:PINHD-1X2
- added R23: OPT, Namenlos:R_0805
- added X11: CON-IDC12ML12, Namenlos:CON-IDC12ML12
- added X14: CON-IDC08ML08, Namenlos:CON-IDC08ML08
- JP3: value (none) -> CON-IDC10ML10; device pinhead:PINHD-2X5 -> Namenlos:CON-IDC10ML10
Connections:
- removed net N$54: JP2.8, R17.2
- new net N$47: R5.S, X11.3
- net +3V3: now also X14.4; no longer JP2.4
- net +5V: now also R5.E, X11.11, X11.2; no longer JP1.15, JP1.2, R5.A
- net DISP_D4: now also X11.7; no longer JP1.11
- net DISP_D5: now also X11.8; no longer JP1.12
- net DISP_D6: now also X11.9; no longer JP1.13
- net DISP_D7: now also X11.10; no longer JP1.14
- net DISP_E: now also X11.6; no longer JP1.6
- net DISP_RS: now also X11.4; no longer JP1.4
- net GND: now also R5.A, X11.1, X11.12, X11.5, X14.3, X14.6; no longer JP1.1, JP1.16, JP1.5, JP2.3, JP2.6, R5.E, X20.2, X21.2
- net N$48: now also R23.1, X14.8; no longer JP1.3, R5.S
- net N$49: now also X14.1; no longer JP2.1
- net N$50: now also X14.2; no longer JP2.2
- net N$51: now also X14.5; no longer JP2.5
- net SD-MISO: now also X14.7; no longer JP2.7
- net SD_DET: now also R23.2; no longer R17.1
- net V-IN: no longer X20.1, X21.1
- net X-MAX: no longer C19.1, R9.1, X15.2
- net X-MIN: now also C19.1, R9.1, X15.2
- net Y-MAX: no longer C17.1, R7.1, X13.2
- net Y-MIN: now also C17.1, R7.1, X13.2
Other:
- moved on the sheet: R5

Commit message: CapPol
Parts:
- C21, C22, C23, C24, C25: value (none) -> 220u 35V; device Namenlos:CAP-POL_D6 -> Namenlos:CAP-POL_E3.5-8-11H
- C9: value (none) -> 220u 6.3V; device Namenlos:CAP-POL_D8 -> Namenlos:CAP-POL_D6
Changed lines of the file:
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@@
 <setting verticaltext="up"/>
 </settings>
-<grid distance="0.1" unitdist="inch" unit="inch" style="lines" multiple="1" display="no" altdistance="0.05" altunitdist="inch" altunit="inch"/>
+<grid distance="0.1" unitdist="inch" unit="inch" style="lines" multiple="1" display="no" altdistance="0.01" altunitdist="inch" altunit="inch"/>
 <layers>
 <layer number="1" name="Top" color="4" fill="1" visible="no" active="no"/>
@@
 <part name="GND4" library="supply1" deviceset="GND" device=""/>
 <part name="C7" library="Namenlos" deviceset="CAP_" device="0805" value="1u"/>
-<part name="C9" library="Namenlos" deviceset="CAP-POL_" device="D8"/>
+<part name="C9" library="Namenlos" deviceset="CAP-POL_" device="D6" value="220u 6.3V "/>
 <part name="C11" library="Namenlos" deviceset="CAP_" device="0805" value="100n"/>
 <part name="P+4" library="supply1" deviceset="+5V" device=""/>
@@
 <part name="R13" library="Namenlos" deviceset="R_" device="0805" value="20R"/>
 <part name="R14" library="Namenlos" deviceset="R_" device="0805" value="20R"/>
-<part name="C21" library="Namenlos" deviceset="CAP-POL_" device="D6"/>
-<part name="C22" library="Namenlos" deviceset="CAP-POL_" device="D6"/>
-<part name="C23" library="Namenlos" deviceset="CAP-POL_" device="D6"/>
-<part name="C24" library="Namenlos" deviceset="CAP-POL_" device="D6"/>
-<part name="C25" library="Namenlos" deviceset="CAP-POL_" device="D6"/>
+<part name="C21" library="Namenlos" deviceset="CAP-POL_" device="E3.5-8-11H" value="220u 35V"/>
+<part name="C22" library="Namenlos" deviceset="CAP-POL_" device="E3.5-8-11H" value="220u 35V"/>
+<part name="C23" library="Namenlos" deviceset="CAP-POL_" device="E3.5-8-11H" value="220u 35V"/>
+<part name="C24" library="Namenlos" deviceset="CAP-POL_" device="E3.5-8-11H" value="220u 35V"/>
+<part name="C25" library="Namenlos" deviceset="CAP-POL_" device="E3.5-8-11H" value="220u 35V"/>
 <part name="GND37" library="supply1" deviceset="GND" device=""/>
 <part name="GND38" library="supply1" deviceset="GND" device=""/>

Commit message: some
Parts:
- removed X7: (no value), pinhead:PINHD-1X4/90
- added JP1: (no value), pinhead:PINHD-2X4/90
- C21, C22, C23, C24, C25: device Namenlos:CAP-POL_E3.5-8-11H -> Namenlos:CAP-POL_E3,5-8-11H
Connections:
- net N$17: now also JP1.1, JP1.2; no longer X7.1
- net N$18: now also JP1.3, JP1.4; no longer X7.2
- net N$19: now also JP1.5, JP1.6; no longer X7.3
- net N$20: now also JP1.7, JP1.8; no longer X7.4
Changed lines of the file:
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@@
 <part name="X5" library="pinhead" deviceset="PINHD-1X4" device="/90"/>
 <part name="X6" library="pinhead" deviceset="PINHD-1X4" device="/90"/>
-<part name="X7" library="pinhead" deviceset="PINHD-1X4" device="/90"/>
 <part name="X8" library="pinhead" deviceset="PINHD-1X4" device="/90"/>
 <part name="X9" library="pinhead" deviceset="PINHD-1X4" device="/90"/>
@@
 <part name="R13" library="Namenlos" deviceset="R_" device="0805" value="20R"/>
 <part name="R14" library="Namenlos" deviceset="R_" device="0805" value="20R"/>
-<part name="C21" library="Namenlos" deviceset="CAP-POL_" device="E3.5-8-11H" value="220u 35V"/>
-<part name="C22" library="Namenlos" deviceset="CAP-POL_" device="E3.5-8-11H" value="220u 35V"/>
-<part name="C23" library="Namenlos" deviceset="CAP-POL_" device="E3.5-8-11H" value="220u 35V"/>
-<part name="C24" library="Namenlos" deviceset="CAP-POL_" device="E3.5-8-11H" value="220u 35V"/>
-<part name="C25" library="Namenlos" deviceset="CAP-POL_" device="E3.5-8-11H" value="220u 35V"/>
+<part name="C21" library="Namenlos" deviceset="CAP-POL_" device="E3,5-8-11H" value="220u 35V"/>
+<part name="C22" library="Namenlos" deviceset="CAP-POL_" device="E3,5-8-11H" value="220u 35V"/>
+<part name="C23" library="Namenlos" deviceset="CAP-POL_" device="E3,5-8-11H" value="220u 35V"/>
+<part name="C24" library="Namenlos" deviceset="CAP-POL_" device="E3,5-8-11H" value="220u 35V"/>
+<part name="C25" library="Namenlos" deviceset="CAP-POL_" device="E3,5-8-11H" value="220u 35V"/>
 <part name="GND37" library="supply1" deviceset="GND" device=""/>
 <part name="GND38" library="supply1" deviceset="GND" device=""/>
@@
 <part name="GND20" library="supply1" deviceset="GND" device=""/>
 <part name="R23" library="Namenlos" deviceset="R_" device="0805" value="OPT"/>
+<part name="JP1" library="pinhead" deviceset="PINHD-2X4" device="/90"/>
 </parts>
 <sheets>
@@
 <instance part="X5" gate="A" x="111.76" y="58.42"/>
 <instance part="X6" gate="A" x="111.76" y="27.94"/>
-<instance part="X7" gate="A" x="111.76" y="-2.54"/>
 <instance part="X8" gate="A" x="111.76" y="-33.02"/>
 <instance part="X9" gate="A" x="111.76" y="-63.5"/>
@@
 <instance part="GND40" gate="1" x="91.44" y="38.1" rot="R90"/>
 <instance part="GND41" gate="1" x="91.44" y="68.58" rot="R90"/>
+<instance part="JP1" gate="A" x="109.22" y="-2.54"/>
 </instances>
 <busses>
@@
 <segment>
 <pinref part="IC6" gate="IC$1" pin="2B"/>
-<pinref part="X7" gate="A" pin="1"/>
-<wire x1="109.22" y1="2.54" x2="73.66" y2="2.54" width="0.1524" layer="91"/>
+<wire x1="109.22" y1="2.54" x2="106.68" y2="2.54" width="0.1524" layer="91"/>
+<wire x1="106.68" y1="2.54" x2="73.66" y2="2.54" width="0.1524" layer="91"/>
+<wire x1="109.22" y1="2.54" x2="114.3" y2="2.54" width="0.1524" layer="91"/>
+<pinref part="JP1" gate="A" pin="1"/>
+<junction x="106.68" y="2.54"/>
+<pinref part="JP1" gate="A" pin="2"/>
 </segment>
 </net>
@@
 <segment>
 <pinref part="IC6" gate="IC$1" pin="2A"/>
-<pinref part="X7" gate="A" pin="2"/>
-<wire x1="109.22" y1="0" x2="73.66" y2="0" width="0.1524" layer="91"/>
+<wire x1="109.22" y1="0" x2="106.68" y2="0" width="0.1524" layer="91"/>
+<wire x1="106.68" y1="0" x2="73.66" y2="0" width="0.1524" layer="91"/>
+<wire x1="109.22" y1="0" x2="114.3" y2="0" width="0.1524" layer="91"/>
+<pinref part="JP1" gate="A" pin="3"/>
+<junction x="106.68" y="0"/>
+<pinref part="JP1" gate="A" pin="4"/>
 </segment>
 </net>
@@
 <segment>
 <pinref part="IC6" gate="IC$1" pin="1A"/>
-<pinref part="X7" gate="A" pin="3"/>
-<wire x1="109.22" y1="-2.54" x2="73.66" y2="-2.54" width="0.1524" layer="91"/>
+<wire x1="109.22" y1="-2.54" x2="106.68" y2="-2.54" width="0.1524" layer="91"/>
+<wire x1="106.68" y1="-2.54" x2="73.66" y2="-2.54" width="0.1524" layer="91"/>
+<wire x1="109.22" y1="-2.54" x2="114.3" y2="-2.54" width="0.1524" layer="91"/>
+<pinref part="JP1" gate="A" pin="5"/>
+<junction x="106.68" y="-2.54"/>
+<pinref part="JP1" gate="A" pin="6"/>
 </segment>
 </net>
@@
 <segment>
 <pinref part="IC6" gate="IC$1" pin="1B"/>
-<pinref part="X7" gate="A" pin="4"/>
-<wire x1="109.22" y1="-5.08" x2="73.66" y2="-5.08" width="0.1524" layer="91"/>
-</segment>
-</net>
+<wire x1="109.22" y1="-5.08" x2="106.68" y2="-5.08" width="0.1524" layer="91"/>
+<wire x1="106.68" y1="-5.08" x2="73.66" y2="-5.08" width="0.1524" layer="91"/>
+<wire x1="109.22" y1="-5.08" x2="114.3" y2="-5.08" width="0.1524" layer="91"/>
+<pinref part="JP1" gate="A" pin="7"/>
+<junction x="106.68" y="-5.08"/>
+<pinref part="JP1" gate="A" pin="8"/>
+</segment>
+</net>
