File: 3DPrinter/PowerSup24V18-20A.brd (EAGLE design)
At the start: 215 x 115 mm, 2 parts, among them X1 CON-7.62-02P

Commit message: StandBy Supply
Parts:
- added C1: 22u 400V, rcl:E5-13
- added C2, C3: 100n, Namenlos:C0805
- added C4, C5: 100u 25V, Namenlos:E2,5-7
- added CY1: 3n3 2kV, rcl:YC7B5
- added D1, D3: ES1J, Namenlos:DO214AC
- added D2: P6KE200A, Namenlos:DO15-12
- added IC1: POWER-TNY264PN, Namenlos:DIP-8B
- added OK1: (no value), Namenlos:DIL04
- added R1, R2, R3, R4: 1M2, Namenlos:R0805
- added R5: 210R, Namenlos:R0805
- added R6: 1K, Namenlos:R0805
- added R7: 43K, Namenlos:R0805
- added R8: 11K, Namenlos:R0805
- added R9: NTC-D12, Namenlos:NTC-D12
- added T1: TRANS-1/1EFD25-10, Namenlos:EFD25_10PIN
- added TL1: IC-TL431CDBZR, Namenlos:SOT23
- moved B1 126.8 mm to (106.7, 44.5), turned to 270 degrees
- moved X1 125.8 mm to (101.6, 33.0)
Connections:
- new net +12V: C4.+, C5.+, D3.C, R5.2, R7.2
- new net GND: C4.-, C5.-, CY1.2, T1.10
- new net N$1: B1.AC2, X1.P$1
- new net N$10: D1.C, D2.C
- new net N$11: C2.1, IC1.1
- new net N$12: R9.2, X1.P$2
- new net N$14: C3.1, OK1.2, R6.1, TL1.1
- new net N$15: OK1.1, R5.1, R6.2
- new net N$16: C3.2, R7.1, R8.2, TL1.2
- new net N$17: R8.1, TL1.3
- new net N$18: D3.A, T1.6
- new net N$2: B1.AC1, R9.1
- new net N$3: B1.+, C1.+, CY1.1, D2.A, R4.2, T1.5
- new net N$4: B1.-, C1.-, C2.2, IC1.2, IC1.3, IC1.7, IC1.8, OK1.3
- new net N$5: R1.2, R2.1
- new net N$6: R2.2, R3.1
- new net N$7: R3.2, R4.1
- new net N$8: IC1.4, OK1.4, R1.1
- new net N$9: D1.A, IC1.5, T1.1
Routing:
- net N$4: track 0.00 -> 80.0 mm
- net GND: track 0.00 -> 55.3 mm
- net N$8: track 0.00 -> 47.0 mm
- net N$3: track 0.00 -> 42.4 mm
- net +12V: track 0.00 -> 28.2 mm
- net N$9: track 0.00 -> 22.8 mm
- net N$1: track 0.00 -> 20.2 mm
- net N$16: track 0.00 -> 13.7 mm
- net N$18: track 0.00 -> 12.0 mm
- net N$14: track 0.00 -> 10.3 mm
- net N$15: track 0.00 -> 9.81 mm
- net N$12: track 0.00 -> 7.40 mm
- net N$2: track 0.00 -> 4.86 mm
- net N$10: track 0.00 -> 4.07 mm
- net N$17: track 0.00 -> 2.93 mm
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Other:
- board size 215 x 115 mm -> 115 x 161.7 mm

Commit message: Something
Parts:
- added B2: (no value), Namenlos:KBL
- added C10, C11, C6, C7, C8, C9: 100u 400V, rcl:E7,5-18
- added C12, C13: 1u5 250V, rcl:C225-074X268
- added C14: 1u 250V, rcl:C225-074X268
- added R10: NTC-D12, Namenlos:NTC-D12
- added R11, R12: 160K, Namenlos:MF-0125
- added T2: _TRANSFORMERS_GDT_20X6.5, Namenlos:_TRANSFORMERS_GDT_20X6.5
- added U1: SG3525AN, Namenlos:DIP254P762X510-16
- moved B1 0.63 mm to (106.7, 45.1)
- moved X1 0.63 mm to (101.6, 33.7)
Connections:
- new net +VI: U1.15
- new net AC1: B1.AC2, B2.AC1, X1.P$1
- new net AC2: R10.2, R9.2, X1.P$2
- new net N$13: B2.+, C10.+, C11.+, C12.1, C6.+, C7.+, C8.+, C9.+, R12.2
- new net N$19: B2.-, C10.-, C11.-, C13.2, C6.-, C7.-, C8.-, C9.-, R11.1
- new net N$20: T2.P1, U1.11
- new net N$21: T2.P2, U1.14
- net N$1: now also B2.AC2, R10.1; no longer B1.AC2, X1.P$1
- net N$12: now also C12.2, C13.1, C14.1, R11.2, R12.1; no longer R9.2, X1.P$2
Routing:
- net N$13: track 0.00 -> 145.6 mm
- net N$19: track 0.00 -> 128.6 mm
- net AC1: track 0.00 -> 48.9 mm
- net AC2: track 0.00 -> 27.1 mm
- net N$12: track 7.40 -> 20.4 mm
- net N$1: track 20.2 -> 14.7 mm
- net N$4: track 80.0 -> 79.4 mm
- net N$2: track 4.86 -> 5.50 mm
- net N$3: track 42.4 -> 41.8 mm

Commit message: Горячая сторона
Parts:
- added C15: 2n, Namenlos:C0805
- added C16, C18: 10u 16V, Namenlos:CT3528
- added C17, C19: 100n, Namenlos:C0805
- added R13, R14, R15: (no value), Namenlos:R1206
- added R16: 7K5, Namenlos:R0805
- added R17: 51R, Namenlos:R0805
- added R18, R19: 15K, Namenlos:R0805
- added R20: 1K5, Namenlos:R0805
- added T3: TRANS-1/1ETD39, Namenlos:ETD39
- added U$1: OPTO-EL3H4(TA)-VG, Namenlos:SSOP4
- added VT1, VT2: STP11NK40Z, Namenlos:TO-220V
- C1: value 22u 400V -> 100u 400V; device rcl:E5-13 -> rcl:E7,5-18
- moved C14 21.0 mm to (84.5, 131.4)
- moved T2 6.54 mm to (5.08, 32.4), turned to 0 degrees
- moved C1 0.63 mm to (106.7, 57.8)
Connections:
- removed net +VI: U1.15
- new net FB1: U$1.1
- new net FB2: U$1.2
- new net N$22: R13.2, T2.P2
- new net N$23: R14.1, T2.S2-1
- new net N$24: R15.1, T2.S1-2
- new net N$25: R14.2, VT1.1
- new net N$26: R15.2, VT2.1
- new net N$27: T2.S2-2, T3.1, T3.2, VT1.3, VT2.2
- new net N$28: C14.2, T3.7, T3.8
- new net N$29: R16.2, U1.6
- new net N$30: C15.2, R17.1, U1.5
- new net N$31: C19.2, R18.2, U$1.3, U1.16
- new net N$32: R17.2, U1.7
- new net N$33: C16.+, C18.+, U1.8
- new net N$34: R18.1, R19.2, U1.2
- new net N$35: C17.2, U1.9
- new net N$36: R20.2, U$1.4, U1.1
- new net TR-OUT1: T3.10, T3.11, T3.9
- new net TR-OUT2: T3.14, T3.15, T3.16
- net +12V: now also U1.13, U1.15
- net GND: now also C15.1, C16.-, C17.1, C18.-, C19.1, R16.1, R19.1, R20.1, U1.12
- net N$13: now also VT1.2
- net N$19: now also T2.S1-1, VT2.3
- net N$20: now also R13.1; no longer T2.P1
- net N$21: now also T2.P1; no longer T2.P2
Routing:
- net N$3: track 41.8 -> 28.7 mm
- net N$4: track 79.4 -> 75.8 mm

Commit message: Всё неправильно
Parts:
- added U$2, U$3: (no value), Namenlos:SK95-3M3_HOLE
- moved U$1 297.7 mm to (128.9, 114.9), turned to 270 degrees
- moved R20 296.9 mm to (125.7, 118.7), turned to 270 degrees
- moved C19 287.7 mm to (99.7, 111.1)
- moved C18 271.3 mm to (78.7, 123.2), turned to 90 degrees
- moved R19 269.8 mm to (94.0, 123.2), turned to 270 degrees
- moved R18 258.7 mm to (95.2, 115.6), turned to 180 degrees
- moved C17 255.6 mm to (80.0, 108.0)
- moved C16 250.0 mm to (75.6, 123.2), turned to 90 degrees
- moved R17 249.4 mm to (83.8, 121.3)
- moved C15 247.1 mm to (86.4, 123.8), turned to 270 degrees
- moved R16 240.2 mm to (83.8, 123.8), turned to 270 degrees
- moved VT2 217.3 mm to (59.7, 127.0)
- moved VT1 196.3 mm to (42.5, 127.0)
- moved R15 191.5 mm to (52.1, 124.5), turned to 180 degrees
- moved R14 177.6 mm to (40.0, 120.7), turned to 90 degrees
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Routing:
- net N$19: track 128.6 -> 213.5 mm
- net N$27: track 0.00 -> 71.5 mm
- net N$13: track 145.6 -> 211.2 mm
- net N$28: track 0.00 -> 59.6 mm
- net GND: track 55.3 -> 81.7 mm
- net N$12: track 20.4 -> 37.0 mm
- net N$21: track 0.00 -> 14.0 mm
- net N$22: track 0.00 -> 11.1 mm
- net +12V: track 28.2 -> 38.4 mm
- net N$23: track 0.00 -> 9.33 mm
- net N$4: track 75.8 -> 83.3 mm
- net N$3: track 28.7 -> 36.0 mm
- net N$34: track 0.00 -> 6.48 mm
- net N$31: track 0.00 -> 6.48 mm
- net N$33: track 0.00 -> 6.12 mm
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
Commit message: Вроде готово
Parts:
- added C20, C21, C22, C23: (no value), rcl:E7,5-16
- added C24: 100n, Namenlos:C0805
- added D4, D5, D6, D7: (no value), Namenlos:TO220ACS
- added D8: LED_3MM, Namenlos:LED3MM
- added JP1, JP2: (no value), pinhead:1X02
- added L1: (no value), Namenlos:D26.9/14.7/11.2
- added R21, R24: 1K, Namenlos:R0805
- added R22, R26: 2K, Namenlos:R0805
- added R23: 9K1, Namenlos:R0805
- added R25: 150R, Namenlos:RJ9W
- added TL2: IC-TL431CDBZR, Namenlos:SOT23
- added U$4, U$5, U$6, U$7: (no value), Namenlos:SK95-3M3_HOLE
- added X2: CON-7.62-02P, Namenlos:KF25C-7.62-02P-13
- R5: value 210R -> 1K
- R6: value 1K -> 2K
- R7: value 43K -> 7K5
- R8: value 11K -> 2K
- moved U$1 97.2 mm to (31.8, 118.1), turned to 90 degrees
- moved R20 92.1 mm to (33.7, 121.9)
- moved R14 72.9 mm to (101.0, 160.7), turned to 180 degrees
- moved U$2 72.4 mm to (108.0, 158.1), turned to 270 degrees
- moved VT1 72.4 mm to (108.0, 158.1), turned to 270 degrees
- moved R12 66.9 mm to (105.4, 114.3), turned to 0 degrees
- moved C19 64.0 mm to (36.8, 123.2), turned to 180 degrees
- moved R9 61.6 mm to (50.2, 33.0)
- moved C12 57.8 mm to (100.3, 109.9), turned to 180 degrees
- moved B1 57.2 mm to (49.5, 46.4)
- moved C1 57.2 mm to (49.5, 59.7)
- moved R1 57.2 mm to (41.9, 57.1)
- moved R2 57.2 mm to (41.9, 61.0)
- moved C2 57.2 mm to (39.4, 47.0)
- moved IC1 57.2 mm to (38.1, 49.5)
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Connections:
- new net N$37: D5.C, D6.C, L1.P$1, L1.P$2
- new net N$38: C20.-, C21.-, C22.-, C23.-, D4.A, D7.A, R24.1, R26.1, TL2.3, X2.P$2
- new net N$39: C20.+, C21.+, C22.+, C23.+, D8.A, L1.P$3, L1.P$4, R21.2, R23.2, X2.P$1
- new net N$40: R24.2, R25.A
- new net N$41: R23.1, R25.B
- new net N$42: C24.2, R25.W, TL2.2
- new net N$43: D8.K, R26.2
- net +12V: now also JP1.1, JP2.1
- net FB1: now also R21.1, R22.2
- net FB2: now also C24.1, R22.1, TL2.1
- net GND: now also JP1.2, JP2.2
- net N$27: now also T3.7, T3.8; no longer T3.1, T3.2
- net N$28: now also T3.1, T3.2; no longer T3.7, T3.8
- net TR-OUT1: now also D4.C, D5.A
- net TR-OUT2: now also D6.A, D7.C
Routing:
- net N$38: track 0.00 -> 262.6 mm, vias 0 -> 12
- net N$39: track 0.00 -> 142.8 mm
- net TR-OUT2: track 0.00 -> 77.1 mm
- net TR-OUT1: track 0.00 -> 77.1 mm
- net GND: track 81.7 -> 146.2 mm, vias 0 -> 2
- net N$27: track 71.5 -> 133.1 mm, vias 0 -> 4
- net N$37: track 0.00 -> 60.5 mm
- net N$23: track 9.33 -> 68.1 mm
- net N$28: track 59.6 -> 18.4 mm
- net N$24: track 5.77 -> 40.3 mm
- net +12V: track 38.4 -> 69.7 mm, vias 0 -> 2
- net N$21: track 14.0 -> 33.0 mm
- net N$3: track 36.0 -> 53.9 mm
- net FB2: track 0.00 -> 12.8 mm
- net N$36: track 0.00 -> 10.9 mm
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- added copper zone on layer 16, net N$37
- added copper zone on layer 16, net N$38
- added copper zone on layer 16, net N$39
- added copper zone on layer 16, net N$52

Commit message: как всегда
Parts:
- added C25: (no value), Namenlos:C050-024X044
- added D10, D9: (no value), Namenlos:DO214AC
- added R27: (no value), Namenlos:MF-2
- C20, C21, C22, C23: device rcl:E7,5-16 -> rcl:E5-13
- moved C23 7.65 mm to (19.1, 56.5)
- moved C22 5.08 mm to (8.26, 66.0)
- moved C21 2.62 mm to (19.1, 75.6)
Connections:
- new net N$44: C25.2, R27.2
- net N$13: now also D10.C
- net N$19: now also D9.A
- net N$27: now also D10.A, D9.C, R27.1
- net N$28: now also C25.1
Routing:
- net N$27: track 133.1 -> 160.0 mm
- net N$28: track 18.4 -> 39.8 mm
- net N$38: track 262.6 -> 247.6 mm
- net N$39: track 142.8 -> 129.0 mm
- net N$13: track 219.4 -> 210.2 mm
- net N$44: track 0.00 -> 2.54 mm
- net N$23: track 68.1 -> 66.3 mm
- net N$24: track 40.3 -> 39.2 mm

Commit message: исправил существенные косяки
Parts:
- moved U$2 213.4 mm to (-105.4, 158.1), flipped to the bottom
- moved U$3 213.4 mm to (-105.4, 136.5), flipped to the bottom
- moved VT1 213.4 mm to (-105.4, 158.1), flipped to the bottom
- moved VT2 213.4 mm to (-105.4, 136.5), flipped to the bottom
- moved D10 209.6 mm to (-103.5, 151.1), flipped to the top
- moved R12 208.3 mm to (-102.9, 114.3), flipped to the bottom
- moved C10 203.2 mm to (-100.3, 81.3), flipped to the bottom
- moved C6 203.2 mm to (-100.3, 44.5), flipped to the bottom
- moved C9 203.2 mm to (-100.3, 62.9), flipped to the bottom
- moved D9 203.2 mm to (-100.3, 129.5), flipped to the top
- moved R14 199.4 mm to (-98.4, 160.7), flipped to the top
- moved R15 199.4 mm to (-98.4, 139.1), flipped to the top
- moved C12 198.1 mm to (-97.8, 109.9), flipped to the bottom
- moved R27 191.8 mm to (-94.6, 157.5), flipped to the bottom
- moved R11 190.5 mm to (-94.0, 106.0), flipped to the bottom
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Connections:
- removed net N$17: R8.1, TL1.3
- net GND: now also R8.1, TL1.3
- net N$31: now also U$1.4; no longer U$1.3
- net N$36: now also U$1.3; no longer U$1.4
Routing:
- net GND: track 146.2 -> 157.7 mm
- net N$17: track 2.93 -> 0.00 mm
- net N$36: track 10.9 -> 13.4 mm
- net +12V: track 69.7 -> 68.0 mm
- net FB2: track 12.8 -> 14.4 mm
- net N$31: track 13.5 -> 12.2 mm
- net N$38: track 247.6 -> 248.3 mm
- added copper zone on layer 1, net N$37
- added copper zone on layer 1, net N$38
- added copper zone on layer 1, net N$39
- added copper zone on layer 1, net N$52
- removed copper zone on layer 16, net N$37
- removed copper zone on layer 16, net N$38
- removed copper zone on layer 16, net N$39
- removed copper zone on layer 16, net N$52
