File: 3DPrinter/PowerSup24V18-20A.sch (EAGLE design)
At the start: 2 parts, among them X1 CON-7.62-02P

Commit message: StandBy Supply
Parts:
- added C1: 22u 400V, rcl:CPOL-EUE5-13
- added C2, C3: 100n, Namenlos:CAP_0805
- added C4, C5: 100u 25V, Namenlos:CAP-POL_E2.5-7
- added CY1: 3n3 2kV, rcl:CYYC7B5
- added D1, D3: ES1J, Namenlos:DIODE_ES1J
- added D2: P6KE200A, Namenlos:SUPRESSORDO-204AC
- added IC1: POWER-TNY264PN, Namenlos:POWER-TNY264PN
- added OK1: (no value), Namenlos:OPTOTRANSPC817
- added R1, R2, R3, R4: 1M2, Namenlos:R_0805
- added R5: 210R, Namenlos:R_0805
- added R6: 1K, Namenlos:R_0805
- added R7: 43K, Namenlos:R_0805
- added R8: 11K, Namenlos:R_0805
- added R9: NTC-D12, Namenlos:NTC-D12
- added T1: TRANS-1/1EFD25-10, Namenlos:TRANS-1/1EFD25-10
- added TL1: IC-TL431CDBZR, Namenlos:IC-TL431CDBZR
Connections:
- new net +12V: C4.+, C5.+, D3.C, R5.2, R7.2
- new net GND: C4.-, C5.-, CY1.2, T1.S1-2
- new net N$1: B1.AC2, X11.KL
- new net N$10: D1.C, D2.C
- new net N$11: C2.1, IC1.BP
- new net N$12: R9.2, X12.KL
- new net N$14: C3.1, OK1.C, R6.1, TL1.C
- new net N$15: OK1.A, R5.1, R6.2
- new net N$16: C3.2, R7.1, R8.2, TL1.R
- new net N$17: R8.1, TL1.A
- new net N$18: D3.A, T1.S1-1
- new net N$2: B1.AC1, R9.1
- new net N$3: B1.+, C1.+, CY1.1, D2.A, R4.2, T1.P1-2
- new net N$4: B1.-, C1.-, C2.2, IC1.S, OK1.EMIT
- new net N$5: R1.2, R2.1
- new net N$6: R2.2, R3.1
- new net N$7: R3.2, R4.1
- new net N$8: IC1.EN, OK1.COL, R1.1
- new net N$9: D1.A, IC1.D, T1.P1-1
Other:
- note added: "Pri: 86 turns 0.2 mm 1 wire Sec: 8 turns 0.56 mm 1 wire Gap 0.115 mm Pimary Inductance 3.512 mH"
- moved on the sheet: B1, X11, X12

Commit message: Something
Parts:
- added B2: (no value), Namenlos:RECTIFIERKBL
- added C10, C11, C6, C7, C8, C9: 100u 400V, rcl:CPOL-EUE7.5-18
- added C12, C13: 1u5 250V, rcl:C-EU225-074X268
- added C14: 1u 250V, rcl:C-EU225-074X268
- added R10: NTC-D12, Namenlos:NTC-D12
- added R11, R12: 160K, Namenlos:R_MF-0125
- added T2: _TRANSFORMERS_GDT_20X6.5, Namenlos:_TRANSFORMERS_GDT_20X6.5
- added U1: SG3525AN, Namenlos:SG3525AN
Connections:
- new net AC1: B1.AC2, B2.AC2, X11.KL
- new net AC2: R10.2, R9.2, X12.KL
- new net N$13: B2.+, C10.+, C11.+, C12.1, C6.+, C7.+, C8.+, C9.+, R12.2
- new net N$19: B2.-, C10.-, C11.-, C13.2, C6.-, C7.-, C8.-, C9.-, R11.1
- new net N$20: T2.P1-1, U1.OUT_A
- new net N$21: T2.P1-2, U1.OUT_B
- net N$1: now also B2.AC1, R10.1; no longer B1.AC2, X11.KL
- net N$12: now also C12.2, C13.1, C14.1, R11.2, R12.1; no longer R9.2, X12.KL

Commit message: Горячая сторона
Parts:
- added C15: 2n, Namenlos:CAP_0805
- added C16, C18: 10u 16V, Namenlos:CAP-POL_3528
- added C17, C19: 100n, Namenlos:CAP_0805
- added R13, R14, R15: (no value), Namenlos:R_1206
- added R16: 7K5, Namenlos:R_0805
- added R17: 51R, Namenlos:R_0805
- added R18, R19: 15K, Namenlos:R_0805
- added R20: 1K5, Namenlos:R_0805
- added T3: TRANS-1/1ETD39, Namenlos:TRANS-1/1ETD39
- added U$1: OPTO-EL3H4(TA)-VG, Namenlos:OPTO-EL3H4(TA)-VG
- added VT1, VT2: STP11NK40Z, Namenlos:FET-NTO-220
- C1: value 22u 400V -> 100u 400V; device rcl:CPOL-EUE5-13 -> rcl:CPOL-EUE7.5-18
Connections:
- new net FB1: U$1.P$1
- new net FB2: U$1.P$2
- new net N$22: R13.2, T2.P1-2
- new net N$23: R14.1, T2.S2-1
- new net N$24: R15.1, T2.S1-2
- new net N$25: R14.2, VT1.G
- new net N$26: R15.2, VT2.G
- new net N$27: T2.S2-2, T3.P1-1, VT1.S, VT2.D
- new net N$28: C14.2, T3.P1-2
- new net N$29: R16.2, U1.RT
- new net N$30: C15.2, R17.1, U1.CT
- new net N$31: C19.2, R18.2, U$1.P$3, U1.VREF
- new net N$32: R17.2, U1.DISCH
- new net N$33: C16.+, C18.+, U1.SOFT_START
- new net N$34: R18.1, R19.2, U1.N.I.IN
- new net N$35: C17.2, U1.COMP
- new net N$36: R20.2, U$1.P$4, U1.INV.IN
- new net TR-OUT1: T3.S1-2
- new net TR-OUT2: T3.S1-1
- net +12V: now also U1.+VI, U1.VC
- net GND: now also C15.1, C16.-, C17.1, C18.-, C19.1, R16.1, R19.1, R20.1, U1.GND
- net N$13: now also VT1.D
- net N$19: now also T2.S1-1, VT2.S
- net N$20: now also R13.1; no longer T2.P1-1
- net N$21: now also T2.P1-1; no longer T2.P1-2
Other:
- note added: "Pimary: 35 turns 3 wires 0.56 mm Secondary: 8 turns 9 wires 0.56 mm"
- moved on the sheet: T2, U1

Commit message: Вроде готово
Parts:
- added C20, C21, C22, C23: (no value), rcl:CPOL-EUE7.5-16
- added C24: 100n, Namenlos:CAP_0805
- added D4, D5, D6, D7: (no value), Namenlos:DIODE_TO-220-2
- added D8: LED_3MM, Namenlos:LED_3MM
- added JP1, JP2: (no value), pinhead:PINHD-1X2
- added L1: (no value), Namenlos:INDUCTORD26.7
- added R21, R24: 1K, Namenlos:R_0805
- added R22, R26: 2K, Namenlos:R_0805
- added R23: 9K1, Namenlos:R_0805
- added R25: 150R, Namenlos:R_POTTURN-X
- added TL2: IC-TL431CDBZR, Namenlos:IC-TL431CDBZR
- added X2: CON-7.62-02P, Namenlos:CON-7.62-02P
- R5: value 210R -> 1K
- R6: value 1K -> 2K
- R7: value 43K -> 7K5
- R8: value 11K -> 2K
Connections:
- new net N$37: D5.C, D6.C, L1.1
- new net N$38: C20.-, C21.-, C22.-, C23.-, D4.A, D7.A, R24.1, R26.1, TL2.A, X22.KL
- new net N$39: C20.+, C21.+, C22.+, C23.+, D8.A, L1.2, R21.2, R23.2, X21.KL
- new net N$40: R24.2, R25.A
- new net N$41: R23.1, R25.E
- new net N$42: C24.2, R25.S, TL2.R
- new net N$43: D8.C, R26.2
- net +12V: now also JP1.1, JP2.1
- net FB1: now also R21.1, R22.2
- net FB2: now also C24.1, R22.1, TL2.C
- net GND: now also JP1.2, JP2.2
- net N$27: now also T3.P1-2; no longer T3.P1-1
- net N$28: now also T3.P1-1; no longer T3.P1-2
- net TR-OUT1: now also D4.C, D5.A
- net TR-OUT2: now also D6.A, D7.C

Commit message: как всегда
Parts:
- added C25: (no value), Namenlos:CAP_C50-024X044
- added D10, D9: (no value), Namenlos:DIODE_ES1J
- added R27: (no value), Namenlos:R_MF-2
- C20, C21, C22, C23: device rcl:CPOL-EUE7.5-16 -> rcl:CPOL-EUE5-13
Connections:
- new net N$44: C25.2, R27.2
- net N$13: now also D10.C
- net N$19: now also D9.A
- net N$27: now also D10.A, D9.C, R27.1
- net N$28: now also C25.1
Changed lines of the file:
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@@
 <?xml version="1.0" encoding="utf-8"?>
 <!DOCTYPE eagle SYSTEM "eagle.dtd">
-<eagle version="8.3.2">
+<eagle version="8.3.1">
 <drawing>
 <settings>
@@
 <part name="JP2" library="pinhead" deviceset="PINHD-1X2" device=""/>
 <part name="L1" library="Namenlos" deviceset="INDUCTOR" device="D26.7"/>
-<part name="C20" library="rcl" library_urn="urn:adsk.eagle:library:334" deviceset="CPOL-EU" device="E7.5-16" package3d_urn="urn:adsk.eagle:package:23382/2"/>
-<part name="C21" library="rcl" library_urn="urn:adsk.eagle:library:334" deviceset="CPOL-EU" device="E7.5-16" package3d_urn="urn:adsk.eagle:package:23382/2"/>
-<part name="C22" library="rcl" library_urn="urn:adsk.eagle:library:334" deviceset="CPOL-EU" device="E7.5-16" package3d_urn="urn:adsk.eagle:package:23382/2"/>
-<part name="C23" library="rcl" library_urn="urn:adsk.eagle:library:334" deviceset="CPOL-EU" device="E7.5-16" package3d_urn="urn:adsk.eagle:package:23382/2"/>
+<part name="C20" library="rcl" library_urn="urn:adsk.eagle:library:334" deviceset="CPOL-EU" device="E5-13" package3d_urn="urn:adsk.eagle:package:23375/1"/>
+<part name="C21" library="rcl" library_urn="urn:adsk.eagle:library:334" deviceset="CPOL-EU" device="E5-13" package3d_urn="urn:adsk.eagle:package:23375/1"/>
+<part name="C22" library="rcl" library_urn="urn:adsk.eagle:library:334" deviceset="CPOL-EU" device="E5-13" package3d_urn="urn:adsk.eagle:package:23375/1"/>
+<part name="C23" library="rcl" library_urn="urn:adsk.eagle:library:334" deviceset="CPOL-EU" device="E5-13" package3d_urn="urn:adsk.eagle:package:23375/1"/>
 <part name="X2" library="Namenlos" deviceset="CON-7.62-02P" device=""/>
 <part name="TL2" library="Namenlos" deviceset="IC-TL431" device="CDBZR"/>
@@
 <part name="D8" library="Namenlos" deviceset="LED_" device="3MM"/>
 <part name="R26" library="Namenlos" deviceset="R_" device="0805" value="2K"/>
+<part name="R27" library="Namenlos" deviceset="R_" device="MF-2"/>
+<part name="C25" library="Namenlos" deviceset="CAP_" device="C50-024X044"/>
+<part name="D9" library="Namenlos" deviceset="DIODE_" device="ES1J"/>
+<part name="D10" library="Namenlos" deviceset="DIODE_" device="ES1J"/>
 </parts>
 <sheets>
@@
 <instance part="U$1" gate="G$1" x="144.78" y="-78.74" rot="MR0"/>
 <instance part="C19" gate="G$1" x="-20.32" y="-25.4" rot="R180"/>
+<instance part="R27" gate="G$1" x="132.08" y="-17.78" rot="R90"/>
+<instance part="C25" gate="G$1" x="132.08" y="-7.62"/>
+<instance part="D9" gate="G$1" x="116.84" y="-35.56" rot="R90"/>
+<instance part="D10" gate="G$1" x="116.84" y="-2.54" rot="R90"/>
 </instances>
 <busses>
@@
 <wire x1="33.02" y1="81.28" x2="33.02" y2="86.36" width="0.1524" layer="91"/>
 <pinref part="C10" gate="G$1" pin="+"/>
-<wire x1="33.02" y1="86.36" x2="43.18" y2="86.36" width="0.1524" layer="91"/>
-<wire x1="43.18" y1="86.36" x2="48.26" y2="86.36" width="0.1524" layer="91"/>
+<wire x1="33.02" y1="86.36" x2="48.26" y2="86.36" width="0.1524" layer="91"/>
 <wire x1="48.26" y1="86.36" x2="53.34" y2="86.36" width="0.1524" layer="91"/>
 <wire x1="53.34" y1="86.36" x2="58.42" y2="86.36" width="0.1524" layer="91"/>
@@
 <junction x="78.74" y="86.36"/>
 <pinref part="VT1" gate="G$1" pin="D"/>
-<wire x1="111.76" y1="2.54" x2="111.76" y2="86.36" width="0.1524" layer="91"/>
+<wire x1="111.76" y1="2.54" x2="111.76" y2="5.08" width="0.1524" layer="91"/>
+<wire x1="111.76" y1="5.08" x2="111.76" y2="86.36" width="0.1524" layer="91"/>
 <wire x1="111.76" y1="86.36" x2="83.82" y2="86.36" width="0.1524" layer="91"/>
 <junction x="83.82" y="86.36"/>
+<pinref part="D10" gate="G$1" pin="C"/>
+<wire x1="116.84" y1="0" x2="116.84" y2="5.08" width="0.1524" layer="91"/>
+<wire x1="116.84" y1="5.08" x2="111.76" y2="5.08" width="0.1524" layer="91"/>
+<junction x="111.76" y="5.08"/>
 </segment>
 </net>
@@
 <segment>
 <pinref part="B2" gate="1" pin="-"/>
-<wire x1="43.18" y1="60.96" x2="33.02" y2="60.96" width="0.1524" layer="91"/>
+<wire x1="48.26" y1="60.96" x2="33.02" y2="60.96" width="0.1524" layer="91"/>
 <wire x1="33.02" y1="60.96" x2="33.02" y2="71.12" width="0.1524" layer="91"/>
 <pinref part="C11" gate="G$1" pin="-"/>
-<wire x1="43.18" y1="60.96" x2="48.26" y2="60.96" width="0.1524" layer="91"/>
 <wire x1="48.26" y1="60.96" x2="53.34" y2="60.96" width="0.1524" layer="91"/>
 <wire x1="53.34" y1="60.96" x2="58.42" y2="60.96" width="0.1524" layer="91"/>
@@
 <junction x="78.74" y="60.96"/>
 <pinref part="VT2" gate="G$1" pin="S"/>
-<wire x1="111.76" y1="-40.64" x2="111.76" y2="-45.72" width="0.1524" layer="91"/>
+<wire x1="111.76" y1="-40.64" x2="111.76" y2="-43.18" width="0.1524" layer="91"/>
+<wire x1="111.76" y1="-43.18" x2="111.76" y2="-45.72" width="0.1524" layer="91"/>
 <wire x1="111.76" y1="-45.72" x2="121.92" y2="-45.72" width="0.1524" layer="91"/>
 <wire x1="121.92" y1="-45.72" x2="121.92" y2="60.96" width="0.1524" layer="91"/>
@@
 <pinref part="T2" gate="G$1" pin="S1-1"/>
 <wire x1="91.44" y1="-30.48" x2="76.2" y2="-30.48" width="0.1524" layer="91"/>
+<pinref part="D9" gate="G$1" pin="A"/>
+<wire x1="116.84" y1="-38.1" x2="116.84" y2="-43.18" width="0.1524" layer="91"/>
+<wire x1="116.84" y1="-43.18" x2="111.76" y2="-43.18" width="0.1524" layer="91"/>
+<junction x="111.76" y="-43.18"/>
 </segment>
 </net>
@@
 <wire x1="76.2" y1="-22.86" x2="111.76" y2="-22.86" width="0.1524" layer="91"/>
 <pinref part="VT2" gate="G$1" pin="D"/>
-<wire x1="111.76" y1="-22.86" x2="111.76" y2="-30.48" width="0.1524" layer="91"/>
+<wire x1="111.76" y1="-22.86" x2="111.76" y2="-27.94" width="0.1524" layer="91"/>
 <pinref part="VT1" gate="G$1" pin="S"/>
-<wire x1="111.76" y1="-22.86" x2="111.76" y2="-7.62" width="0.1524" layer="91"/>
+<wire x1="111.76" y1="-27.94" x2="111.76" y2="-30.48" width="0.1524" layer="91"/>
+<wire x1="111.76" y1="-22.86" x2="111.76" y2="-10.16" width="0.1524" layer="91"/>
 <junction x="111.76" y="-22.86"/>
+<wire x1="111.76" y1="-10.16" x2="111.76" y2="-7.62" width="0.1524" layer="91"/>
 <wire x1="137.16" y1="-17.78" x2="137.16" y2="-22.86" width="0.1524" layer="91"/>
-<wire x1="137.16" y1="-22.86" x2="111.76" y2="-22.86" width="0.1524" layer="91"/>
+<wire x1="137.16" y1="-22.86" x2="132.08" y2="-22.86" width="0.1524" layer="91"/>
 <pinref part="T3" gate="G$1" pin="P1-2"/>
+<wire x1="132.08" y1="-22.86" x2="111.76" y2="-22.86" width="0.1524" layer="91"/>
 <wire x1="137.16" y1="-17.78" x2="139.7" y2="-17.78" width="0.1524" layer="91"/>
+<pinref part="R27" gate="G$1" pin="1"/>
+<junction x="132.08" y="-22.86"/>
+<pinref part="D10" gate="G$1" pin="A"/>
+<wire x1="116.84" y1="-5.08" x2="116.84" y2="-10.16" width="0.1524" layer="91"/>
+<wire x1="116.84" y1="-10.16" x2="111.76" y2="-10.16" width="0.1524" layer="91"/>
+<junction x="111.76" y="-10.16"/>
+<pinref part="D9" gate="G$1" pin="C"/>
+<wire x1="116.84" y1="-33.02" x2="116.84" y2="-27.94" width="0.1524" layer="91"/>
+<wire x1="116.84" y1="-27.94" x2="111.76" y2="-27.94" width="0.1524" layer="91"/>
+<junction x="111.76" y="-27.94"/>
 </segment>
 </net>
@@
 <pinref part="C14" gate="G$1" pin="2"/>
 <wire x1="99.06" y1="73.66" x2="132.08" y2="73.66" width="0.1524" layer="91"/>
-<wire x1="132.08" y1="73.66" x2="132.08" y2="-7.62" width="0.1524" layer="91"/>
+<wire x1="132.08" y1="73.66" x2="132.08" y2="-5.08" width="0.1524" layer="91"/>
 <pinref part="T3" gate="G$1" pin="P1-1"/>
+<wire x1="132.08" y1="-5.08" x2="132.08" y2="-7.62" width="0.1524" layer="91"/>
 <wire x1="139.7" y1="-7.62" x2="132.08" y2="-7.62" width="0.1524" layer="91"/>
+<pinref part="C25" gate="G$1" pin="1"/>
+<junction x="132.08" y="-5.08"/>
 </segment>
 </net>
@@
 </segment>
 </net>
+<net name="N$44" class="0">
+<segment>
+<pinref part="R27" gate="G$1" pin="2"/>
+<pinref part="C25" gate="G$1" pin="2"/>
+</segment>
+</net>

Commit message: исправил существенные косяки
Connections:
- removed net N$17: R8.1, TL1.A
- net GND: now also R8.1, TL1.A
- net N$31: now also U$1.P$4; no longer U$1.P$3
- net N$36: now also U$1.P$3; no longer U$1.P$4
Changed lines of the file:
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@@
 <?xml version="1.0" encoding="utf-8"?>
 <!DOCTYPE eagle SYSTEM "eagle.dtd">
-<eagle version="8.3.1">
+<eagle version="8.3.2">
 <drawing>
 <settings>
@@
 <instance part="C18" gate="C$1" x="-7.62" y="-48.26"/>
 <instance part="R20" gate="G$1" x="-5.08" y="-68.58"/>
-<instance part="U$1" gate="G$1" x="144.78" y="-78.74" rot="MR0"/>
+<instance part="U$1" gate="G$1" x="144.78" y="-78.74" rot="R180"/>
 <instance part="C19" gate="G$1" x="-20.32" y="-25.4" rot="R180"/>
 <instance part="R27" gate="G$1" x="132.08" y="-17.78" rot="R90"/>
@@
 <wire x1="-20.32" y1="-20.32" x2="-22.86" y2="-20.32" width="0.1524" layer="91"/>
 <wire x1="-22.86" y1="-20.32" x2="-22.86" y2="-22.86" width="0.1524" layer="91"/>
-<pinref part="U$1" gate="G$1" pin="P$3"/>
-<wire x1="134.62" y1="-81.28" x2="-27.94" y2="-81.28" width="0.1524" layer="91"/>
 <wire x1="-27.94" y1="-81.28" x2="-27.94" y2="-20.32" width="0.1524" layer="91"/>
 <wire x1="-27.94" y1="-20.32" x2="-22.86" y2="-20.32" width="0.1524" layer="91"/>
@@
 <pinref part="C19" gate="G$1" pin="2"/>
 <junction x="-20.32" y="-20.32"/>
+<pinref part="U$1" gate="G$1" pin="P$4"/>
+<wire x1="134.62" y1="-81.28" x2="-27.94" y2="-81.28" width="0.1524" layer="91"/>
 </segment>
 </net>
@@
 <pinref part="U1" gate="A" pin="INV.IN"/>
 <wire x1="5.08" y1="-48.26" x2="17.78" y2="-48.26" width="0.1524" layer="91"/>
-<pinref part="U$1" gate="G$1" pin="P$4"/>
-<wire x1="134.62" y1="-76.2" x2="5.08" y2="-76.2" width="0.1524" layer="91"/>
 <wire x1="5.08" y1="-76.2" x2="5.08" y2="-68.58" width="0.1524" layer="91"/>
 <junction x="5.08" y="-68.58"/>
+<pinref part="U$1" gate="G$1" pin="P$3"/>
+<wire x1="5.08" y1="-76.2" x2="134.62" y2="-76.2" width="0.1524" layer="91"/>
 </segment>
 </net>
@@
 <segment>
 <pinref part="U$1" gate="G$1" pin="P$1"/>
+<wire x1="154.94" y1="-81.28" x2="160.02" y2="-81.28" width="0.1524" layer="91"/>
+<label x="157.48" y="-81.28" size="1.778" layer="95"/>
+</segment>
+</net>
+<net name="FB2" class="0">
+<segment>
+<pinref part="U$1" gate="G$1" pin="P$2"/>
 <wire x1="154.94" y1="-76.2" x2="160.02" y2="-76.2" width="0.1524" layer="91"/>
 <label x="157.48" y="-76.2" size="1.778" layer="95"/>
-</segment>
-</net>
-<net name="FB2" class="0">
-<segment>
-<pinref part="U$1" gate="G$1" pin="P$2"/>
-<wire x1="154.94" y1="-81.28" x2="160.02" y2="-81.28" width="0.1524" layer="91"/>
-<label x="157.48" y="-81.28" size="1.778" layer="95"/>
 </segment>
 </net>
@@
 </segment>
 </net>
-<net name="N$17" class="0">
-<segment>
-<pinref part="TL1" gate="G$1" pin="A"/>
-<wire x1="152.4" y1="-12.7" x2="152.4" y2="-15.24" width="0.1524" layer="91"/>
-<pinref part="R8" gate="G$1" pin="1"/>
-<wire x1="152.4" y1="-15.24" x2="177.8" y2="-15.24" width="0.1524" layer="91"/>
-<wire x1="177.8" y1="-15.24" x2="177.8" y2="-12.7" width="0.1524" layer="91"/>
-</segment>
-</net>
 <net name="N$18" class="0">
 <segment>
@@
 <junction x="187.96" y="76.2"/>
 <junction x="187.96" y="66.04"/>
-</segment>
-</net>
+<pinref part="TL1" gate="G$1" pin="A"/>
+<wire x1="152.4" y1="-12.7" x2="152.4" y2="-15.24" width="0.1524" layer="91"/>
+<pinref part="R8" gate="G$1" pin="1"/>
+<wire x1="152.4" y1="-15.24" x2="177.8" y2="-15.24" width="0.1524" layer="91"/>
+<wire x1="177.8" y1="-15.24" x2="177.8" y2="-12.7" width="0.1524" layer="91"/>
+<wire x1="177.8" y1="-15.24" x2="187.96" y2="-15.24" width="0.1524" layer="91"/>
+<wire x1="187.96" y1="-15.24" x2="187.96" y2="66.04" width="0.1524" layer="91"/>
+<junction x="177.8" y="-15.24"/>
+</segment>
+</net>
