File: 3DPrinter/Power_ToOctoPi.sch (EAGLE design)
At the start: 39 parts, among them IC1 7805DT, K1 G5LE, K2 G5LE

Commit message: _
Parts:
- removed IC1: 7805DT, linear:7805DT
- added C11: 100n, Namenlos:CAP_0805
- added C8: 470p, Namenlos:CAP_0805
- added C9: 220u 6.3V, Namenlos:CAP-POL_D6
- added D2: MBRA130LT3G, Namenlos:DIODE-SH_SMA
- added L2: SCDS127T-221M-N, Namenlos:INDUCTOR0705
- added R18, R19, R20: 1R, Namenlos:R_0805
- added R21: 3K9, Namenlos:R_0805
- added R22: 1K3, Namenlos:R_0805
- added U$4: MC33063/MC34063D, adafruit:MC33063/MC34063D
Connections:
- removed net N$18: K22.S, RALAY1.KL
- new net N$55: R18.2, R19.2, R20.2, U$4.DC, U$4.IPK, U$4.SWC
- new net N$56: D2.C, L2.1, U$4.SWE
- new net N$57: C8.1, U$4.TC
- new net N$59: R21.1, R22.2, U$4.COMP
- net +12V: now also R18.1, R19.1, R20.1, U$4.VCC; no longer IC1.VI
- net +5V: now also C11.1, C9.+, L2.2, R21.2; no longer IC1.VO
- net GND: now also C11.2, C8.2, C9.-, D2.A, R22.1, U$4.GND; no longer IC1.GND
- net N$1: now also K22.S
- net N$2: now also RALAY1.KL
Other:
- moved on the sheet: K2, RALAY1, RALAY2

Commit message: _
Parts:
- removed OVERLIGHT: (no value), pinhead:PINHD-1X2
- added R12, R2: 100R, Namenlos:R_0805
- R4: device pot:TRIM_EU-S75H -> Namenlos:R_POTTURN-X
- VT1, VT2: device Namenlos:FET-NSOT-23 -> Namenlos:FET-NPF-6X5
Connections:
- new net N$13: CONTROL.1, R2.1
- new net N$18: CONTROL.2, R12.2
- net GND: no longer OVERLIGHT.2
- net N$34: now also R2.2; no longer CONTROL.1
- net N$35: now also R12.1; no longer CONTROL.2
- net N$36: no longer OVERLIGHT.1
Changed lines of the file:
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@@
 <?xml version="1.0" encoding="utf-8"?>
 <!DOCTYPE eagle SYSTEM "eagle.dtd">
-<eagle version="8.4.0">
+<eagle version="8.3.2">
 <drawing>
 <settings>
@@
 <part name="R6" library="rcl" deviceset="R-EU_" device="R1206" value="1R1"/>
 <part name="D3" library="Namenlos" deviceset="DIODE_" device="ES1J"/>
-<part name="R4" library="pot" deviceset="TRIM_EU-" device="S75H"/>
+<part name="R4" library="Namenlos" deviceset="R_POT" device="TURN-X"/>
 <part name="P+1" library="supply1" library_urn="urn:adsk.eagle:library:371" deviceset="+12V" device=""/>
 <part name="GND1" library="supply1" library_urn="urn:adsk.eagle:library:371" deviceset="GND" device=""/>
@@
 <part name="P+4" library="supply1" library_urn="urn:adsk.eagle:library:371" deviceset="+12V" device=""/>
 <part name="P+5" library="supply1" library_urn="urn:adsk.eagle:library:371" deviceset="+12V" device=""/>
-<part name="VT1" library="Namenlos" deviceset="FET-N" device="SOT-23"/>
-<part name="VT2" library="Namenlos" deviceset="FET-N" device="SOT-23"/>
+<part name="VT1" library="Namenlos" deviceset="FET-N" device="PF-6X5"/>
+<part name="VT2" library="Namenlos" deviceset="FET-N" device="PF-6X5"/>
 <part name="GND3" library="supply1" library_urn="urn:adsk.eagle:library:371" deviceset="GND" device=""/>
 <part name="GND4" library="supply1" library_urn="urn:adsk.eagle:library:371" deviceset="GND" device=""/>
 <part name="R9" library="Namenlos" deviceset="R_" device="0805" value="11K"/>
 <part name="R11" library="Namenlos" deviceset="R_" device="0805" value="11K"/>
-<part name="OVERLIGHT" library="pinhead" deviceset="PINHD-1X2" device=""/>
 <part name="CONTROL" library="pinhead" deviceset="PINHD-1X2" device=""/>
 <part name="5V" library="pinhead" deviceset="PINHD-1X2" device=""/>
@@
 <part name="P+7" library="supply1" library_urn="urn:adsk.eagle:library:371" deviceset="+12V" device=""/>
 <part name="GND6" library="supply1" library_urn="urn:adsk.eagle:library:371" deviceset="GND" device=""/>
-<part name="GND7" library="supply1" library_urn="urn:adsk.eagle:library:371" deviceset="GND" device=""/>
 <part name="RALAY" library="Namenlos" deviceset="CON-7.62-02P" device=""/>
 <part name="C5" library="Namenlos" deviceset="CAP-POL_" device="E5-10.5" value="470u"/>
@@
 <part name="GND43" library="supply1" deviceset="GND" device=""/>
 <part name="P+3" library="supply1" library_urn="urn:adsk.eagle:library:371" deviceset="+12V" device=""/>
+<part name="R2" library="Namenlos" deviceset="R_" device="0805" value="100R"/>
+<part name="R12" library="Namenlos" deviceset="R_" device="0805" value="100R"/>
 </parts>
 <sheets>
@@
 <instance part="R6" gate="G$1" x="71.12" y="-35.56" rot="R90"/>
 <instance part="D3" gate="G$1" x="99.06" y="66.04"/>
-<instance part="R4" gate="1" x="149.86" y="-17.78" rot="R180"/>
+<instance part="R4" gate="G$1" x="149.86" y="-17.78" rot="R180"/>
 <instance part="P+1" gate="1" x="233.68" y="66.04" rot="R270"/>
 <instance part="GND1" gate="1" x="233.68" y="40.64" rot="R90"/>
@@
 <instance part="R9" gate="G$1" x="254" y="-30.48" rot="R90"/>
 <instance part="R11" gate="G$1" x="254" y="-93.98" rot="R90"/>
-<instance part="OVERLIGHT" gate="G$1" x="332.74" y="22.86"/>
 <instance part="CONTROL" gate="G$1" x="226.06" y="-53.34" rot="MR0"/>
 <instance part="5V" gate="G$1" x="175.26" y="-33.02" rot="MR0"/>
@@
 <instance part="P+7" gate="1" x="320.04" y="48.26"/>
 <instance part="GND6" gate="1" x="309.88" y="10.16"/>
-<instance part="GND7" gate="1" x="325.12" y="10.16"/>
 <instance part="RALAY" gate="1" x="-2.54" y="50.8" rot="R90"/>
 <instance part="RALAY" gate="2" x="-40.64" y="2.54" rot="R180"/>
@@
 <instance part="GND43" gate="1" x="121.92" y="-124.46"/>
 <instance part="P+3" gate="1" x="111.76" y="-78.74"/>
+<instance part="R2" gate="G$1" x="238.76" y="-35.56" rot="R90"/>
+<instance part="R12" gate="G$1" x="238.76" y="-66.04" rot="R90"/>
 </instances>
 <busses>
@@
 <pinref part="U$3" gate="G$1" pin="R"/>
 <wire x1="129.54" y1="-22.86" x2="129.54" y2="-17.78" width="0.1524" layer="91"/>
-<pinref part="R4" gate="1" pin="S"/>
+<pinref part="R4" gate="G$1" pin="S"/>
 <wire x1="144.78" y1="-17.78" x2="129.54" y2="-17.78" width="0.1524" layer="91"/>
 </segment>
@@
 <pinref part="C7" gate="G$1" pin="2"/>
 <wire x1="142.24" y1="-10.16" x2="149.86" y2="-10.16" width="0.1524" layer="91"/>
-<pinref part="R4" gate="1" pin="A"/>
+<pinref part="R4" gate="G$1" pin="A"/>
 <wire x1="149.86" y1="-12.7" x2="149.86" y2="-10.16" width="0.1524" layer="91"/>
 <junction x="149.86" y="-10.16"/>
@@
 <segment>
 <pinref part="R8" gate="G$1" pin="2"/>
-<pinref part="R4" gate="1" pin="E"/>
+<pinref part="R4" gate="G$1" pin="E"/>
 </segment>
 </net>
@@
 </segment>
 <segment>
-<pinref part="OVERLIGHT" gate="G$1" pin="2"/>
-<pinref part="GND7" gate="1" pin="GND"/>
-<wire x1="330.2" y1="22.86" x2="325.12" y2="22.86" width="0.1524" layer="91"/>
-<wire x1="325.12" y1="22.86" x2="325.12" y2="12.7" width="0.1524" layer="91"/>
-</segment>
-<segment>
 <pinref part="U$4" gate="G$1" pin="GND"/>
 <pinref part="GND33" gate="1" pin="GND"/>
@@
 <wire x1="254" y1="-22.86" x2="238.76" y2="-22.86" width="0.1524" layer="91"/>
 <junction x="254" y="-22.86"/>
-<pinref part="CONTROL" gate="G$1" pin="1"/>
-<wire x1="228.6" y1="-50.8" x2="238.76" y2="-50.8" width="0.1524" layer="91"/>
-<wire x1="238.76" y1="-50.8" x2="238.76" y2="-22.86" width="0.1524" layer="91"/>
+<pinref part="R2" gate="G$1" pin="2"/>
+<wire x1="238.76" y1="-30.48" x2="238.76" y2="-22.86" width="0.1524" layer="91"/>
 </segment>
 </net>
@@
 <wire x1="254" y1="-86.36" x2="241.3" y2="-86.36" width="0.1524" layer="91"/>
 <junction x="254" y="-86.36"/>
-<pinref part="CONTROL" gate="G$1" pin="2"/>
-<wire x1="228.6" y1="-53.34" x2="238.76" y2="-53.34" width="0.1524" layer="91"/>
-<wire x1="238.76" y1="-53.34" x2="238.76" y2="-86.36" width="0.1524" layer="91"/>
 <wire x1="238.76" y1="-86.36" x2="241.3" y2="-86.36" width="0.1524" layer="91"/>
+<pinref part="R12" gate="G$1" pin="1"/>
+<wire x1="238.76" y1="-71.12" x2="238.76" y2="-86.36" width="0.1524" layer="91"/>
 </segment>
 </net>
@@
 <wire x1="325.12" y1="38.1" x2="320.04" y2="38.1" width="0.1524" layer="91"/>
 <wire x1="320.04" y1="38.1" x2="320.04" y2="30.48" width="0.1524" layer="91"/>
-<pinref part="OVERLIGHT" gate="G$1" pin="1"/>
 <wire x1="320.04" y1="30.48" x2="320.04" y2="27.94" width="0.1524" layer="91"/>
-<wire x1="330.2" y1="25.4" x2="325.12" y2="25.4" width="0.1524" layer="91"/>
-<wire x1="325.12" y1="25.4" x2="325.12" y2="30.48" width="0.1524" layer="91"/>
-<wire x1="325.12" y1="30.48" x2="320.04" y2="30.48" width="0.1524" layer="91"/>
-<junction x="320.04" y="30.48"/>
 </segment>
 </net>
@@
 </segment>
 </net>
+<net name="N$13" class="0">
+<segment>
+<pinref part="CONTROL" gate="G$1" pin="1"/>
+<wire x1="228.6" y1="-50.8" x2="238.76" y2="-50.8" width="0.1524" layer="91"/>
+<pinref part="R2" gate="G$1" pin="1"/>
+<wire x1="238.76" y1="-50.8" x2="238.76" y2="-40.64" width="0.1524" layer="91"/>
+</segment>
+</net>
+<net name="N$18" class="0">
+<segment>
+<pinref part="CONTROL" gate="G$1" pin="2"/>
+<wire x1="228.6" y1="-53.34" x2="238.76" y2="-53.34" width="0.1524" layer="91"/>
+<pinref part="R12" gate="G$1" pin="2"/>
+<wire x1="238.76" y1="-53.34" x2="238.76" y2="-60.96" width="0.1524" layer="91"/>
+</segment>
+</net>

Commit message: !
Parts:
- removed 5V, CONTROL: (no value), pinhead:PINHD-1X2
- removed C11: 100n, Namenlos:CAP_0805
- removed D2: MBRA130LT3G, Namenlos:DIODE-SH_SMA
- removed L2: SCDS127T-221M-N, Namenlos:INDUCTOR0705
- removed R18, R19, R20: 1R, Namenlos:R_0805
- removed R21: 3K9, Namenlos:R_0805
- removed R22: 1K3, Namenlos:R_0805
- removed U$4: MC33063/MC34063D, adafruit:MC33063/MC34063D
- added D4: (no value), Namenlos:DIODE_ES1J
- added JP1: (no value), pinhead:PINHD-2X2
- added R13: 1R1, rcl:R-EU_R1206
- C8: value 470p -> (none)
- C9: value 220u 6.3V -> (none); device Namenlos:CAP-POL_D6 -> Namenlos:CAP_0805
- R3: value 1k -> 200R
- R4: value (none) -> 4k7; device Namenlos:R_POTTURN-X -> rcl:R-EU_R1206
- R8: value 1k2 -> 1R1
Connections:
- removed net N$32: C7.2, R4.A, R7.1
- removed net N$33: R4.E, R8.2
- removed net N$55: R18.2, R19.2, R20.2, U$4.DC, U$4.IPK, U$4.SWC
- removed net N$56: D2.C, L2.1, U$4.SWE
- removed net N$57: C8.1, U$4.TC
- removed net N$59: R21.1, R22.2, U$4.COMP
- new net N$28: D4.A, U$2.5
- net +12V: now also C9.1; no longer C6.+, R18.1, R19.1, R20.1, R3.2, R7.2, U$4.VCC
- net +5V: now also C6.+, C8.1, D4.C, JP1.2, R3.2, R7.2; no longer 5V.1, C11.1, C9.+, L2.2, R21.2
- net GND: now also C9.2, JP1.4, R4.1; no longer 5V.2, C11.2, C9.-, D2.A, R22.1, R8.1, U$4.GND
- net N$13: now also JP1.1; no longer CONTROL.1
- net N$18: now also JP1.3; no longer CONTROL.2
- net N$19: now also C7.2, R4.2, R7.1; no longer R4.S
- net N$4: now also R13.2, R8.2
- net N$5: now also R13.1, R8.1
Other:
- moved on the sheet: C5, C6, C8, R8
