File: 3DPrinter/TMC2208 OTP.sch (EAGLE design)
At the start: 3 parts

Commit message: TMC OTP
Parts:
- removed JP1: (no value), pinhead:PINHD-1X5/90
- added C1: 0u1, Namenlos:CAP_0805
- added C2: 1u, Namenlos:CAP_0805
- added ESD1: (no value), Namenlos:ESDAXXSC5
- added IC2: CP2101, Namenlos:CP2101
- added R2: 0, Namenlos:R_0805
- added X1: USB-MINIMICROMINI-SMD1, Namenlos:USB-MINIMICROMINI-SMD1
- R1: value (none) -> 1K; device Namenlos:R_1206 -> Namenlos:R_0805
Connections:
- new net N$1: C1.1, IC2.VDD
- new net N$4: IC2.D+, R2.2
- new net N$5: ESD1.C3, IC2.D-, X1G$1.D-
- new net N$6: ESD1.C2, R2.1, X1G$1.D+
- net +5V: now also C2.1, ESD1.C4, IC2.REGIN, IC2.VBUS, X1G$1.VCC; no longer JP1.2
- net GND: now also C1.2, C2.2, ESD1.A, IC2.GND, IC2.GND@EXP, IC2.GND@M, X1G$1.GND, X1S.S1; no longer JP1.5
- net N$2: now also IC2.TXD; no longer JP1.3
- net N$3: now also IC2.RXD; no longer JP1.4
Other:
- moved on the sheet: R1
