File: 3DPrinter/Driver Board.brd (EAGLE design)
At the start: 124.4 x 40.3 mm, 32 parts, among them X1 CON-7.62-02P, X2 CON-CP-04, X3 CON-CP-04, X4 CON-CP-04, X5 CON-CP-04, X6 CON-CP-04

Commit message: Так всем будет лучше
Parts:
- moved JP1 6.35 mm to (19.1, 72.4), turned to 270 degrees
Routing:
- net GND: track 392.4 -> 189.5 mm
- net +3V3: track 158.3 -> 153.7 mm, vias 10 -> 8
Changed lines of the file:
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@@
 <?xml version="1.0" encoding="utf-8"?>
 <!DOCTYPE eagle SYSTEM "eagle.dtd">
-<eagle version="8.3.0">
+<eagle version="8.4.0">
 <drawing>
 <settings>
@@
 <wire x1="124.44" y1="79.68" x2="0" y2="79.68" width="0" layer="20"/>
 <wire x1="0" y1="79.68" x2="0" y2="39.37" width="0" layer="20"/>
-<hole x="2.54" y="41.91" drill="3.2"/>
-<hole x="121.92" y="41.91" drill="3.2"/>
-<text x="7.62" y="57.15" size="1.778" layer="16" ratio="15" rot="MR0">+</text>
-<text x="11.43" y="73.66" size="1.778" layer="16" ratio="15" rot="MR0">+</text>
-<hole x="2.54" y="77.47" drill="3.2"/>
-<hole x="121.92" y="77.47" drill="3.2"/>
+<hole x="3.81" y="43.18" drill="3.2"/>
+<hole x="120.65" y="43.18" drill="3.2"/>
+<text x="8.89" y="54.61" size="1.778" layer="16" ratio="15" rot="MR0">+</text>
+<text x="16.891" y="72.898" size="1.778" layer="16" ratio="15" rot="MR0">+</text>
+<hole x="3.81" y="76.2" drill="3.2"/>
+<hole x="120.65" y="76.2" drill="3.2"/>
 </plain>
 <attributes>
@@
 <param name="dpMaxLengthDifference" value="10mm"/>
 <param name="dpGapFactor" value="2.5"/>
-<param name="checkGrid" value="0"/>
-<param name="checkAngle" value="0"/>
 <param name="checkFont" value="1"/>
 <param name="checkRestrict" value="1"/>
+<param name="checkStop" value="0"/>
 <param name="useDiameter" value="13"/>
 <param name="maxErrors" value="50"/>
@@
 <element name="IC5" library="Namenlos" package="DRV-BRK" value="" x="107.95" y="59.69"/>
 <element name="X1" library="Namenlos" package="KF25C-7.62-02P-13" value="CON-7.62-02P" x="8.89" y="64.77" rot="R90"/>
-<element name="JP1" library="pinhead" package="1X02" value="" x="13.97" y="76.2" rot="R90"/>
+<element name="JP1" library="pinhead" package="1X02" value="" x="19.05" y="72.39" rot="R270"/>
 <element name="JP2" library="pinhead" package="1X04" value="" x="31.75" y="45.72"/>
 <element name="JP3" library="pinhead" package="1X04" value="" x="52.07" y="45.72"/>
@@
 <contactref element="IC2" pad="P$15"/>
 <contactref element="IC1" pad="P$15"/>
-<wire x1="8.89" y1="68.58" x2="19.05" y2="68.58" width="1.016" layer="16"/>
-<wire x1="19.05" y1="68.58" x2="20.32" y2="67.31" width="1.016" layer="16"/>
-<wire x1="20.32" y1="67.31" x2="20.32" y2="66.04" width="1.016" layer="16"/>
-<wire x1="91.44" y1="77.47" x2="96.52" y2="77.47" width="1.016" layer="16"/>
-<wire x1="76.2" y1="77.47" x2="91.44" y2="77.47" width="1.016" layer="16"/>
-<wire x1="71.12" y1="77.47" x2="76.2" y2="77.47" width="1.016" layer="16"/>
-<wire x1="55.88" y1="77.47" x2="71.12" y2="77.47" width="1.016" layer="16"/>
-<wire x1="50.8" y1="77.47" x2="55.88" y2="77.47" width="1.016" layer="16"/>
-<wire x1="35.56" y1="77.47" x2="50.8" y2="77.47" width="1.016" layer="16"/>
-<wire x1="20.32" y1="77.47" x2="13.97" y2="77.47" width="1.016" layer="16"/>
-<wire x1="20.32" y1="77.47" x2="35.56" y2="77.47" width="1.016" layer="16"/>
-<wire x1="96.52" y1="77.47" x2="111.76" y2="77.47" width="1.016" layer="16"/>
-<wire x1="111.76" y1="77.47" x2="116.84" y2="72.39" width="1.016" layer="16"/>
-<wire x1="116.84" y1="72.39" x2="116.84" y2="66.04" width="1.016" layer="16"/>
-<wire x1="101.6" y1="66.04" x2="101.6" y2="72.39" width="1.016" layer="16"/>
-<wire x1="101.6" y1="72.39" x2="96.52" y2="77.47" width="1.016" layer="16"/>
-<wire x1="96.52" y1="66.04" x2="96.52" y2="72.39" width="1.016" layer="16"/>
-<wire x1="96.52" y1="72.39" x2="91.44" y2="77.47" width="1.016" layer="16"/>
-<wire x1="81.28" y1="66.04" x2="81.28" y2="72.39" width="1.016" layer="16"/>
-<wire x1="81.28" y1="72.39" x2="76.2" y2="77.47" width="1.016" layer="16"/>
-<wire x1="76.2" y1="66.04" x2="76.2" y2="72.39" width="1.016" layer="16"/>
-<wire x1="76.2" y1="72.39" x2="71.12" y2="77.47" width="1.016" layer="16"/>
-<wire x1="60.96" y1="66.04" x2="60.96" y2="72.39" width="1.016" layer="16"/>
-<wire x1="60.96" y1="72.39" x2="55.88" y2="77.47" width="1.016" layer="16"/>
-<wire x1="55.88" y1="66.04" x2="55.88" y2="72.39" width="1.016" layer="16"/>
-<wire x1="55.88" y1="72.39" x2="50.8" y2="77.47" width="1.016" layer="16"/>
-<wire x1="40.64" y1="70.163346875" x2="40.64" y2="66.04" width="1.016" layer="16"/>
-<wire x1="40.64" y1="70.163346875" x2="40.64" y2="72.39" width="1.016" layer="16"/>
-<wire x1="40.64" y1="72.39" x2="35.56" y2="77.47" width="1.016" layer="16"/>
 <wire x1="116.84" y1="45.72" x2="116.84" y2="43.18" width="1.27" layer="16"/>
 <wire x1="116.84" y1="43.18" x2="115.57" y2="41.91" width="1.27" layer="16"/>
@@
 <wire x1="3.81" y1="66.04" x2="6.35" y2="68.58" width="1.27" layer="16"/>
 <wire x1="6.35" y1="68.58" x2="8.89" y2="68.58" width="1.27" layer="16"/>
-<wire x1="20.32" y1="66.04" x2="20.32" y2="77.47" width="1.016" layer="16"/>
 <wire x1="35.56" y1="45.72" x2="35.56" y2="41.91" width="1.016" layer="16"/>
 <wire x1="55.88" y1="45.72" x2="55.88" y2="41.91" width="1.016" layer="16"/>
@@
 <vertex x="124.46" y="39.37"/>
 </polygon>
-<wire x1="35.56" y1="66.04" x2="35.56" y2="68.58" width="1.5" layer="16"/>
-<wire x1="35.56" y1="68.58" x2="36.83" y2="69.85" width="1.5" layer="16"/>
-<wire x1="36.83" y1="69.85" x2="40.326653125" y2="69.85" width="1.5" layer="16"/>
-<wire x1="40.326653125" y1="69.85" x2="40.64" y2="70.163346875" width="1.5" layer="16"/>
+<wire x1="20.32" y1="66.04" x2="20.32" y2="68.58" width="1.5" layer="16"/>
+<wire x1="20.32" y1="68.58" x2="19.05" y2="69.85" width="1.5" layer="16"/>
+<wire x1="35.56" y1="66.04" x2="35.56" y2="69.85" width="1.5" layer="16"/>
+<wire x1="40.64" y1="66.04" x2="40.64" y2="69.85" width="1.5" layer="16"/>
+<wire x1="55.88" y1="66.04" x2="55.88" y2="69.85" width="1.5" layer="16"/>
+<wire x1="60.96" y1="66.04" x2="60.96" y2="69.85" width="1.5" layer="16"/>
+<wire x1="76.2" y1="66.04" x2="76.2" y2="69.85" width="1.5" layer="16"/>
+<wire x1="81.28" y1="66.04" x2="81.28" y2="69.85" width="1.5" layer="16"/>
+<wire x1="96.52" y1="66.04" x2="96.52" y2="69.85" width="1.5" layer="16"/>
+<wire x1="101.6" y1="66.04" x2="101.6" y2="69.85" width="1.5" layer="16"/>
+<wire x1="35.56" y1="69.85" x2="36.83" y2="69.85" width="1.5" layer="16"/>
 </signal>
 <signal name="+3V3">
@@
 <contactref element="IC2" pad="P$10"/>
 <contactref element="IC1" pad="P$10"/>
-<wire x1="13.97" y1="74.93" x2="17.78" y2="74.93" width="1.5" layer="16"/>
-<via x="17.78" y="74.93" extent="1-16" drill="0.6" diameter="0.9"/>
-<wire x1="17.78" y1="74.93" x2="22.86" y2="74.93" width="1.5" layer="1"/>
-<via x="22.86" y="74.93" extent="1-16" drill="0.6" diameter="0.9"/>
-<wire x1="22.86" y1="74.93" x2="30.48" y2="74.93" width="1.5" layer="16"/>
-<wire x1="30.48" y1="74.93" x2="33.02" y2="72.39" width="1.5" layer="16"/>
+<wire x1="33.02" y1="72.39" x2="30.48" y2="74.93" width="1.5" layer="16"/>
 <wire x1="33.02" y1="72.39" x2="33.02" y2="66.04" width="1.5" layer="16"/>
 <wire x1="33.02" y1="66.04" x2="33.02" y2="63.5" width="1.5" layer="16"/>
@@
 <wire x1="104.14" y1="58.325" x2="104.14" y2="58.42" width="0.8128" layer="16"/>
 <wire x1="106.68" y1="58.325" x2="106.68" y2="58.42" width="0.8128" layer="16"/>
+<wire x1="30.48" y1="74.93" x2="20.32" y2="74.93" width="1.5" layer="16"/>
+<wire x1="20.32" y1="74.93" x2="19.05" y2="73.66" width="1.5" layer="16"/>
 </signal>
 <signal name="+24V">

Commit message: SMPS
Parts:
- added C1: 200p, Namenlos:C0805
- added C2: 68p, Namenlos:C0805
- added C3: (no value), Namenlos:E3,5-8
- added D1: (no value), Namenlos:DO214AC
- added JP7: (no value), pinhead:2X02
- added L1: (no value), Namenlos:CW68
- added R16, R17, R18: 1R, Namenlos:R0805
- added R19: 1K5, Namenlos:R0805
- added R20: 13K, Namenlos:R0805
- added U$1: MC33063/MC34063P, adafruit:DIL08
- X2, X3, X4, X5, X6: value CON-CP-04 -> CON-XH-04; device Namenlos:CON-CT-04 -> Namenlos:XH-04
- moved X1 6.35 mm to (12.7, 69.8)
- moved X4 3.86 mm to (71.1, 71.8)
- moved X5 3.86 mm to (91.4, 71.8)
- moved X6 3.86 mm to (111.8, 71.8)
- moved X2 3.86 mm to (30.5, 71.8)
- moved X3 3.86 mm to (50.8, 71.8)
- moved IC3 3.81 mm to (71.1, 59.7)
- moved IC4 3.81 mm to (91.4, 59.7)
- moved IC5 3.81 mm to (111.8, 59.7)
- moved R10 3.81 mm to (85.1, 57.1)
- moved R11 3.81 mm to (87.6, 57.1)
- moved R12 3.81 mm to (90.2, 57.1)
- moved R13 3.81 mm to (105.4, 57.1)
- moved R14 3.81 mm to (108.0, 57.1)
- moved R2 3.81 mm to (26.7, 57.1)
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Connections:
- new net +12V: C3.+, JP7.1, JP7.2, L1.P$2, R20.2
- new net N$51: C1.1, C2.1, U$1.3
- new net N$52: R16.1, R17.1, R18.1, U$1.1, U$1.7, U$1.8
- new net N$54: D1.C, L1.P$1, U$1.2
- new net N$55: R19.1, R20.1, U$1.5
- net +24V: now also R16.2, R17.2, R18.2, U$1.6
- net GND: now also C1.2, C2.2, C3.-, D1.A, JP7.3, JP7.4, R19.2, U$1.4
Routing:
- net GND: track 189.5 -> 125.8 mm, vias 0 -> 2
- net +12V: track 0.00 -> 28.0 mm
- net +24V: track 116.9 -> 134.7 mm
- net N$54: track 0.00 -> 13.2 mm
- net N$52: track 0.00 -> 10.8 mm
- net N$55: track 0.00 -> 10.0 mm
- net N$51: track 0.00 -> 4.75 mm
- net N$16: track 14.8 -> 10.3 mm
- net N$20: track 14.8 -> 10.3 mm
- net N$1: track 14.8 -> 10.3 mm
- net N$7: track 14.8 -> 10.3 mm
- net N$11: track 14.8 -> 10.3 mm
- net N$18: track 8.67 -> 12.5 mm
- net N$14: track 8.67 -> 12.5 mm
- net N$9: track 8.67 -> 12.5 mm
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
Commit message: более универсально
Parts:
- removed R1, R10, R11, R12, R13, R14, R15, R2, R3, R4, R5, R6, R7, R8, R9: (no value), Namenlos:R0805
- added JP10, JP11, JP12, JP8, JP9: (no value), pinhead:1X02
- added S1, S2, S3, S4, S5: (no value), Namenlos:DIP03YL
- moved JP5 5.68 mm to (97.8, 48.3)
- moved JP2 5.68 mm to (36.8, 48.3)
- moved JP3 5.68 mm to (57.1, 48.3)
- moved JP4 5.68 mm to (77.5, 48.3)
- moved JP6 5.68 mm to (118.1, 48.3)
Connections:
- new net N$53: IC4.P$3, S4.5
- new net N$56: IC4.P$2, S4.6
- new net N$57: IC5.P$4, S5.4
- new net N$58: IC5.P$3, S5.5
- new net N$59: IC5.P$2, S5.6
- net +3V3: now also JP10.2, JP11.2, JP12.2, JP8.2, JP9.2, S1.1, S1.2, S1.3, S2.1, S2.2, S2.3, S3.1, S3.2, S3.3, S4.1, S4.2, S4.3, S5.1, S5.2, S5.3; no longer R1.1, R10.1, R11.1, R12.1, R13.1, R14.1, R15.1, R2.1, R3.1, R4.1, R5.1, R6.1, R7.1, R8.1, R9.1
- net N$36: now also IC1.P$4, S1.4; no longer IC1.P$2, R1.2
- net N$37: now also S1.5; no longer R2.2
- net N$38: now also IC1.P$2, S1.6; no longer IC1.P$4, R3.2
- net N$39: now also IC5.P$5, IC5.P$6, JP12.1; no longer IC2.P$2, R4.2
- net N$40: now also IC4.P$5, IC4.P$6, JP11.1; no longer IC2.P$3, R5.2
- net N$41: now also IC3.P$5, IC3.P$6, JP10.1; no longer IC2.P$4, R6.2
- net N$42: now also IC2.P$5, IC2.P$6, JP9.1; no longer IC3.P$2, R7.2
- net N$43: now also IC1.P$5, IC1.P$6, JP8.1; no longer IC3.P$3, R8.2
- net N$44: now also IC2.P$4, S2.4; no longer IC3.P$4, R9.2
- net N$45: now also IC2.P$3, S2.5; no longer IC4.P$2, R10.2
- net N$46: now also IC2.P$2, S2.6; no longer IC4.P$3, R11.2
- net N$47: now also IC3.P$4, S3.4; no longer IC4.P$4, R12.2
- net N$48: now also IC3.P$3, S3.5; no longer IC5.P$2, R13.2
- net N$49: now also IC3.P$2, S3.6; no longer IC5.P$3, R14.2
- net N$50: now also IC4.P$4, S4.4; no longer IC5.P$4, R15.2
Routing:
- net +3V3: track 155.7 -> 289.8 mm
- net GND: track 125.8 -> 243.1 mm
- net N$41: track 2.63 -> 13.2 mm
- net N$40: track 2.63 -> 13.2 mm
- net N$43: track 2.63 -> 13.2 mm
- net N$42: track 2.63 -> 13.2 mm
- net N$39: track 2.63 -> 13.2 mm
- net N$20: track 10.3 -> 17.6 mm
- net N$11: track 10.3 -> 17.6 mm
- net N$16: track 10.3 -> 17.6 mm
- net N$7: track 10.3 -> 17.2 mm
- net N$1: track 10.3 -> 17.2 mm
- net N$5: track 12.5 -> 5.61 mm
- net N$3: track 12.5 -> 5.61 mm
- net N$18: track 12.5 -> 5.61 mm
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Other:
- board size 124.4 x 40.3 mm -> 127.6 x 42.2 mm
