File: Power/Charger Li-Ion/Charger_18V-1.35A_СС.sch (EAGLE design)
At the start: 20 parts, among them Q1 STP11NM60ND, T1 TRANS-1/1EFD20

Commit message: Added some info
Parts:
- U$1: value NCP1216D100 -> NCP1200D60
Other:
- note added: "4.5V 0.75A 1 - 121 Turns 0,2x1 2 - 8 Turns 0.56x1 Gap - 0.06 - 6.455 mH R - 5.736 Omh"
- note removed: "1 - 60 Turns 0,355x1 2 - 9 Turns 0.56x2 Gap - 0.24 / 2"
Changed lines of the file:
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@@
 <grid distance="0.1" unitdist="inch" unit="inch" style="lines" multiple="1" display="no" altdistance="0.01" altunitdist="inch" altunit="inch"/>
 <layers>
-<layer number="1" name="Top" color="4" fill="1" visible="yes" active="no"/>
-<layer number="2" name="Route2" color="1" fill="3" visible="yes" active="no"/>
-<layer number="3" name="Route3" color="4" fill="3" visible="yes" active="no"/>
-<layer number="4" name="Route4" color="1" fill="4" visible="yes" active="no"/>
-<layer number="5" name="Route5" color="4" fill="4" visible="yes" active="no"/>
-<layer number="6" name="Route6" color="1" fill="8" visible="yes" active="no"/>
-<layer number="7" name="Route7" color="4" fill="8" visible="yes" active="no"/>
-<layer number="8" name="Route8" color="1" fill="2" visible="yes" active="no"/>
-<layer number="9" name="Route9" color="4" fill="2" visible="yes" active="no"/>
-<layer number="10" name="Route10" color="1" fill="7" visible="yes" active="no"/>
-<layer number="11" name="Route11" color="4" fill="7" visible="yes" active="no"/>
-<layer number="12" name="Route12" color="1" fill="5" visible="yes" active="no"/>
-<layer number="13" name="Route13" color="4" fill="5" visible="yes" active="no"/>
-<layer number="14" name="Route14" color="1" fill="6" visible="yes" active="no"/>
-<layer number="15" name="Route15" color="4" fill="6" visible="yes" active="no"/>
-<layer number="16" name="Bottom" color="1" fill="1" visible="yes" active="no"/>
-<layer number="17" name="Pads" color="2" fill="1" visible="yes" active="no"/>
-<layer number="18" name="Vias" color="2" fill="1" visible="yes" active="no"/>
-<layer number="19" name="Unrouted" color="6" fill="1" visible="yes" active="no"/>
-<layer number="20" name="Dimension" color="15" fill="1" visible="yes" active="no"/>
-<layer number="21" name="tPlace" color="7" fill="1" visible="yes" active="no"/>
-<layer number="22" name="bPlace" color="7" fill="1" visible="yes" active="no"/>
-<layer number="23" name="tOrigins" color="15" fill="1" visible="yes" active="no"/>
-<layer number="24" name="bOrigins" color="15" fill="1" visible="yes" active="no"/>
-<layer number="25" name="tNames" color="7" fill="1" visible="yes" active="no"/>
-<layer number="26" name="bNames" color="7" fill="1" visible="yes" active="no"/>
-<layer number="27" name="tValues" color="7" fill="1" visible="yes" active="no"/>
-<layer number="28" name="bValues" color="7" fill="1" visible="yes" active="no"/>
+<layer number="1" name="Top" color="4" fill="1" visible="no" active="no"/>
+<layer number="2" name="Route2" color="1" fill="3" visible="no" active="no"/>
+<layer number="3" name="Route3" color="4" fill="3" visible="no" active="no"/>
+<layer number="4" name="Route4" color="1" fill="4" visible="no" active="no"/>
+<layer number="5" name="Route5" color="4" fill="4" visible="no" active="no"/>
+<layer number="6" name="Route6" color="1" fill="8" visible="no" active="no"/>
+<layer number="7" name="Route7" color="4" fill="8" visible="no" active="no"/>
+<layer number="8" name="Route8" color="1" fill="2" visible="no" active="no"/>
+<layer number="9" name="Route9" color="4" fill="2" visible="no" active="no"/>
+<layer number="10" name="Route10" color="1" fill="7" visible="no" active="no"/>
+<layer number="11" name="Route11" color="4" fill="7" visible="no" active="no"/>
+<layer number="12" name="Route12" color="1" fill="5" visible="no" active="no"/>
+<layer number="13" name="Route13" color="4" fill="5" visible="no" active="no"/>
+<layer number="14" name="Route14" color="1" fill="6" visible="no" active="no"/>
+<layer number="15" name="Route15" color="4" fill="6" visible="no" active="no"/>
+<layer number="16" name="Bottom" color="1" fill="1" visible="no" active="no"/>
+<layer number="17" name="Pads" color="2" fill="1" visible="no" active="no"/>
+<layer number="18" name="Vias" color="2" fill="1" visible="no" active="no"/>
+<layer number="19" name="Unrouted" color="6" fill="1" visible="no" active="no"/>
+<layer number="20" name="Dimension" color="15" fill="1" visible="no" active="no"/>
+<layer number="21" name="tPlace" color="7" fill="1" visible="no" active="no"/>
+<layer number="22" name="bPlace" color="7" fill="1" visible="no" active="no"/>
+<layer number="23" name="tOrigins" color="15" fill="1" visible="no" active="no"/>
+<layer number="24" name="bOrigins" color="15" fill="1" visible="no" active="no"/>
+<layer number="25" name="tNames" color="7" fill="1" visible="no" active="no"/>
+<layer number="26" name="bNames" color="7" fill="1" visible="no" active="no"/>
+<layer number="27" name="tValues" color="7" fill="1" visible="no" active="no"/>
+<layer number="28" name="bValues" color="7" fill="1" visible="no" active="no"/>
 <layer number="29" name="tStop" color="7" fill="3" visible="no" active="no"/>
 <layer number="30" name="bStop" color="7" fill="6" visible="no" active="no"/>
@@
 <layer number="35" name="tGlue" color="7" fill="4" visible="no" active="no"/>
 <layer number="36" name="bGlue" color="7" fill="5" visible="no" active="no"/>
-<layer number="37" name="tTest" color="7" fill="1" visible="yes" active="no"/>
-<layer number="38" name="bTest" color="7" fill="1" visible="yes" active="no"/>
+<layer number="37" name="tTest" color="7" fill="1" visible="no" active="no"/>
+<layer number="38" name="bTest" color="7" fill="1" visible="no" active="no"/>
 <layer number="39" name="tKeepout" color="4" fill="11" visible="no" active="no"/>
 <layer number="40" name="bKeepout" color="1" fill="11" visible="no" active="no"/>
@@
 <layer number="44" name="Drills" color="7" fill="1" visible="no" active="no"/>
 <layer number="45" name="Holes" color="7" fill="1" visible="no" active="no"/>
-<layer number="46" name="Milling" color="3" fill="1" visible="yes" active="no"/>
-<layer number="47" name="Measures" color="7" fill="1" visible="yes" active="no"/>
-<layer number="48" name="Document" color="7" fill="1" visible="yes" active="no"/>
-<layer number="49" name="Reference" color="7" fill="1" visible="yes" active="no"/>
-<layer number="50" name="dxf" color="7" fill="1" visible="yes" active="no"/>
-<layer number="51" name="tDocu" color="7" fill="1" visible="yes" active="no"/>
-<layer number="52" name="bDocu" color="7" fill="1" visible="yes" active="no"/>
-<layer number="53" name="tGND_GNDA" color="7" fill="9" visible="yes" active="no"/>
-<layer number="54" name="bGND_GNDA" color="1" fill="9" visible="yes" active="no"/>
-<layer number="56" name="wert" color="7" fill="1" visible="yes" active="no"/>
-<layer number="57" name="tCAD" color="7" fill="1" visible="yes" active="no"/>
-<layer number="58" name="bCopper" color="7" fill="1" visible="yes" active="no"/>
-<layer number="59" name="tCarbon" color="7" fill="1" visible="yes" active="no"/>
-<layer number="60" name="bCarbon" color="7" fill="1" visible="yes" active="no"/>
+<layer number="46" name="Milling" color="3" fill="1" visible="no" active="no"/>
+<layer number="47" name="Measures" color="7" fill="1" visible="no" active="no"/>
+<layer number="48" name="Document" color="7" fill="1" visible="no" active="no"/>
+<layer number="49" name="Reference" color="7" fill="1" visible="no" active="no"/>
+<layer number="50" name="dxf" color="7" fill="1" visible="no" active="no"/>
+<layer number="51" name="tDocu" color="7" fill="1" visible="no" active="no"/>
+<layer number="52" name="bDocu" color="7" fill="1" visible="no" active="no"/>
+<layer number="53" name="tGND_GNDA" color="7" fill="9" visible="no" active="no"/>
+<layer number="54" name="bGND_GNDA" color="1" fill="9" visible="no" active="no"/>
+<layer number="56" name="wert" color="7" fill="1" visible="no" active="no"/>
+<layer number="57" name="tCAD" color="7" fill="1" visible="no" active="no"/>
+<layer number="58" name="bCopper" color="7" fill="1" visible="no" active="no"/>
+<layer number="59" name="tCarbon" color="7" fill="1" visible="no" active="no"/>
+<layer number="60" name="bCarbon" color="7" fill="1" visible="no" active="no"/>
 <layer number="90" name="Modules" color="5" fill="1" visible="yes" active="yes"/>
 <layer number="91" name="Nets" color="2" fill="1" visible="yes" active="yes"/>
@@
 <part name="NTC" library="rcl" deviceset="R-US_" device="0207/7"/>
 <part name="C1" library="rcl" deviceset="CPOL-EU" device="E7.5-18" value="22u 400V"/>
-<part name="U$1" library="NCP1200" deviceset="NCP1200-100" device="DIL" value="NCP1216D100"/>
+<part name="U$1" library="NCP1200" deviceset="NCP1200-100" device="DIL" value="NCP1200D60"/>
 <part name="P6KE200" library="Namenlos" deviceset="SUPRESSOR" device="DO-204AC"/>
 <part name="D1" library="diode" deviceset="DIODE-" device="DO-214AC" value="ES1J"/>
@@
 <sheet>
 <plain>
-<text x="66.04" y="73.66" size="1.778" layer="97">1 - 60 Turns 0,355x1
-2 - 9 Turns 0.56x2
-Gap - 0.24 / 2</text>
+<text x="66.04" y="73.66" size="1.778" layer="97">4.5V 0.75A
+1 - 121 Turns 0,2x1
+2 - 8 Turns 0.56x1
+Gap - 0.06 - 6.455 mH
+R - 5.736 Omh</text>
 </plain>
 <instances>

Commit message: DO NOT
Parts:
- removed R19: 1R3, rcl:R-EU_0309/12
- added OP1: TSV6394AIPT, Namenlos:OP-AMP-4LMV324IPT
- added TL1: TLV431ACDBZR, Namenlos:IC-TL431CDBZR
Connections:
- net N$12: no longer R19.2
- net N$16: no longer R19.1
Changed lines of the file:
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@@
 <part name="R18" library="rcl" deviceset="R-EU_" device="R1206" value="0"/>
 <part name="CY1" library="rcl" deviceset="CY" device="YC10B4"/>
-<part name="R19" library="rcl" deviceset="R-EU_" device="0309/12" value="1R3"/>
 <part name="1" library="wirepad" deviceset="3,81/1,4" device=""/>
 <part name="2" library="wirepad" deviceset="3,81/1,4" device=""/>
@@
 <part name="B1" library="Namenlos" deviceset="BRIDGE" device="DBS"/>
 <part name="T1" library="Namenlos" deviceset="TRANS-1/1" device="EFD20"/>
+<part name="OP1" library="Namenlos" deviceset="OP-AMP-4" device="LMV324IPT" value="TSV6394AIPT"/>
+<part name="TL1" library="Namenlos" deviceset="IC-TL431" device="CDBZR" value="TLV431ACDBZR"/>
 </parts>
 <sheets>
@@
 <instance part="R18" gate="G$1" x="15.24" y="-10.16"/>
 <instance part="CY1" gate="G$1" x="83.82" y="30.48" rot="R90"/>
-<instance part="R19" gate="G$1" x="63.5" y="-33.02" rot="R90"/>
 <instance part="1" gate="1" x="0" y="50.8"/>
 <instance part="2" gate="1" x="0" y="40.64"/>
@@
 <instance part="B1" gate="1" x="7.62" y="50.8" rot="R90"/>
 <instance part="T1" gate="G$1" x="78.74" y="60.96" rot="MR180"/>
+<instance part="OP1" gate="A" x="160.02" y="10.16"/>
+<instance part="OP1" gate="PW" x="160.02" y="10.16"/>
+<instance part="OP1" gate="B" x="193.04" y="10.16"/>
+<instance part="OP1" gate="C" x="223.52" y="10.16"/>
+<instance part="TL1" gate="G$1" x="139.7" y="-15.24" rot="MR90"/>
 </instances>
 <busses>
@@
 <wire x1="17.78" y1="-20.32" x2="63.5" y2="-20.32" width="0.1524" layer="91"/>
 <junction x="71.12" y="-20.32"/>
-<pinref part="R19" gate="G$1" pin="2"/>
 <wire x1="63.5" y1="-20.32" x2="71.12" y2="-20.32" width="0.1524" layer="91"/>
-<wire x1="63.5" y1="-27.94" x2="63.5" y2="-20.32" width="0.1524" layer="91"/>
-<junction x="63.5" y="-20.32"/>
 </segment>
 </net>
@@
 <wire x1="81.28" y1="30.48" x2="38.1" y2="30.48" width="0.1524" layer="91"/>
 <junction x="38.1" y="30.48"/>
-<pinref part="R19" gate="G$1" pin="1"/>
-<wire x1="63.5" y1="-38.1" x2="63.5" y2="-45.72" width="0.1524" layer="91"/>
-<junction x="63.5" y="-45.72"/>
 <wire x1="20.32" y1="43.18" x2="33.02" y2="43.18" width="0.1524" layer="91"/>
 <junction x="33.02" y="43.18"/>
