File: MicroControl/KitchenTimer/KitchenTimer.brd (EAGLE design)
At the start: 79.1 x 22.4 mm, 33 parts, among them IC1 STM8L151X4/6G6U6, P1 BATTERY18650X1, SW1 BUTTON1212, U1 POWER-STC4054, U2 TPS73130DBVT, X1 USB-MINIMICROMICRO, X2 STM-SWIMPOGOPADS

Commit message: _
Parts:
- added R16: 20K, Flamberm:RESC3216X60
- added SW2: SW-200D, Flamberm:SW-200D
- C1, C2, C3: value 470n -> 330n
- R13: value (none) -> 3K3
- R14: value (none) -> 20K
- R15: value (none) -> 27R
- VT1, VT2, VT3: device Flamberm:SOT23 -> Flamberm:SOT95P240X115-3
- turned VT1 to 180 degrees
- turned VT2 to 270 degrees
- turned VT3 to 0 degrees
Connections:
- new net VIBRO: IC1.25, R16.1, SW2.G
- net +3V: now also R16.2
- net GND: now also SW2.S
Routing:
- net VIBRO: track 0.00 -> 18.6 mm
- net GND: track 189.0 -> 183.5 mm
- net N$21: track 15.1 -> 13.2 mm
- net +3V: track 73.9 -> 75.6 mm
