File: Monitors/Samsung 23/PowerBoard.sch (EAGLE design)
At the start: 6 parts, among them X1 CON-MONPANEL, X2 CON-2MM-14P

Commit message: _
Connections:
- new net 15V: X2.2
- new net BL-ANALOG: X2.8
- new net BL-PWM: X2.1
- new net ON-OFF: X2.9
Changed lines of the file:
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@@
+</segment>
+</net>
+<net name="BL-PWM" class="0">
+<segment>
+<pinref part="X2" gate="G$1" pin="1"/>
+<wire x1="5.08" y1="45.72" x2="33.02" y2="45.72" width="0.1524" layer="91"/>
+<label x="22.86" y="45.72" size="1.778" layer="95"/>
+</segment>
+</net>
+<net name="15V" class="0">
+<segment>
+<pinref part="X2" gate="G$1" pin="2"/>
+<wire x1="5.08" y1="43.18" x2="33.02" y2="43.18" width="0.1524" layer="91"/>
+<label x="22.86" y="43.18" size="1.778" layer="95"/>
+</segment>
+</net>
+<net name="BL-ANALOG" class="0">
+<segment>
+<pinref part="X2" gate="G$1" pin="8"/>
+<wire x1="5.08" y1="27.94" x2="33.02" y2="27.94" width="0.1524" layer="91"/>
+<label x="22.86" y="27.94" size="1.778" layer="95"/>
+</segment>
+</net>
+<net name="ON-OFF" class="0">
+<segment>
+<pinref part="X2" gate="G$1" pin="9"/>
+<wire x1="5.08" y1="25.4" x2="33.02" y2="25.4" width="0.1524" layer="91"/>
+<label x="22.86" y="25.4" size="1.778" layer="95"/>
 </segment>
 </net>

Commit message: The Begining
Parts:
- added B2: (no value), Flamberm:BRIDGEDBS
- added C4: 400v 22u, Namenlos:CAP-POL_E3.5-8
- added C6: 22u 16V, Namenlos:CAP-POL_3528
- added D1: ES1J, Flamberm:DIODE_ES1J
- added IC2: HV9961NG-G, Flamberm:HV9910BNG
- added L2: SL1016T, Namenlos:INDUCTORSL1016
- added OK1, OK2: (no value), Flamberm:OPTOTRANSPC817
- added PAD10, PAD11, PAD12, PAD5, PAD6, PAD7, PAD8, PAD9: (no value), wirepad:2,54/1,1
- added R1, R9: 39K, Flamberm:R_R0805
- added R10: (no value), Flamberm:R_POT3296X
- added R2, R3: 2K, Flamberm:R_R0805
- added R4: 160K, Flamberm:R_MF-0125
- added R6: 68K, Flamberm:R_R0805
- added R8: 1R1, Flamberm:R_MF-05
- added VT2: STD1NK60T4, Namenlos:FET-NDPAK
Connections:
- new net AC1: B2.AC1
- new net AC2: B2.AC2
- new net LED+: B2.+, C4.+, D1.C, IC2.VIN, PAD11.P, PAD5.P, PAD7.P, PAD9.P, R4.2
- new net LED-: L2.2, PAD10.P, PAD12.P, PAD6.P, PAD8.P
- new net N$10: IC2.RT, R6.1
- new net N$11: IC2.GATE, VT2.G
- new net N$18: D1.A, L2.1, VT2.D
- new net N$24: IC2.CS, R8.2, VT2.S
- new net N$25: B2.-, C4.-, C6.-, IC2.GND, R1.1, R10.A, R4.1, R6.2, R8.1
- new net N$26: C6.+, IC2.LD, R10.S
- new net N$27: R10.E, R9.2
- new net N$29: IC2.VDD, OK1.COL, R9.1
- new net N$6: OK1.EMIT, OK2.COL
- new net N$7: IC2.PWMD, OK2.EMIT, R1.2
- new net N$8: OK1.C, R3.1
- new net N$9: OK2.C, R2.1
- net BL-PWM: now also OK2.A
- net GND: now also R2.2, R3.2
- net ON-OFF: now also OK1.A
Other:
- note added: "C3 - SoftStart JP1 - POT 10K JP2 - Close-ON, Open-OFF"

Commit message: Почти
Parts:
- removed OK2: (no value), Flamberm:OPTOTRANSPC817
- added B1: (no value), rectifier:KBL
- added C1: 100u, Flamberm:CAP-POL_E5-13-35-H
- added C10: (no value), Flamberm:CAP_0805
- added C2: 1n, Namenlos:CAP_C50-024X044
- added C3: 22u 16V, Namenlos:CAP-POL_E2.5-7
- added C5, C8: 100n, Flamberm:CAP_1206
- added C7, C9: 1000u 6.3V, Flamberm:CAP-POL_E3.5-8
- added CX1: 470n 275V, rcl:CXXC15B10
- added CX2: 100n 275V, rcl:CXXC15B6
- added D2: (no value), Flamberm:DIODE_ES1J
- added D3: (no value), Flamberm:DIODE_TO-220-2
- added F1: FUSETR5, fuse:FUSETR5
- added L1: MFE, inductors:MFE
- added NTC: NTC-D12, Namenlos:NTC-D12
- added OK3: ILD621, optocoupler:ILD621
- added P6KE200: (no value), Flamberm:SUPRESSORDO-204AC
- added Q1: (no value), Namenlos:FET-NTO-220
- added R11, R18: 3k3, Flamberm:R_R1206
- added R12: 160K, Namenlos:R_MF-0125
- added R13, R14: 2R2, Flamberm:R_MF-025
- added R5: 51k, Flamberm:R_SQP-5
- added R7: 220R, Flamberm:R_R1206
- added T1: TRANS-1/1EFD25-10, Flamberm:TRANS-1/1EFD25-10
- added U$1: PW-NCP12NCP1200D, Namenlos:PW-NCP12NCP1200D
- added U$3: IC-TL431DBV, Flamberm:IC-TL431DBV
- OK1: device Flamberm:OPTOTRANSPC817 -> Namenlos:OPTOTRANSPC817
- R2, R3: value 2K -> 1K5; device Flamberm:R_R0805 -> Flamberm:R_MF-025
Connections:
- new net N$12: NTC.2, PAD1.P
- new net N$13: B1.+, C1.+, P6KE200.A, R12.2, R5.2, T1.P1-2
- new net N$14: D2.A, Q1.D, T1.P1-1
- new net N$15: R5.1, U$1.HV
- new net N$16: C3.+, U$1.VCC
- new net N$17: C5.1, OK1.COL, U$1.FB
- new net N$19: D2.C, P6KE200.C
- new net N$20: F1.1, PAD2.P
- new net N$21: OK1.A, R7.1
- new net N$22: Q1.G, U$1.DRV
- new net N$23: C8.2, R11.1, R18.2, U$3.R
- new net N$30: B1.-, C1.-, C2.1, C3.-, C5.2, OK1.EMIT, R12.1, R13.1, R14.1, U$1.ADJ, U$1.GND
- new net N$31: C8.1, OK1.C, U$3.C
- new net N$33: Q1.S, R13.2, R14.2, U$1.CS
- new net N$35: CX1.1, L1.3, NTC.1
- new net N$36: CX1.2, F1.2, L1.1
- new net N$38: L1.2, PAD3.P
- new net N$41: D3.A, T1.S1-1
- net +5V: now also C10.1, C7.+, C9.+, D3.C, R11.2, R7.2
- net AC1: now also B1.AC1, CX2.2, PAD4.P
- net AC2: now also B1.AC2, CX2.1, L1.4
- net BL-PWM: now also R2.1; no longer OK2.A
- net GND: now also C10.2, C2.2, C7.-, C9.-, OK3A.C, OK3B.C, R18.1, T1.S1-2, U$3.A; no longer R2.2, R3.2
- net N$29: now also OK3A.COL; no longer OK1.COL
- net N$6: now also OK3A.EMIT, OK3B.COL; no longer OK1.EMIT, OK2.COL
- net N$7: now also OK3B.EMIT; no longer OK2.EMIT
- net N$8: now also OK3A.A; no longer OK1.C
- net N$9: now also OK3B.A, R2.2; no longer OK2.C, R2.1
- net ON-OFF: now also R3.2; no longer OK1.A
Other:
- note added: "Pri: 65 turns, 1x0.355mm Sec: 3 turns, 8x0.355mm Prim. Ind.= 1,3 mH"
