File: Monitors/Samsung 743n/PowerBoard.brd (EAGLE design)
At the start: 160 x 128 mm, 59 parts, among them IC2 HV9961NG-G, T1 TRANS-1/1EFD25-10, X1 CON-MONPANEL, X2 CON-2MM-12P

Commit message: Понемногу
Parts:
- L2: value SL1016T -> SL1016T-123K
- R6: value 68K -> 75K
- R8: value 1R1 -> 2R2
- U$1: value PW-NCP12NCP1200D -> POWER-NCP12DIP; device Namenlos:SO8 -> Flamberm:DIP-8
- moved D2 30.7 mm to (146.7, 68.6), turned to 270 degrees
- moved P6KE200 25.0 mm to (147.6, 81.0), turned to 90 degrees
- moved C5 12.1 mm to (109.2, 63.5)
- moved OK1 12.1 mm to (109.2, 70.8)
- moved C2 10.4 mm to (113.3, 72.7)
- moved T1 10.2 mm to (130.8, 76.5), turned to 180 degrees
- moved C3 8.11 mm to (109.2, 51.8), turned to 180 degrees
- moved CX2 5.41 mm to (83.5, 57.1)
- moved NTC 4.32 mm to (74.6, 17.9), turned to 0 degrees
- moved D3 4.07 mm to (134.6, 102.6)
- moved U$4 4.07 mm to (134.6, 102.6)
- moved C7 4.07 mm to (119.4, 100.6)
- moved C8 4.07 mm to (106.4, 94.3)
- moved R11 4.07 mm to (110.5, 96.2)
- moved R18 4.07 mm to (110.5, 91.4)
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Routing:
- net AC1: track 178.0 -> 111.6 mm
- net GND: track 493.1 -> 451.5 mm
- net N$14: track 48.9 -> 26.1 mm
- net N$13: track 100.0 -> 113.0 mm
- net N$17: track 29.6 -> 17.1 mm
- net N$20: track 0.00 -> 10.9 mm
- net AC2: track 113.7 -> 103.4 mm
- net N$21: track 4.51 -> 13.6 mm
- net N$31: track 14.1 -> 23.2 mm
- net N$41: track 9.74 -> 0.67 mm
- net N$12: track 1.58 -> 10.1 mm
- net N$30: track 187.1 -> 179.9 mm
- net N$35: track 16.6 -> 23.1 mm
- net N$36: track 13.5 -> 16.7 mm
- net N$16: track 9.37 -> 10.9 mm
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
Commit message: почти
Parts:
- added C11: 10u 16V, Flamberm:E2,5-7
- C2: device Namenlos:C050-024X044 -> Flamberm:C050-024X044
- C3: device Namenlos:E2,5-7 -> Flamberm:E2,5-7
- C4: device Namenlos:E3,5-8 -> Flamberm:E5-13,5
- C6: value 22u 16V -> 10u 16V; device Namenlos:CT3528 -> Flamberm:E2,5-7
- L2: device Namenlos:SL1016 -> Flamberm:SL1016
- NTC: device Namenlos:NTC-D12 -> Flamberm:NTC-D12
- OK1: device Namenlos:DIL04 -> Flamberm:DIL04
- Q1: device Namenlos:TO-220V -> Flamberm:TO-220V
- R12: device Namenlos:MF-0125 -> Flamberm:MF-0125
- VT2: device Namenlos:DPAK -> Flamberm:DPAK
- moved R12 34.6 mm to (113.0, 26.7)
- moved C10 20.9 mm to (139.1, 111.8), turned to 90 degrees
- moved C6 11.2 mm to (44.5, 65.1), flipped to the top, turned to 0 degrees
- moved C7 10.4 mm to (129.5, 102.9)
- moved C9 10.4 mm to (129.5, 111.1)
- moved R11 6.30 mm to (114.6, 101.0)
- moved R18 6.30 mm to (114.6, 96.2)
- moved C8 6.30 mm to (110.5, 99.1)
- moved R7 6.30 mm to (109.2, 91.4)
- moved U$3 6.30 mm to (110.5, 95.9)
- moved D3 4.97 mm to (139.1, 100.3), turned to 270 degrees
- moved U$4 4.97 mm to (139.1, 100.3), turned to 270 degrees
- moved C1 3.84 mm to (148.6, 26.7)
- moved R9 3.35 mm to (40.7, 62.8), turned to 270 degrees
- moved X2 3.19 mm to (148.3, 107.3)
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Connections:
- net N$11: now also VT2.1; no longer VT2.G
- net N$18: now also VT2.2(PAD); no longer VT2.D
- net N$24: now also VT2.3; no longer VT2.S
- net N$25: now also C11.-
- net N$26: now also C11.+; no longer C6.+
- net N$29: now also C6.+
Routing:
- net GROUND: track 0.00 -> 203.8 mm, vias 3 -> 7
- net GND: track 451.5 -> 302.6 mm, vias 0 -> 2
- net BL-PWM: track 164.5 -> 111.6 mm, vias 0 -> 2
- net LED+: track 80.4 -> 42.7 mm
- net K2: track 225.8 -> 259.3 mm
- net K1: track 223.8 -> 252.3 mm
- net LED-FR: track 222.9 -> 245.5 mm
- net N$41: track 0.67 -> 21.6 mm
- net N$4: track 20.3 -> 0.00 mm, vias 2 -> 0
- net N$5: track 20.3 -> 0.00 mm, vias 2 -> 0
- net +3V3: track 220.9 -> 238.3 mm
- net N$30: track 179.9 -> 194.2 mm
- net N$29: track 34.9 -> 42.3 mm
- net N$18: track 14.0 -> 19.7 mm
- net N$31: track 23.2 -> 27.3 mm
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
Commit message: Релиз
Connections:
- new net N$3: PAD10.1, PAD12.1, PAD5.1, PAD7.1
- net LED+: now also PAD11.1, PAD9.1
- net LED-: now also PAD6.1, PAD8.1
Routing:
- net N$3: track 0.00 -> 92.4 mm
- net LED+: track 42.7 -> 84.6 mm
- net LED-: track 24.3 -> 34.0 mm
- added copper zone on layer 16, net GROUND
Changed lines of the file:
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@@
 <wire x1="28.3225" y1="46.97" x2="22.29" y2="53.0025" width="1.27" layer="16"/>
 <wire x1="22.29" y1="53.0025" x2="22.29" y2="56.495" width="1.27" layer="16"/>
-<wire x1="22.29" y1="74.91" x2="22.245" y2="74.9325" width="0" layer="19" extent="16-16"/>
+<contactref element="PAD9" pad="1"/>
+<contactref element="PAD11" pad="1"/>
+<wire x1="12" y1="43.0475" x2="12" y2="46.205" width="2.54" layer="16"/>
+<wire x1="12" y1="46.205" x2="16.39375" y2="50.59875" width="2.54" layer="16"/>
+<wire x1="16.39375" y1="50.59875" x2="22.29" y2="56.495" width="2.54" layer="16"/>
+<wire x1="12" y1="29.1475" x2="13.2725" y2="29.1475" width="2.54" layer="16"/>
+<wire x1="13.2725" y1="29.1475" x2="16.51" y2="32.385" width="2.54" layer="16"/>
+<wire x1="16.51" y1="32.385" x2="16.51" y2="50.4825" width="2.54" layer="16"/>
+<wire x1="16.51" y1="50.4825" x2="16.39375" y2="50.59875" width="2.54" layer="16"/>
+<wire x1="22.245" y1="74.9325" x2="22.2675" y2="74.9325" width="2.54" layer="16"/>
+<wire x1="22.2675" y1="74.9325" x2="22.29" y2="74.91" width="2.54" layer="16"/>
 </signal>
 <signal name="LED-">
 <contactref element="L2" pad="P$2"/>
-<wire x1="22.65" y1="111.85" x2="26" y2="108.5" width="2.54" layer="16"/>
-<wire x1="26" y1="108.5" x2="26" y2="89.055" width="2.54" layer="16"/>
 <wire x1="26" y1="89.055" x2="26.1" y2="88.955" width="2.54" layer="16"/>
+<contactref element="PAD8" pad="1"/>
+<contactref element="PAD6" pad="1"/>
+<wire x1="26.1" y1="88.955" x2="16.8575" y2="98.1975" width="2.54" layer="16"/>
+<wire x1="16.8575" y1="98.1975" x2="12" y2="98.1975" width="2.54" layer="16"/>
+<wire x1="12" y1="84.615" x2="21.76" y2="84.615" width="2.54" layer="16"/>
+<wire x1="21.76" y1="84.615" x2="26.1" y2="88.955" width="2.54" layer="16"/>
 </signal>
 <signal name="N$7">
@@
 <wire x1="5.25" y1="17.9275" x2="18.1815" y2="4.996" width="0.508" layer="16"/>
 <wire x1="78.996" y1="4.996" x2="81" y2="7" width="0.508" layer="16"/>
+<polygon width="0.4064" layer="16" isolate="1.27" orphans="yes" rank="6">
+<vertex x="0" y="128.27"/>
+<vertex x="160.02" y="128.27"/>
+<vertex x="160.02" y="-0.635"/>
+<vertex x="-0.3175" y="-0.635"/>
+<vertex x="-0.3175" y="127.9525"/>
+<vertex x="-0.3175" y="128.27"/>
+</polygon>
 </signal>
 <signal name="K2">
@@
 <contactref element="X2" pad="7"/>
 </signal>
+<signal name="N$3">
+<contactref element="PAD7" pad="1"/>
+<contactref element="PAD5" pad="1"/>
+<contactref element="PAD10" pad="1"/>
+<contactref element="PAD12" pad="1"/>
+<wire x1="12" y1="104.915" x2="8.255" y2="101.17" width="2.54" layer="16"/>
+<wire x1="8.255" y1="26.9425" x2="12" y2="23.1975" width="2.54" layer="16"/>
+<wire x1="8.255" y1="101.17" x2="8.255" y2="91.1225" width="2.54" layer="16"/>
+<wire x1="8.255" y1="91.1225" x2="8.255" y2="36.5125" width="2.54" layer="16"/>
+<wire x1="8.255" y1="36.5125" x2="8.255" y2="26.9425" width="2.54" layer="16"/>
+<wire x1="12" y1="36.6475" x2="8.39" y2="36.6475" width="2.54" layer="16"/>
+<wire x1="8.39" y1="36.6475" x2="8.255" y2="36.5125" width="2.54" layer="16"/>
+<wire x1="12" y1="91.015" x2="11.8925" y2="91.1225" width="2.54" layer="16"/>
+<wire x1="11.8925" y1="91.1225" x2="8.255" y2="91.1225" width="2.54" layer="16"/>
+</signal>
 </signals>

Commit message: _)
Parts:
- U$3: value IC-TL431DBV -> IC-TL431CDBZR; device Flamberm:SOT95P280X145-5 -> Flamberm:SOT95P240X115-3
- moved U$3 0.32 mm to (110.5, 95.6), turned to 270 degrees
Connections:
- net GND: now also U$3.3; no longer U$3.5
- net N$23: now also U$3.2; no longer U$3.4
- net N$31: now also U$3.1; no longer U$3.3
Routing:
- net GND: track 302.6 -> 303.7 mm
- net N$23: track 7.40 -> 6.86 mm
Changed lines of the file:
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@@
 </layers>
 <board>
+<fusionsync huburn="a.cGVyc29uYWw6dWUyOGRlMGUz" projecturn="a.cGVyc29uYWw6dWUyOGRlMGUzIzIwMTgxMjA3MTY0MzUzMzMx" f3durn="urn:adsk.wipprod:dm.lineage:CbOk_p9-Sm28mP2tJHSDlw" pcbguid="25285c78-3eb6-47c6-8325-666efd53a6fb" lastpulledtime="" lastsyncedchangeguid="d28009d4-24da-5f07-1719-9be39d882890"/>
 <plain>
 <wire x1="0" y1="0" x2="160" y2="0" width="0" layer="20"/>
@@
 <attribute name="VALUE" x="132.6642" y="106.0958" size="1.27" layer="27" ratio="10" rot="R180"/>
 </element>
-<element name="U$3" library="Flamberm" library_urn="urn:adsk.eagle:library:2654185" package="SOT95P280X145-5" package3d_urn="urn:adsk.eagle:package:4135333/1" value="IC-TL431DBV" x="110.49" y="95.885" smashed="yes" rot="MR180">
-<attribute name="NAME" x="108.712" y="98.933" size="1.27" layer="26" ratio="10" rot="MR270"/>
-<attribute name="VALUE" x="113.538" y="98.933" size="1.27" layer="28" ratio="10" rot="MR270"/>
+<element name="U$3" library="Flamberm" library_urn="urn:adsk.eagle:library:2654185" package="SOT95P240X115-3" package3d_urn="urn:adsk.eagle:package:4135509/1" value="IC-TL431CDBZR" x="110.49" y="95.5675" smashed="yes" rot="MR270">
+<attribute name="NAME" x="113.538" y="97.3455" size="1.27" layer="26" ratio="10" rot="MR0"/>
+<attribute name="VALUE" x="113.538" y="92.5195" size="1.27" layer="28" ratio="10" rot="MR0"/>
 </element>
 <element name="R7" library="Flamberm" library_urn="urn:adsk.eagle:library:2654185" package="RESC3216X60" package3d_urn="urn:adsk.eagle:package:4015759/1" value="220R" x="109.22" y="91.44" smashed="yes" rot="MR0">
@@
 <wire x1="49.8475" y1="88.5825" x2="49.8475" y2="89.535" width="0.508" layer="16"/>
 <contactref element="C2" pad="2"/>
-<contactref element="U$3" pad="5"/>
+<contactref element="U$3" pad="3"/>
 <contactref element="R18" pad="1"/>
 <contactref element="C7" pad="-"/>
@@
 <wire x1="114.6175" y1="94.5775" x2="114.6175" y2="91.313" width="0.508" layer="16"/>
 <wire x1="114.6175" y1="91.313" x2="115.8875" y2="90.043" width="0.508" layer="16"/>
-<wire x1="111.7321" y1="94.935" x2="114.26" y2="94.935" width="0.508" layer="16"/>
-<wire x1="114.26" y1="94.935" x2="114.6175" y2="94.5775" width="0.508" layer="16"/>
 <wire x1="127.762" y1="111.125" x2="120.9675" y2="111.125" width="0.508" layer="16"/>
 <wire x1="120.9675" y1="111.125" x2="116.205" y2="106.3625" width="0.508" layer="16"/>
@@
 <wire x1="63.8175" y1="106.3625" x2="61.9125" y2="104.4575" width="0.508" layer="16"/>
 <wire x1="60.96" y1="104.4575" x2="49.8475" y2="104.4575" width="0.508" layer="1"/>
+<wire x1="114.6175" y1="94.5775" x2="110.5245" y2="94.5775" width="0.508" layer="16"/>
+<wire x1="110.5245" y1="94.5775" x2="110.49" y2="94.543" width="0.508" layer="16"/>
 </signal>
 <signal name="+5V">
@@
 <signal name="N$31">
 <contactref element="OK1" pad="2"/>
-<contactref element="U$3" pad="3"/>
+<contactref element="U$3" pad="1"/>
 <contactref element="C8" pad="1"/>
-<wire x1="107.95" y1="96.52" x2="108.2675" y2="96.8375" width="0.508" layer="16"/>
-<wire x1="108.2675" y1="96.8375" x2="108.27" y2="96.835" width="0.508" layer="16"/>
-<wire x1="108.27" y1="96.835" x2="109.2479" y2="96.835" width="0.508" layer="16"/>
 <wire x1="108.84" y1="99.06" x2="107.95" y2="98.17" width="0.508" layer="16"/>
-<wire x1="107.95" y1="98.17" x2="107.95" y2="96.52" width="0.508" layer="16"/>
 <wire x1="107.95" y1="93.6625" x2="109.22" y2="92.3925" width="0.508" layer="16"/>
 <wire x1="109.22" y1="92.3925" x2="109.22" y2="88.265" width="0.508" layer="16"/>
 <wire x1="109.22" y1="88.265" x2="107.95" y2="86.995" width="0.508" layer="16"/>
 <wire x1="107.95" y1="86.995" x2="107.95" y2="74.6125" width="0.508" layer="16"/>
+<wire x1="107.95" y1="98.17" x2="107.95" y2="96.52" width="0.508" layer="16"/>
 <wire x1="107.95" y1="96.52" x2="107.95" y2="93.6625" width="0.508" layer="16"/>
+<wire x1="107.95" y1="96.52" x2="108.022" y2="96.592" width="0.508" layer="16"/>
+<wire x1="108.022" y1="96.592" x2="109.54" y2="96.592" width="0.508" layer="16"/>
 </signal>
 <signal name="N$22">
@@
 </signal>
 <signal name="N$23">
-<contactref element="U$3" pad="4"/>
+<contactref element="U$3" pad="2"/>
 <contactref element="R11" pad="1"/>
 <contactref element="C8" pad="2"/>
@@
 <wire x1="112.42" y1="99.34" x2="114.6175" y2="99.34" width="0.508" layer="16"/>
 <wire x1="114.6175" y1="97.8275" x2="114.6175" y2="99.34" width="0.508" layer="16"/>
-<wire x1="111.7321" y1="96.835" x2="113.625" y2="96.835" width="0.508" layer="16"/>
-<wire x1="113.625" y1="96.835" x2="114.6175" y2="97.8275" width="0.508" layer="16"/>
+<wire x1="111.44" y1="96.592" x2="112.14" y2="97.292" width="0.508" layer="16"/>
+<wire x1="112.14" y1="97.292" x2="112.14" y2="99.06" width="0.508" layer="16"/>
 </signal>
 <signal name="N$30">
@@
 </note>
 <note version="8.3" severity="warning">
+Since Version 8.3, EAGLE supports Fusion synchronisation.
+This feature will not be available in this version and saving
+the document will break the link to the Fusion PCB feature.
+</note>
+<note version="8.3" severity="warning">

Commit message: _
Parts:
- removed R13: 2R2, Flamberm:MF-025
- R14: value 2R2 -> 1R8
- R2, R3: device Flamberm:MF-025 -> Flamberm:RESC2012X50
- moved R2 3.49 mm to (47.3, 93.3)
- moved R3 3.49 mm to (52.4, 93.3)
Connections:
- net N$30: no longer R13.1
- net N$33: no longer R13.2
Routing:
- net GND: track 303.7 -> 293.2 mm
- net ON-OFF: track 133.7 -> 139.9 mm
- net BL-PWM: track 111.6 -> 117.9 mm
- net N$33: track 24.0 -> 19.3 mm
- net N$30: track 194.2 -> 191.7 mm
- net GROUND: track 203.8 -> 205.9 mm
- net N$9: track 3.49 -> 2.76 mm
- net N$8: track 3.49 -> 2.76 mm
