File: Monitors/Samsung 743n/PowerBoard.sch (EAGLE design)
At the start: 57 parts, among them IC2 HV9961NG-G, T1 TRANS-1/1EFD25-10, X1 CON-MONPANEL, X2 CON-2MM-12P

Commit message: Понемногу
Parts:
- L2: value SL1016T -> SL1016T-123K
- R6: value 68K -> 75K
- R8: value 1R1 -> 2R2
- U$1: value PW-NCP12NCP1200D -> POWER-NCP12DIP; device Namenlos:PW-NCP12NCP1200D -> Flamberm:POWER-NCP12DIP
Other:
- note added: "Pri: 109 turns, 1x0.2mm Sec: 5 turns, 2x0.56mm Prim. Ind.= 3,557 mH Gap = 0.24"
- note added: "Rcs = 1.875 Ohm"
- note removed: "Pri: 65 turns, 1x0.355mm Sec: 3 turns, 8x0.355mm Prim. Ind.= 1,3 mH"
Changed lines of the file:
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@@
 <part name="R4" library="Flamberm" library_urn="urn:adsk.eagle:library:2654185" deviceset="R_" device="MF-0125" package3d_urn="urn:adsk.eagle:package:2654533/2" value="160K"/>
 <part name="IC2" library="Flamberm" library_urn="urn:adsk.eagle:library:2654185" deviceset="HV9910B" device="NG" package3d_urn="urn:adsk.eagle:package:2654601/1" value="HV9961NG-G"/>
-<part name="R6" library="Flamberm" library_urn="urn:adsk.eagle:library:2654185" deviceset="R_" device="R0805" package3d_urn="urn:adsk.eagle:package:4015756/1" value="68K"/>
+<part name="R6" library="Flamberm" library_urn="urn:adsk.eagle:library:2654185" deviceset="R_" device="R0805" package3d_urn="urn:adsk.eagle:package:4015756/1" value="75K"/>
 <part name="VT2" library="Namenlos" deviceset="FET-N" device="DPAK" value="STD1NK60T4"/>
-<part name="L2" library="Namenlos" deviceset="INDUCTOR" device="SL1016" value="SL1016T"/>
+<part name="L2" library="Namenlos" deviceset="INDUCTOR" device="SL1016" value="SL1016T-123K"/>
 <part name="D1" library="Flamberm" library_urn="urn:adsk.eagle:library:2654185" deviceset="DIODE_" device="ES1J" package3d_urn="urn:adsk.eagle:package:2654514/2" value="ES1J"/>
-<part name="R8" library="Flamberm" library_urn="urn:adsk.eagle:library:2654185" deviceset="R_" device="MF-05" package3d_urn="urn:adsk.eagle:package:2654531/2" value="1R1"/>
+<part name="R8" library="Flamberm" library_urn="urn:adsk.eagle:library:2654185" deviceset="R_" device="MF-05" package3d_urn="urn:adsk.eagle:package:2654531/2" value="2R2"/>
 <part name="R9" library="Flamberm" library_urn="urn:adsk.eagle:library:2654185" deviceset="R_" device="R0805" package3d_urn="urn:adsk.eagle:package:4015756/1" value="39K"/>
 <part name="C6" library="Namenlos" deviceset="CAP-POL_" device="3528" value="22u 16V"/>
@@
 <part name="B1" library="rectifier" library_urn="urn:adsk.eagle:library:336" deviceset="KBL" device="" package3d_urn="urn:adsk.eagle:package:23884/1"/>
 <part name="C1" library="Flamberm" library_urn="urn:adsk.eagle:library:2654185" deviceset="CAP-POL_" device="E5-13-35-H" package3d_urn="urn:adsk.eagle:package:2654539/3" value="100u"/>
-<part name="U$1" library="Namenlos" deviceset="PW-NCP12*" device="NCP1200D"/>
+<part name="U$1" library="Flamberm" library_urn="urn:adsk.eagle:library:2654185" deviceset="POWER-NCP12*" device="DIP" package3d_urn="urn:adsk.eagle:package:7282522/1"/>
 <part name="P6KE200" library="Flamberm" library_urn="urn:adsk.eagle:library:2654185" deviceset="SUPRESSOR" device="DO-204AC" package3d_urn="urn:adsk.eagle:package:2654542/1"/>
 <part name="D2" library="Flamberm" library_urn="urn:adsk.eagle:library:2654185" deviceset="DIODE_" device="ES1J" package3d_urn="urn:adsk.eagle:package:2654514/2"/>
@@
 <sheet>
 <plain>
-<text x="99.06" y="149.86" size="1.778" layer="97">Pri: 65 turns, 1x0.355mm
-Sec: 3 turns, 8x0.355mm
-Prim. Ind.= 1,3 mH</text>
+<text x="99.06" y="149.86" size="1.778" layer="97">Pri: 109 turns, 1x0.2mm
+Sec: 5 turns, 2x0.56mm
+Prim. Ind.= 3,557 mH
+Gap = 0.24</text>
+<text x="83.82" y="33.02" size="1.778" layer="97">Rcs = 1.875 Ohm</text>
 </plain>
 <instances>

Commit message: почти
Parts:
- added C11: 10u 16V, Flamberm:CAP-POL_E2.5-7
- C2: device Namenlos:CAP_C50-024X044 -> Flamberm:CAP_C50-024X044
- C3: device Namenlos:CAP-POL_E2.5-7 -> Flamberm:CAP-POL_E2.5-7
- C4: device Namenlos:CAP-POL_E3.5-8 -> Flamberm:CAP-POL_E5-13,5
- C6: value 22u 16V -> 10u 16V; device Namenlos:CAP-POL_3528 -> Flamberm:CAP-POL_E2.5-7
- L2: device Namenlos:INDUCTORSL1016 -> Flamberm:INDUCTORSL1016
- NTC: device Namenlos:NTC-D12 -> Flamberm:NTC-D12
- OK1: device Namenlos:OPTOTRANSPC817 -> Flamberm:OPTOTRANSPC817
- Q1: device Namenlos:FET-NTO-220 -> Flamberm:FET-NTO-220
- R12: device Namenlos:R_MF-0125 -> Flamberm:R_MF-0125
- VT2: device Namenlos:FET-NDPAK -> Flamberm:FET-NDPAK
Connections:
- net N$25: now also C11.-
- net N$26: now also C11.+; no longer C6.+
- net N$29: now also C6.+
Other:
- moved on the sheet: R9

Commit message: Релиз
Connections:
- new net N$3: PAD10.P, PAD12.P, PAD5.P, PAD7.P
- net LED+: now also PAD11.P, PAD9.P
- net LED-: now also PAD6.P, PAD8.P
Changed lines of the file:
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@@
+</segment>
+</net>
+<net name="LED+" class="0">
+<segment>
+<pinref part="PAD9" gate="1" pin="P"/>
+<wire x1="60.96" y1="45.72" x2="58.42" y2="45.72" width="0.1524" layer="91"/>
+<pinref part="PAD11" gate="1" pin="P"/>
+<wire x1="58.42" y1="45.72" x2="45.72" y2="45.72" width="0.1524" layer="91"/>
+<wire x1="60.96" y1="35.56" x2="58.42" y2="35.56" width="0.1524" layer="91"/>
+<wire x1="58.42" y1="35.56" x2="58.42" y2="45.72" width="0.1524" layer="91"/>
+<junction x="58.42" y="45.72"/>
+<label x="45.72" y="45.72" size="1.778" layer="95"/>
+</segment>
+</net>
+<net name="LED-" class="0">
+<segment>
+<pinref part="PAD8" gate="1" pin="P"/>
+<wire x1="60.96" y1="68.58" x2="55.88" y2="68.58" width="0.1524" layer="91"/>
+<pinref part="PAD6" gate="1" pin="P"/>
+<wire x1="55.88" y1="68.58" x2="45.72" y2="68.58" width="0.1524" layer="91"/>
+<wire x1="60.96" y1="78.74" x2="55.88" y2="78.74" width="0.1524" layer="91"/>
+<wire x1="55.88" y1="78.74" x2="55.88" y2="68.58" width="0.1524" layer="91"/>
+<junction x="55.88" y="68.58"/>
+<label x="45.72" y="68.58" size="1.778" layer="95"/>
+</segment>
+</net>
+<net name="N$3" class="0">
+<segment>
+<pinref part="PAD7" gate="1" pin="P"/>
+<wire x1="60.96" y1="73.66" x2="58.42" y2="73.66" width="0.1524" layer="91"/>
+<wire x1="58.42" y1="73.66" x2="58.42" y2="83.82" width="0.1524" layer="91"/>
+<pinref part="PAD5" gate="1" pin="P"/>
+<wire x1="58.42" y1="83.82" x2="60.96" y2="83.82" width="0.1524" layer="91"/>
+<wire x1="58.42" y1="73.66" x2="53.34" y2="73.66" width="0.1524" layer="91"/>
+<wire x1="53.34" y1="73.66" x2="53.34" y2="40.64" width="0.1524" layer="91"/>
+<junction x="58.42" y="73.66"/>
+<pinref part="PAD10" gate="1" pin="P"/>
+<wire x1="53.34" y1="40.64" x2="60.96" y2="40.64" width="0.1524" layer="91"/>
+<pinref part="PAD12" gate="1" pin="P"/>
+<wire x1="53.34" y1="40.64" x2="53.34" y2="30.48" width="0.1524" layer="91"/>
+<wire x1="53.34" y1="30.48" x2="60.96" y2="30.48" width="0.1524" layer="91"/>
+<junction x="53.34" y="40.64"/>
 </segment>
 </net>

Commit message: _)
Parts:
- U$3: value IC-TL431DBV -> IC-TL431CDBZR; device Flamberm:IC-TL431DBV -> Flamberm:IC-TL431CDBZR
Changed lines of the file:
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@@
 <part name="OK1" library="Flamberm" library_urn="urn:adsk.eagle:library:2654185" deviceset="OPTOTRANS" device="PC817" package3d_urn="urn:adsk.eagle:package:2654547/2"/>
 <part name="C7" library="Flamberm" library_urn="urn:adsk.eagle:library:2654185" deviceset="CAP-POL_" device="E3.5-8" package3d_urn="urn:adsk.eagle:package:2654549/1" value="1000u 6.3V"/>
-<part name="U$3" library="Flamberm" library_urn="urn:adsk.eagle:library:2654185" deviceset="IC-TL431" device="DBV" package3d_urn="urn:adsk.eagle:package:4135333/1"/>
+<part name="U$3" library="Flamberm" library_urn="urn:adsk.eagle:library:2654185" deviceset="IC-TL431" device="CDBZR" package3d_urn="urn:adsk.eagle:package:4135509/1" value="IC-TL431CDBZR"/>
 <part name="R7" library="Flamberm" library_urn="urn:adsk.eagle:library:2654185" deviceset="R_" device="R1206" package3d_urn="urn:adsk.eagle:package:4015759/1" value="220R"/>
 <part name="R11" library="Flamberm" library_urn="urn:adsk.eagle:library:2654185" deviceset="R_" device="R1206" package3d_urn="urn:adsk.eagle:package:4015759/1" value="3k3"/>

Commit message: _
Parts:
- removed R13: 2R2, Flamberm:R_MF-025
- R14: value 2R2 -> 1R8
- R2, R3: device Flamberm:R_MF-025 -> Flamberm:R_R0805
Connections:
- net N$30: no longer R13.1
- net N$33: no longer R13.2
Changed lines of the file:
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@@
 <part name="B2" library="Flamberm" library_urn="urn:adsk.eagle:library:2654185" deviceset="BRIDGE" device="DBS" package3d_urn="urn:adsk.eagle:package:2654606/2"/>
 <part name="R1" library="Flamberm" library_urn="urn:adsk.eagle:library:2654185" deviceset="R_" device="R0805" package3d_urn="urn:adsk.eagle:package:4015756/1" value="39K"/>
-<part name="R2" library="Flamberm" library_urn="urn:adsk.eagle:library:2654185" deviceset="R_" device="MF-025" package3d_urn="urn:adsk.eagle:package:2654532/2" value="1K5"/>
-<part name="R3" library="Flamberm" library_urn="urn:adsk.eagle:library:2654185" deviceset="R_" device="MF-025" package3d_urn="urn:adsk.eagle:package:2654532/2" value="1K5"/>
+<part name="R2" library="Flamberm" library_urn="urn:adsk.eagle:library:2654185" deviceset="R_" device="R0805" package3d_urn="urn:adsk.eagle:package:4015756/1" value="1K5"/>
+<part name="R3" library="Flamberm" library_urn="urn:adsk.eagle:library:2654185" deviceset="R_" device="R0805" package3d_urn="urn:adsk.eagle:package:4015756/1" value="1K5"/>
 <part name="GND3" library="supply1" library_urn="urn:adsk.eagle:library:371" deviceset="GND" device=""/>
 <part name="GND4" library="supply1" library_urn="urn:adsk.eagle:library:371" deviceset="GND" device=""/>
@@
 <part name="C10" library="Flamberm" library_urn="urn:adsk.eagle:library:2654185" deviceset="CAP_" device="0805" package3d_urn="urn:adsk.eagle:package:4015421/2"/>
 <part name="T1" library="Flamberm" library_urn="urn:adsk.eagle:library:2654185" deviceset="TRANS-1/1" device="EFD25-10" package3d_urn="urn:adsk.eagle:package:2654554/3"/>
-<part name="R13" library="Flamberm" library_urn="urn:adsk.eagle:library:2654185" deviceset="R_" device="MF-025" package3d_urn="urn:adsk.eagle:package:2654532/2" value="2R2"/>
-<part name="R14" library="Flamberm" library_urn="urn:adsk.eagle:library:2654185" deviceset="R_" device="MF-025" package3d_urn="urn:adsk.eagle:package:2654532/2" value="2R2"/>
+<part name="R14" library="Flamberm" library_urn="urn:adsk.eagle:library:2654185" deviceset="R_" device="MF-025" package3d_urn="urn:adsk.eagle:package:2654532/2" value="1R8"/>
 <part name="D3" library="Flamberm" library_urn="urn:adsk.eagle:library:2654185" deviceset="DIODE_" device="TO-220-2" package3d_urn="urn:adsk.eagle:package:2654516/1"/>
 <part name="GND5" library="supply1" library_urn="urn:adsk.eagle:library:371" deviceset="GND" device=""/>
@@
 <attribute name="VALUE" x="100.584" y="145.415" size="1.778" layer="96" rot="MR180"/>
 </instance>
-<instance part="R13" gate="G$1" x="88.9" y="48.26" smashed="yes" rot="R90">
-<attribute name="NAME" x="87.4014" y="44.45" size="1.778" layer="95" rot="R90"/>
-<attribute name="VALUE" x="92.202" y="44.45" size="1.778" layer="96" rot="R90"/>
-</instance>
 <instance part="R14" gate="G$1" x="96.52" y="48.26" smashed="yes" rot="R90">
 <attribute name="NAME" x="95.0214" y="44.45" size="1.778" layer="95" rot="R90"/>
@@
 <wire x1="114.3" y1="35.56" x2="96.52" y2="35.56" width="0.1524" layer="91"/>
 <pinref part="C3" gate="C$1" pin="-"/>
-<wire x1="96.52" y1="35.56" x2="88.9" y2="35.56" width="0.1524" layer="91"/>
-<wire x1="88.9" y1="35.56" x2="78.74" y2="35.56" width="0.1524" layer="91"/>
+<wire x1="96.52" y1="35.56" x2="78.74" y2="35.56" width="0.1524" layer="91"/>
 <wire x1="78.74" y1="50.8" x2="78.74" y2="35.56" width="0.1524" layer="91"/>
 <pinref part="U$1" gate="G$1" pin="GND"/>
@@
 <wire x1="58.42" y1="127" x2="58.42" y2="124.46" width="0.1524" layer="91"/>
 <junction x="58.42" y="124.46"/>
-<pinref part="R13" gate="G$1" pin="1"/>
-<wire x1="88.9" y1="43.18" x2="88.9" y2="35.56" width="0.1524" layer="91"/>
-<junction x="88.9" y="35.56"/>
 <pinref part="R14" gate="G$1" pin="1"/>
 <wire x1="96.52" y1="43.18" x2="96.52" y2="35.56" width="0.1524" layer="91"/>
@@
 <pinref part="U$1" gate="G$1" pin="CS"/>
 <wire x1="43.18" y1="76.2" x2="45.72" y2="76.2" width="0.1524" layer="91"/>
-<wire x1="43.18" y1="60.96" x2="88.9" y2="60.96" width="0.1524" layer="91"/>
+<wire x1="43.18" y1="60.96" x2="96.52" y2="60.96" width="0.1524" layer="91"/>
 <pinref part="Q1" gate="G$1" pin="S"/>
-<wire x1="88.9" y1="60.96" x2="96.52" y2="60.96" width="0.1524" layer="91"/>
 <wire x1="96.52" y1="68.58" x2="96.52" y2="60.96" width="0.1524" layer="91"/>
 <wire x1="43.18" y1="76.2" x2="43.18" y2="60.96" width="0.1524" layer="91"/>
-<pinref part="R13" gate="G$1" pin="2"/>
-<wire x1="88.9" y1="53.34" x2="88.9" y2="60.96" width="0.1524" layer="91"/>
-<junction x="88.9" y="60.96"/>
 <pinref part="R14" gate="G$1" pin="2"/>
 <wire x1="96.52" y1="53.34" x2="96.52" y2="60.96" width="0.1524" layer="91"/>
