File: LED/PocketLamp/MainBoard.brd (EAGLE design)
At the start: 77.5 x 20.9 mm, 41 parts, among them P1 BATTERY18650X1, SW1 BUTTON2X4-SIDE, U1 POWER-STC4054, X1 USB-MINIMICROMICRO

Commit message: _
Parts:
- removed LED2: GREEN, Flamberm:LED1206
- removed R1: 2K, Flamberm:RESC2012X50
- LED10, LED11, LED12, LED13, LED14, LED15, LED16, LED17, LED18, LED3, LED4, LED5, LED6, LED7, LED8, LED9: value LED_5630 -> LED_5730
- moved SW1 76.0 mm to (0.83, 15.9), turned to 90 degrees
- moved R11 4.18 mm to (74.6, 14.6), turned to 90 degrees
- moved X1 0.64 mm to (74.6, 4.76)
- turned LED10 to 270 degrees
- turned LED11 to 270 degrees
- turned LED12 to 270 degrees
- turned LED13 to 270 degrees
- turned LED14 to 270 degrees
- turned LED15 to 270 degrees
- turned LED16 to 270 degrees
- turned LED17 to 270 degrees
- turned LED18 to 270 degrees
- turned LED3 to 270 degrees
- turned LED4 to 270 degrees
- turned LED5 to 270 degrees
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Connections:
- removed net N$27: LED10.A, LED10.A1, R11.2
- removed net N$3: LED2.A, R1.1
- removed net N$4: LED10.C, LED11.C, LED12.C, LED13.C, LED14.C, LED15.C, LED16.C, LED17.C, LED18.C, LED3.C, LED4.C, LED5.C, LED6.C, LED7.C, LED8.C, LED9.C, P1.+, U1.3
- removed net N$7: R10.1, R11.1, R12.1, R13.1, R14.1, R15.1, R16.1, R17.1, R18.1, R19.1, R4.1, R5.1, R6.1, R7.1, R8.1, R9.1, SW1.1
- new net N$11: LED6.C, R7.2
- new net N$23: LED18.C, R19.2
- new net N$84: LED10.A, LED10.A1, LED11.A, LED11.A1, LED12.A, LED12.A1, LED13.A, LED13.A1, LED14.A, LED14.A1, LED15.A, LED15.A1, LED16.A, LED16.A1, LED17.A, LED17.A1, LED18.A, LED18.A1, LED3.A, LED3.A1, LED4.A, LED4.A1, LED5.A, LED5.A1, LED6.A, LED6.A1, LED7.A, LED7.A1, LED8.A, LED8.A1, LED9.A, LED9.A1, SW1.2
- net +5V: no longer R1.2
- net GND: now also R10.1, R11.1, R12.1, R13.1, R14.1, R15.1, R16.1, R17.1, R18.1, R19.1, R4.1, R5.1, R6.1, R7.1, R8.1, R9.1; no longer LED2.C, SW1.2
- net N$10: now also LED5.C, R6.2; no longer LED11.A, LED11.A1, R12.2
- net N$12: now also LED7.C, R8.2; no longer LED5.A, LED5.A1, R6.2
- net N$13: now also LED8.C, R9.2; no longer LED12.A, LED12.A1, R13.2
- net N$14: now also LED9.C, R10.2; no longer LED13.A, LED13.A1, R14.2
- net N$15: now also LED10.C, R11.2; no longer LED6.A, LED6.A1, R7.2
- net N$16: now also LED11.C, R12.2; no longer LED14.A, LED14.A1, R15.2
- net N$17: now also LED12.C, R13.2; no longer LED15.A, LED15.A1, R16.2
- net N$18: now also LED13.C, R14.2; no longer LED7.A, LED7.A1, R8.2
- net N$19: now also LED14.C, R15.2; no longer LED16.A, LED16.A1, R17.2
- net N$20: now also LED15.C, R16.2; no longer LED17.A, LED17.A1, R18.2
- net N$21: now also LED16.C, R17.2; no longer LED8.A, LED8.A1, R9.2
- net N$22: now also LED17.C, R18.2; no longer LED18.A, LED18.A1, R19.2
- net N$24: now also P1.+, SW1.1, U1.3; no longer LED9.A, LED9.A1, R10.2
- net N$6: now also LED3.C; no longer LED3.A, LED3.A1
- net N$9: now also LED4.C; no longer LED4.A, LED4.A1
Routing:
- net N$4: track 140.1 -> 0.00 mm
- net N$84: track 0.00 -> 111.6 mm
- net N$7: track 82.8 -> 0.00 mm
- net GND: track 51.6 -> 115.1 mm
- net N$24: track 5.43 -> 65.4 mm
- net N$27: track 5.04 -> 0.00 mm
- net N$3: track 2.79 -> 0.00 mm
- net N$23: track 0.00 -> 2.73 mm
- net N$11: track 0.00 -> 2.73 mm
- net N$10: track 5.43 -> 2.73 mm
- net N$17: track 5.43 -> 2.73 mm
- net N$14: track 5.43 -> 2.73 mm
- net N$20: track 5.43 -> 2.73 mm
- net N$19: track 5.43 -> 2.73 mm
- net N$13: track 5.43 -> 2.73 mm
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- added copper zone on layer 1, net N$24
- removed copper zone on layer 1, net N$4
