File: Power/POWER/Power 5V-4A, 12V-1A.brd (EAGLE design)
At the start: 95.2 x 61.9 mm, 48 parts, among them T1 TRANS-2/2, U1 POWER-UC3843B, X1 CON-7.62-02P, X2 CON-5.08-03P, X3 CON-5.08-03P

Commit message: _
Parts:
- C10: value 1000u 25V -> 2200u 25V
Changed lines of the file:
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@@
 <attribute name="VALUE" x="32.766" y="29.0751" size="1.27" layer="28" rot="MR0" align="top-center"/>
 </element>
-<element name="C10" library="Flamberm" library_urn="urn:adsk.eagle:library:2654185" package="E5-10,5" package3d_urn="urn:adsk.eagle:package:2654545/1" value="1000u 25V" x="83.82" y="6.35" smashed="yes" rot="R270">
+<element name="C10" library="Flamberm" library_urn="urn:adsk.eagle:library:2654185" package="E5-10,5" package3d_urn="urn:adsk.eagle:package:2654545/1" value="2200u 25V" x="83.82" y="6.35" smashed="yes" rot="R270">
 <attribute name="NAME" x="86.5632" y="1.651" size="1.27" layer="25" ratio="10" rot="R270"/>
 <attribute name="VALUE" x="80.5942" y="9.4742" size="1.27" layer="27" ratio="10" rot="R270"/>
