File: Power/POWER/Power 5V-4A, 12V-1A.sch (EAGLE design)
At the start: 45 parts, among them T1 TRANS-2/2, U1 POWER-UC3843B, X1 CON-7.62-02P, X2 CON-5.08-03P, X3 CON-5.08-03P

Commit message: _
Parts:
- C10: value 1000u 25V -> 2200u 25V
Changed lines of the file:
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@@
 <drawing>
 <settings>
-<setting alwaysvectorfont="no"/>
+<setting alwaysvectorfont="yes"/>
 <setting verticaltext="up"/>
 </settings>
@@
 <part name="C8" library="Flamberm" library_urn="urn:adsk.eagle:library:2654185" deviceset="CAP-POL_" device="E5-10.5" package3d_urn="urn:adsk.eagle:package:2654545/1" value="1000u 10V"/>
 <part name="C9" library="Flamberm" library_urn="urn:adsk.eagle:library:2654185" deviceset="CAP_" device="1206" package3d_urn="urn:adsk.eagle:package:4015425/2" value="220p"/>
-<part name="C10" library="Flamberm" library_urn="urn:adsk.eagle:library:2654185" deviceset="CAP-POL_" device="E5-10.5" package3d_urn="urn:adsk.eagle:package:2654545/1" value="1000u 25V"/>
+<part name="C10" library="Flamberm" library_urn="urn:adsk.eagle:library:2654185" deviceset="CAP-POL_" device="E5-10.5" package3d_urn="urn:adsk.eagle:package:2654545/1" value="2200u 25V"/>
 <part name="C11" library="Flamberm" library_urn="urn:adsk.eagle:library:2654185" deviceset="CAP_" device="1206" package3d_urn="urn:adsk.eagle:package:4015425/2" value="220p"/>
 <part name="TL1" library="Flamberm" library_urn="urn:adsk.eagle:library:2654185" deviceset="IC-TL431" device="CDBZR" package3d_urn="urn:adsk.eagle:package:4135509/1"/>
