File: MicroControl/FlashArduinoProgrammer/FlashProgrammer03.sch (EAGLE design)
At the start: 11 parts, among them U1 VREG-LD2985, X1 POGOPIN, X2 POGOPIN, X3 POGOPIN, X4 POGOPIN, X5 POGOPIN, X6 POGOPIN, X7 POGOPIN, X8 POGOPIN

Commit message: _
Parts:
- removed X1, X2, X3, X4, X5, X6, X7, X8: POGOPIN, Flamberm:POGOPIN
- added PAD1, PAD2, PAD3, PAD4, PAD5, PAD6, PAD7, PAD8: (no value), wirepad:1,6/0,8
Connections:
- removed net GND: U$1.GND@1, U$2.GND, U1.GND, X4.S
- removed net N$7 (its old number): U$2.A1, X5.S
- removed net P2: U$2.A2, X2.S
- removed net P3,P8,P7: U$2.OE, U$2.VCCA, U1.VOUT, X3.S, X7.S, X8.S
- new net N$10: PAD5.P, U$2.A3
- new net N$11: PAD1.P, U$2.A4
- new net N$6: U$1.16, U$2.B3
- new net N$9: PAD2.P, U$2.A2
- net N$2: now also PAD4.P, U$1.GND@1, U$2.GND, U1.GND; no longer U$1.15, U$2.B3
- net N$3: now also U$1.15; no longer U$1.16
- net N$4: now also PAD3.P, PAD7.P, PAD8.P, U$2.OE, U$2.VCCA, U1.VOUT; no longer U$2.A4, X1.S
- net N$8: now also PAD6.P, U$2.A1; no longer U$2.A3, X6.S
Other:
- moved on the sheet: U$2, U1
