File: USB-COM25/Integrated Adapter.brd (EAGLE design)
At the start: 37 x 30 mm, 1 part, among them IC1 FT232RL

Commit message: _
Parts:
- added C1: 100n, Flamberm:CAP0805
- added C2, C3, C4, C5: 0.1u, Flamberm:CAPMP3317X180
- added IC2: ADM213EARZ, Flamberm:SO28L
- added R1: 110K, Flamberm:RESC2012X50
- added X1: DP-25, Flamberm:DB-25F_SMD
- added X3: USB-MINIMICROMICRO, Flamberm:USB-B-MICRO-SMD
- moved IC1 21.0 mm to (19.7, 12.1), flipped to the bottom, turned to 270 degrees
Connections:
- removed net VCC: IC1.20
- removed net VCCIO: IC1.4
- new net +5V: C4.2, IC1.20, IC1.4, IC2.11, R1.1, X3.VBUS
- new net C1+: C2.1, IC2.12
- new net C1-: C2.2, IC2.14
- new net C2+: C3.1, IC2.15
- new net C2-: C3.2, IC2.16
- new net N$1: IC1.15, X3.D+
- new net N$10: IC1.9, IC2.26
- new net N$11: IC1.10, IC2.22
- new net N$12: IC1.11, IC2.19
- new net N$13: IC2.2, X1.P3
- new net N$14: IC2.9, X1.P2
- new net N$15: IC2.1, X1.P4
- new net N$16: IC2.18, X1.P5
- new net N$17: IC2.27, X1.P6
- new net N$18: IC2.3, X1.P20
- new net N$19: IC2.4, X1.P22
- new net N$2: IC1.16, X3.D-
- new net N$20: IC2.23, X1.P8
- new net N$3: C1.2, IC1.17
- new net N$4: IC1.19, R1.2
- new net N$5: IC1.1, IC2.7
- new net N$6: IC1.2, IC2.6
- new net N$7: IC1.3, IC2.20
- new net N$8: IC1.5, IC2.8
- new net N$9: IC1.6, IC2.5
- new net V+: C4.1, IC2.13
- new net V-: C5.2, IC2.17
- net GND: now also C1.1, C5.1, IC1.26, IC2.10, X1.P7, X3.GND, X3.SHIELD1, X3.SHIELD2, X3.SHIELD3
Routing:
- net N$16: track 0.00 -> 22.5 mm
- net N$19: track 0.00 -> 19.1 mm, vias 0 -> 1
- net N$14: track 0.00 -> 18.0 mm
- net N$18: track 0.00 -> 15.4 mm, vias 0 -> 1
- net N$20: track 0.00 -> 15.0 mm
- net N$17: track 0.00 -> 13.0 mm
- net N$13: track 0.00 -> 7.96 mm
- net N$15: track 0.00 -> 5.04 mm

Commit message: _
Parts:
- moved R1 24.8 mm to (23.5, 20.3), turned to 180 degrees
- moved X3 24.3 mm to (18.4, 1.27), turned to 90 degrees
- moved C1 23.5 mm to (26.9, 15.6), turned to 90 degrees
- moved C2 9.67 mm to (10.2, 4.45), turned to 90 degrees
- moved C4 7.73 mm to (14.0, 5.71), turned to 0 degrees
- moved C5 3.18 mm to (24.8, 8.89), turned to 90 degrees
- moved IC1 2.29 mm to (21.0, 14.0), turned to 90 degrees
- moved C3 1.42 mm to (22.2, 6.99)
Connections:
- net N$1 renamed USB_P
- net N$2 renamed USB_N
Routing:
- net GND: track 0.00 -> 80.3 mm, vias 0 -> 4
- net +5V: track 0.00 -> 41.7 mm, vias 0 -> 3
- net USB_P: track 0.00 -> 26.8 mm, vias 0 -> 1
- net USB_N: track 0.00 -> 26.3 mm, vias 0 -> 1
- net N$6: track 0.00 -> 13.7 mm, vias 0 -> 1
- net N$5: track 0.00 -> 13.3 mm, vias 0 -> 1
- net N$9: track 0.00 -> 12.8 mm, vias 0 -> 1
- net N$12: track 0.00 -> 12.0 mm, vias 0 -> 1
- net N$7: track 0.00 -> 11.1 mm, vias 0 -> 1
- net C1+: track 0.00 -> 9.99 mm
- net N$10: track 0.00 -> 9.74 mm, vias 0 -> 1
- net N$8: track 0.00 -> 8.50 mm, vias 0 -> 1
- net N$4: track 0.00 -> 6.62 mm
- net N$11: track 0.00 -> 6.40 mm, vias 0 -> 1
- net V+: track 0.00 -> 5.03 mm
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